File: hardware/ecp5_mainboard/power.sch (KiCad schematic (older format))
At the start: 32 parts

Commit message: ecp5_mainboard/power: Add 1.8V, 2.5V and 3.3V regulators
Signed-off-by: David Shah <davey1576@gmail.com>
Parts:
- added C? (x9): 10µ, symbol Device:C_Small
- added C? (x3): 120p, symbol Device:C_Small
- added D? (x3): GREEN, symbol Device:LED
- added L? (x3): 470n/IHLP1212, symbol Device:L
- added Q? (x3): BSH111BKR, Package_TO_SOT_SMD:SOT-23, symbol Transistor_FET:2N7002
- added R?: 453k, symbol Device:R_Small
- added R? (x3): 100k, symbol Device:R_Small
- added R?: 316k, symbol Device:R_Small
- added R?: 200k, symbol Device:R_Small
- added R? (x3): 10k, symbol Device:R_Small
- added R? (x3): 1k, symbol Device:R_Small
- added U? (x3): TPS62823, symbol eco_power:TPS62823
- Q?: value 2N7002 -> BSH111BKR
- R?: value 10k -> 4.7k
Connections:
- net labels added: +1V8, +2V5, +3V3, 1V8_EN, 1V8_PG, 2V5_EN, 2V5_PG, 3V3_EN, 3V3_PG
- wire segments 141 -> 280
Other:
- moved on the sheet: Q?

Commit message: ecp5_mainboard/power: Add 1.35V DDR3 and 1.2V FPGA core regulators
Signed-off-by: David Shah <davey1576@gmail.com>
Parts:
- added C? (x5): 10µ, symbol Device:C_Small
- added C?: 120p, symbol Device:C_Small
- added C?: 100n, symbol Device:C_Small
- added C?: 1.8n, symbol Device:C_Small
- added C?: 180p, symbol Device:C_Small
- added C?: 750p, symbol Device:C_Small
- added D? (x2): GREEN, symbol Device:LED
- added L?: 470n/IHLP1212, symbol Device:L
- added L?: 800nH/XAL5030, symbol Device:L
- added Q? (x2): BSH111BKR, Package_TO_SOT_SMD:SOT-23, symbol Transistor_FET:2N7002
- added R?: 124k, symbol Device:R_Small
- added R?: 100k, symbol Device:R_Small
- added R? (x4): 10k, symbol Device:R_Small
- added R? (x2): 1k, symbol Device:R_Small
- added R?: 10, symbol Device:R_Small
- added R?: 47k, symbol Device:R_Small
- added R?: 4.7k, symbol Device:R_Small
- added R?: 470k, symbol Device:R_Small
- added U?: TPS62823, symbol eco_power:TPS62823
- added U?: LM21212-2, symbol eco_power:LM21212-2
Connections:
- net labels added: +1V2, +1V35, 1V2_EN, 1V2_PG, 1V35_EN, 1V35_PG
- wire segments 280 -> 413
- no-connect marks 2 -> 3
Other:
- note added: "1.35V/3A"
- note added: "1.8V/3A"
- note added: "2.5V/3A"
- note added: "3.3V/3A"
- moved on the sheet: Q?

Commit message: ecp5_mainboard/power: Add 1.2V analog and termination supplies
Signed-off-by: David Shah <davey1576@gmail.com>
Parts:
- added C? (x2): 1µ, symbol Device:C_Small
- added C? (x2): 10µ, symbol Device:C_Small
- added D? (x2): GREEN, symbol Device:LED
- added Q? (x2): BC850, Package_TO_SOT_SMD:SOT-23, symbol Transistor_BJT:BC850
- added R? (x2): 10k, symbol Device:R_Small
- added R? (x2): 1k, symbol Device:R_Small
- added U? (x2): TLV75712PDR, symbol eco_power:TLV75712PDR
Connections:
- net labels added: +1V2A, +1V2T
- wire segments 413 -> 465
Other:
- note added: "1.2V/1A\nSERDES analog"
- note added: "1.2V/1A\nSERDES termination"

Commit message: ecp5_mainboard/power: Add startup/sequencing control
Signed-off-by: David Shah <davey1576@gmail.com>
Parts:
- removed D?: GREEN, symbol Device:LED
- removed R?: 1.5k, symbol Device:R_Small
- added D?: RED, symbol Device:LED
- added D?: GREEN, symbol Device:LED
- added Q?: BSH111BKR, Package_TO_SOT_SMD:SOT-23, symbol Transistor_FET:2N7002
- added R? (x2): 1.5k, symbol Device:R_Small
- added RN?: 10k, symbol Device:R_Pack04
- added U?: LM3880, Package_TO_SOT_SMD:SOT-23-6, symbol Power_Supervisor:LM3880
- added U?: MAX811MEUS-T, Package_TO_SOT_SMD:SOT-143, symbol Power_Supervisor:MAX811MEUS-T
Connections:
- net labels added: PWR_EN
- wire segments 465 -> 498
- no-connect marks 3 -> 6
