File: hardware/ecp5_mainboard/power.sch (KiCad schematic (older format))
At the start: 103 parts, among them J201 12V_EXT, Q201 BSH111BKR, Q203 BC850, Q204 BSH111BKR, Q205 BC850, Q206 BSH111BKR, Q207 BSH111BKR, Q208 BSH111BKR, Q209 BSH111BKR, U201 MAX811MEUS-T, U202 LM3880, U204 TLV75712PDR, U205 LM21212-2, U206 TPS565208, U207 TLV75712PDR, U208 TPS62823, U209 TPS62823, U210 TPS62823, U211 TPS62823

Commit message: hardware/mainboard: Re-annotate and fix ERC
Signed-off-by: David Shah <dave@ds0.me>
Parts:
- renumbered C203 to C1, C212 to C10, C213 to C11, C214 to C12, C215 to C13, C216 to C14, C217 to C15, C218 to C16, C219 to C17, C220 to C18, C221 to C19, C204 to C2, C222 to C20, C223 to C21, C224 to C22, C225 to C23, C226 to C24, C227 to C25, C228 to C26, C229 to C27, C230 to C28, C231 to C29, C205 to C3, C232 to C30, C206 to C4, C207 to C5, C209 to C6, C208 to C7, C210 to C8, C211 to C9, D201 to D1, D211 to D10, D212 to D11, D202 to D2, D203 to D3, D204 to D4, D206 to D5, D207 to D6, D208 to D7, D209 to D8, D210 to D9, F201 to F1, F202 to F2, FL201 to FL1, J201 to J1, L201 to L1, L202 to L2, L203 to L3, L204 to L4, L205 to L5, L206 to L6, Q201 to Q1, Q203 to Q2, Q204 to Q3, Q205 to Q4, Q206 to Q5, Q207 to Q6, Q208 to Q7, Q209 to Q8, R203 to R1, R220 to R10, R221 to R11, R223 to R12, R224 to R13, R222 to R14, R225 to R15, R226 to R16, R227 to R17, R228 to R18, R229 to R19, R205 to R2, R230 to R20, R231 to R21, R232 to R22, R233 to R23, R234 to R24, R235 to R25, R236 to R26, R237 to R27, R238 to R28, R239 to R29, R212 to R3, R240 to R30, R241 to R31, R242 to R32, R243 to R33, R213 to R4, R214 to R5, R216 to R6, R217 to R7, R218 to R8, R219 to R9, RN201 to RN1, U201 to U1, U211 to U10, U202 to U2, U204 to U3, U206 to U4, U205 to U5, U207 to U6, U208 to U7, U209 to U8, U210 to U9

Commit message: hardware/mainboard: Assign some footprints
Signed-off-by: David Shah <dave@ds0.me>
Parts:
- C1, C10: footprint (none) -> Capacitor_SMD:C_0603_1608Metric
- C11, C12, C19, C20, C21, C22, C7, C9: footprint (none) -> Capacitor_SMD:C_0402_1005Metric
- C13: footprint (none) -> Capacitor_SMD:C_1210_3225Metric
- C14, C15, C16, C17, C18, C23, C24, C25, C26, C27, C28, C29, C3, C30, C4, C5, C8: footprint (none) -> Capacitor_SMD:C_0805_2012Metric
- C6: footprint 22u/25V -> Capacitor_SMD:C_1206_3216Metric
- D1, D10, D11, D2, D4, D5, D6, D7, D8, D9: footprint (none) -> LED_SMD:LED_0805_2012Metric
- R1, R10, R11, R12, R13, R14, R15, R16, R17, R18, R19, R2, R20, R21, R22, R23, R24, R25, R26, R27, R28, R29, R3, R30, R31, R32, R33, R4, R5, R6, R7, R8, R9: footprint (none) -> Resistor_SMD:R_0402_1005Metric
- RN1: footprint (none) -> Resistor_SMD:R_Array_Convex_4x0402
- U4: footprint (none) -> Package_TO_SOT_SMD:SOT-23-6
- U5: footprint (none) -> Package_SO:HTSSOP-20-1EP_4.4x6.5mm_P0.65mm_EP3.4x6.5mm

Commit message: hardware/mainboard: Assign more footprints
Signed-off-by: David Shah <dave@ds0.me>
Parts:
- C2: footprint (none) -> Capacitor_SMD:CP_Elec_6.3x5.8
- J1: footprint (none) -> Connector_BarrelJack:BarrelJack_Horizontal
- L1: footprint (none) -> Inductor_SMD:L_Coilcraft_XAL5030
- L3, L4, L5, L6: footprint (none) -> Inductor_SMD:L_Vishay_IHLP-1212
Changed lines of the file:
@@
 F 0 "J1" H 1478 2975 50  0000 C CNN
 F 1 "12V_EXT" H 1478 2884 50  0000 C CNN
-F 2 "" H 1450 2610 50  0001 C CNN
+F 2 "Connector_BarrelJack:BarrelJack_Horizontal" H 1450 2610 50  0001 C CNN
 F 3 "~" H 1450 2610 50  0001 C CNN
 	1    1400 2650
@@
 F 0 "C2" H 3968 2746 50  0000 L CNN
 F 1 "100µF/25V" H 3968 2655 50  0000 L CNN
-F 2 "" H 3888 2550 50  0001 C CNN
+F 2 "Capacitor_SMD:CP_Elec_6.3x5.8" H 3888 2550 50  0001 C CNN
 F 3 "~" H 3850 2700 50  0001 C CNN
 	1    3850 2700
@@
 F 0 "L4" V 12340 1750 50  0000 C CNN
 F 1 "470n/IHLP1212" V 12249 1750 50  0000 C CNN
-F 2 "" H 12150 1750 50  0001 C CNN
+F 2 "Inductor_SMD:L_Vishay_IHLP-1212" H 12150 1750 50  0001 C CNN
 F 3 "~" H 12150 1750 50  0001 C CNN
 	1    12150 1750
@@
 F 0 "L5" V 12340 3250 50  0000 C CNN
 F 1 "470n/IHLP1212" V 12249 3250 50  0000 C CNN
-F 2 "" H 12150 3250 50  0001 C CNN
+F 2 "Inductor_SMD:L_Vishay_IHLP-1212" H 12150 3250 50  0001 C CNN
 F 3 "~" H 12150 3250 50  0001 C CNN
 	1    12150 3250
@@
 F 0 "L6" V 12340 4800 50  0000 C CNN
 F 1 "470n/IHLP1212" V 12249 4800 50  0000 C CNN
-F 2 "" H 12150 4800 50  0001 C CNN
+F 2 "Inductor_SMD:L_Vishay_IHLP-1212" H 12150 4800 50  0001 C CNN
 F 3 "~" H 12150 4800 50  0001 C CNN
 	1    12150 4800
@@
 F 0 "L3" V 12290 6250 50  0000 C CNN
 F 1 "470n/IHLP1212" V 12199 6250 50  0000 C CNN
-F 2 "" H 12100 6250 50  0001 C CNN
+F 2 "Inductor_SMD:L_Vishay_IHLP-1212" H 12100 6250 50  0001 C CNN
 F 3 "~" H 12100 6250 50  0001 C CNN
 	1    12100 6250
@@
 F 0 "L1" V 7590 6200 50  0000 C CNN
 F 1 "800nH/XAL5030" V 7499 6200 50  0000 C CNN
-F 2 "" H 7400 6200 50  0001 C CNN
+F 2 "Inductor_SMD:L_Coilcraft_XAL5030" H 7400 6200 50  0001 C CNN
 F 3 "~" H 7400 6200 50  0001 C CNN
 	1    7400 6200

Commit message: hardware: Creating and assigning some misc footprints
Signed-off-by: David Shah <dave@ds0.me>
Parts:
- F1, F2: footprint (none) -> Custom Parts:FuseHolder_SMD_Shurter_0031.7701.11
- L2: footprint (none) -> Custom Parts:L_CoilCraft_XAL60xx
- U3, U6: footprint (none) -> Custom Parts:TI_WSON8_2x2mm_p0.65mm
Changed lines of the file:
@@
 F 0 "F2" V 1953 2550 50  0000 C CNN
 F 1 "3A" V 2044 2550 50  0000 C CNN
-F 2 "" V 2080 2550 50  0001 C CNN
+F 2 "Custom Parts:FuseHolder_SMD_Shurter_0031.7701.11" V 2080 2550 50  0001 C CNN
 F 3 "~" H 2150 2550 50  0001 C CNN
 	1    2150 2550
@@
 F 0 "F1" V 1853 3600 50  0000 C CNN
 F 1 "3A/DNF" V 1944 3600 50  0000 C CNN
-F 2 "" V 1980 3600 50  0001 C CNN
+F 2 "Custom Parts:FuseHolder_SMD_Shurter_0031.7701.11" V 1980 3600 50  0001 C CNN
 F 3 "~" H 2050 3600 50  0001 C CNN
 	1    2050 3600
@@
 F 0 "L2" V 7690 2200 50  0000 C CNN
 F 1 "3.3µH/XAL6030-332" V 7599 2200 50  0000 C CNN
-F 2 "" H 7500 2200 50  0001 C CNN
+F 2 "Custom Parts:L_CoilCraft_XAL60xx" H 7500 2200 50  0001 C CNN
 F 3 "~" H 7500 2200 50  0001 C CNN
 	1    7500 2200
@@
 F 0 "U3" H 4100 10315 50  0000 C CNN
 F 1 "TLV75712PDR" H 4100 10224 50  0000 C CNN
-F 2 "" H 4100 9850 50  0001 C CNN
+F 2 "Custom Parts:TI_WSON8_2x2mm_p0.65mm" H 4100 9850 50  0001 C CNN
 F 3 "" H 4100 9850 50  0001 C CNN
 	1    4100 9850
@@
 F 0 "U6" H 8850 10365 50  0000 C CNN
 F 1 "TLV75712PDR" H 8850 10274 50  0000 C CNN
-F 2 "" H 8850 9900 50  0001 C CNN
+F 2 "Custom Parts:TI_WSON8_2x2mm_p0.65mm" H 8850 9900 50  0001 C CNN
 F 3 "" H 8850 9900 50  0001 C CNN
 	1    8850 9900

Commit message: hardware/mainboard: More footprint assignment, other small tweaks
Signed-off-by: David Shah <dave@ds0.me>
Parts:
- removed FL1: EMI_Filter_CommonMode, symbol Device:EMI_Filter_CommonMode
- D3: value PPS1040 -> MBR15U60
- U10, U7, U8, U9: footprint (none) -> Custom Parts:TI_VSON-HR_1.5x2mm_p0.5mm
Connections:
- net +12V: now also F2.1
- net GND: now also J1.2, J1.3
Other:
- moved on the sheet: F2, J1
Changed lines of the file:
@@
 L ecp5_mainboard-rescue:Barrel_Jack-Connector J1
 U 1 1 5B5D9C9C
-P 1400 2650
-F 0 "J1" H 1478 2975 50  0000 C CNN
-F 1 "12V_EXT" H 1478 2884 50  0000 C CNN
-F 2 "Connector_BarrelJack:BarrelJack_Horizontal" H 1450 2610 50  0001 C CNN
-F 3 "~" H 1450 2610 50  0001 C CNN
-	1    1400 2650
+P 1950 2650
+F 0 "J1" H 2028 2975 50  0000 C CNN
+F 1 "12V_EXT" H 2028 2884 50  0000 C CNN
+F 2 "Connector_BarrelJack:BarrelJack_Horizontal" H 2000 2610 50  0001 C CNN
+F 3 "~" H 2000 2610 50  0001 C CNN
+	1    1950 2650
 	1    0    0    -1
 $EndComp
@@
 L Device:Fuse F2
 U 1 1 5B5DA0F9
-P 2150 2550
-F 0 "F2" V 1953 2550 50  0000 C CNN
-F 1 "3A" V 2044 2550 50  0000 C CNN
-F 2 "Custom Parts:FuseHolder_SMD_Shurter_0031.7701.11" V 2080 2550 50  0001 C CNN
-F 3 "~" H 2150 2550 50  0001 C CNN
-	1    2150 2550
+P 2700 2550
+F 0 "F2" V 2503 2550 50  0000 C CNN
+F 1 "3A" V 2594 2550 50  0000 C CNN
+F 2 "Custom Parts:FuseHolder_SMD_Shurter_0031.7701.11" V 2630 2550 50  0001 C CNN
+F 3 "~" H 2700 2550 50  0001 C CNN
+	1    2700 2550
 	0    1    1    0
 $EndComp
 Wire Wire Line
-	1700 2550 2000 2550
-Wire Wire Line
-	1700 2750 1800 2750
-Wire Wire Line
-	1900 2750 1900 2850
-$Comp
-L Device:EMI_Filter_CommonMode FL1
-U 1 1 5B5DA3C4
-P 2750 2700
-F 0 "FL1" H 2750 2978 50  0000 C CNN
-F 1 "EMI_Filter_CommonMode" H 2750 2887 50  0000 C CNN
-F 2 "" V 2750 2740 50  0001 C CNN
-F 3 "~" V 2750 2740 50  0000 C CNN
-	1    2750 2700
-	1    0    0    -1
-$EndComp
-Wire Wire Line
-	2300 2550 2450 2550
-Wire Wire Line
-	2450 2550 2450 2600
-Wire Wire Line
-	2450 2600 2550 2600
-Wire Wire Line
-	2550 2800 2450 2800
-Wire Wire Line
-	2450 2800 2450 2850
-Wire Wire Line
-	1900 2850 2450 2850
-Wire Wire Line
-	2950 2800 3050 2800
-Wire Wire Line
-	3050 2800 3050 3350
+	2250 2550 2550 2550
+Wire Wire Line
+	2250 2750 2350 2750
 Wire Wire Line
 	3050 3350 3200 3350
-Wire Wire Line
-	2950 2600 3050 2600
-Wire Wire Line
-	3050 2600 3050 2400
 Wire Wire Line
 	3050 2400 3200 2400
@@
 P 3200 2700
 F 0 "D3" V 3154 2768 50  0000 L CNN
-F 1 "PPS1040" V 3245 2768 50  0000 L CNN
+F 1 "MBR15U60" V 3245 2768 50  0000 L CNN
 F 2 "" V 3200 2700 50  0001 C CNN
 F 3 "~" V 3200 2700 50  0001 C CNN
@@
 	3200 2800 3200 3350
 Wire Wire Line
-	1700 2650 1800 2650
-Wire Wire Line
-	1800 2650 1800 2750
-Connection ~ 1800 2750
-Wire Wire Line
-	1800 2750 1900 2750
+	2250 2650 2350 2650
+Wire Wire Line
+	2350 2650 2350 2750
+Connection ~ 2350 2750
 Connection ~ 3200 3350
 $Comp
@@
 Wire Wire Line
 	2200 3600 2600 3600
-Text Notes 1950 2700 0    50   ~ 0
+Text Notes 2550 2650 0    50   ~ 0
 in socket
 Text Notes 1800 3900 0    50   ~ 0
@@
 Wire Wire Line
 	8050 2150 8050 2200
-Text Notes 1250 2950 0    50   ~ 0
+Text Notes 1800 2950 0    50   ~ 0
 12V/2.5A\ninput
 $Comp
@@
 F 0 "U8" H 11150 2615 50  0000 C CNN
 F 1 "TPS62823" H 11150 2524 50  0000 C CNN
-F 2 "" H 11150 2050 50  0001 C CNN
+F 2 "Custom Parts:TI_VSON-HR_1.5x2mm_p0.5mm" H 11150 2050 50  0001 C CNN
 F 3 "http://www.ti.com/lit/ds/symlink/tps62823.pdf" H 11150 2050 50  0001 C CNN
 	1    11150 2050
@@
 F 0 "U9" H 11150 4115 50  0000 C CNN
 F 1 "TPS62823" H 11150 4024 50  0000 C CNN
-F 2 "" H 11150 3550 50  0001 C CNN
+F 2 "Custom Parts:TI_VSON-HR_1.5x2mm_p0.5mm" H 11150 3550 50  0001 C CNN
 F 3 "http://www.ti.com/lit/ds/symlink/tps62823.pdf" H 11150 3550 50  0001 C CNN
 	1    11150 3550
@@
 F 0 "U10" H 11150 5665 50  0000 C CNN
 F 1 "TPS62823" H 11150 5574 50  0000 C CNN
-F 2 "" H 11150 5100 50  0001 C CNN
+F 2 "Custom Parts:TI_VSON-HR_1.5x2mm_p0.5mm" H 11150 5100 50  0001 C CNN
 F 3 "http://www.ti.com/lit/ds/symlink/tps62823.pdf" H 11150 5100 50  0001 C CNN
 	1    11150 5100
@@
 F 0 "U7" H 11100 7115 50  0000 C CNN
 F 1 "TPS62823" H 11100 7024 50  0000 C CNN
-F 2 "" H 11100 6550 50  0001 C CNN
+F 2 "Custom Parts:TI_VSON-HR_1.5x2mm_p0.5mm" H 11100 6550 50  0001 C CNN
 F 3 "http://www.ti.com/lit/ds/symlink/tps62823.pdf" H 11100 6550 50  0001 C CNN
 	1    11100 6550
@@
 	8500 2150 8500 2200
 Connection ~ 8500 2200
+Wire Wire Line
+	3050 2750 3050 3350
+Wire Wire Line
+	2350 2750 3050 2750
+Wire Wire Line
+	3050 2550 3050 2400
+Wire Wire Line
+	2850 2550 3050 2550
 $EndSCHEMATC

Commit message: hardware/mainboard: All footprints assigned
Signed-off-by: David Shah <dave@ds0.me>
Parts:
- removed D3: MBR15U60, symbol Device:D_Small
- added D3: MBR15U60, Package_TO_SOT_SMD:TO-277B, symbol Device:D_Schottky_AAK
Connections:
- net +12V: now also D3.3 (K)
- net GND: now also D3.1 (A), D3.2 (A)
Changed lines of the file:
@@
 Wire Wire Line
 	3050 2400 3200 2400
-$Comp
-L Device:D_Small D3
-U 1 1 5B5DA9BE
-P 3200 2700
-F 0 "D3" V 3154 2768 50  0000 L CNN
-F 1 "MBR15U60" V 3245 2768 50  0000 L CNN
-F 2 "" V 3200 2700 50  0001 C CNN
-F 3 "~" V 3200 2700 50  0001 C CNN
-	1    3200 2700
-	0    1    1    0
-$EndComp
 Wire Wire Line
 	3200 2600 3200 2400
-Wire Wire Line
-	3200 2800 3200 3350
 Wire Wire Line
 	2250 2650 2350 2650
@@
 	3850 2400 4550 2400
 Wire Wire Line
-	3200 3350 3850 3350
+	3200 3350 3300 3350
 $Comp
 L power:PWR_FLAG #FLG0101
@@
 Wire Wire Line
 	2850 2550 3050 2550
+$Comp
+L Device:D_Schottky_AAK D3
+U 1 1 5C219D75
+P 3200 2750
+F 0 "D3" V 3179 2890 50  0000 L CNN
+F 1 "MBR15U60" V 3270 2890 50  0000 L CNN
+F 2 "Package_TO_SOT_SMD:TO-277B" H 3200 2750 50  0001 C CNN
+F 3 "~" H 3200 2750 50  0001 C CNN
+	1    3200 2750
+	0    1    1    0
+$EndComp
+Wire Wire Line
+	3200 2950 3200 3350
+Wire Wire Line
+	3300 2950 3300 3350
+Connection ~ 3300 3350
+Wire Wire Line
+	3300 3350 3850 3350
 $EndSCHEMATC

Commit message: hardware/mainboard: Power related placement
Signed-off-by: David Shah <dave@ds0.me>
Parts:
- added C256: 47µ, Capacitor_SMD:C_1210_3225Metric, symbol Device:C_Small
Connections:
- net +1V2: now also C256.1
- net GND: now also C256.2
Changed lines of the file:
@@
 U 1 1 5B7059F5
 P 11150 2050
+AR Path="/5B7059F5" Ref="U8"  Part="1"
+AR Path="/5B5D9B41/5B7059F5" Ref="U8"  Part="1"
 F 0 "U8" H 11150 2615 50  0000 C CNN
 F 1 "TPS62823" H 11150 2524 50  0000 C CNN
@@
 U 1 1 5B7A0A18
 P 11150 3550
+AR Path="/5B7A0A18" Ref="U9"  Part="1"
+AR Path="/5B5D9B41/5B7A0A18" Ref="U9"  Part="1"
 F 0 "U9" H 11150 4115 50  0000 C CNN
 F 1 "TPS62823" H 11150 4024 50  0000 C CNN
@@
 U 1 1 5B7AA29B
 P 11150 5100
+AR Path="/5B7AA29B" Ref="U10"  Part="1"
+AR Path="/5B5D9B41/5B7AA29B" Ref="U10"  Part="1"
 F 0 "U10" H 11150 5665 50  0000 C CNN
 F 1 "TPS62823" H 11150 5574 50  0000 C CNN
@@
 U 1 1 5B989F17
 P 11100 6550
+AR Path="/5B989F17" Ref="U7"  Part="1"
+AR Path="/5B5D9B41/5B989F17" Ref="U7"  Part="1"
 F 0 "U7" H 11100 7115 50  0000 C CNN
 F 1 "TPS62823" H 11100 7024 50  0000 C CNN
@@
 Wire Wire Line
 	3300 3350 3850 3350
+$Comp
+L Device:C_Small C256
+U 1 1 5BF9B9FF
+P 8650 6650
+F 0 "C256" H 8742 6696 50  0000 L CNN
+F 1 "47µ" H 8742 6605 50  0000 L CNN
+F 2 "Capacitor_SMD:C_1210_3225Metric" H 8650 6650 50  0001 C CNN
+F 3 "~" H 8650 6650 50  0001 C CNN
+	1    8650 6650
+	1    0    0    -1
+$EndComp
+Wire Wire Line
+	8350 6200 8650 6200
+Wire Wire Line
+	8650 6200 8650 6550
+Connection ~ 8350 6200
+Wire Wire Line
+	8650 6750 8650 6900
+$Comp
+L power:GND #PWR0253
+U 1 1 5C00AE24
+P 8650 6900
+F 0 "#PWR0253" H 8650 6650 50  0001 C CNN
+F 1 "GND" H 8655 6727 50  0000 C CNN
+F 2 "" H 8650 6900 50  0001 C CNN
+F 3 "" H 8650 6900 50  0001 C CNN
+	1    8650 6900
+	1    0    0    -1
+$EndComp
 $EndSCHEMATC
