File: hardware/ecp5_mainboard/power.sch (KiCad schematic (older format))
At the start: 103 parts, among them J1 12V_EXT, Q1 BSH111BKR, Q2 BC850, Q3 BSH111BKR, Q4 BC850, Q5 BSH111BKR, Q6 BSH111BKR, Q7 BSH111BKR, Q8 BSH111BKR, U1 MAX811MEUS-T, U10 TPS62823, U2 LM3880, U3 TLV75712PDR, U4 TPS565208, U5 LM21212-2, U6 TLV75712PDR, U7 TPS62823, U8 TPS62823, U9 TPS62823

Commit message: hardware/mainboard: Power circuitry placed
Signed-off-by: David Shah <dave@ds0.me>
Parts:
- removed D1: RED, LED_SMD:LED_0805_2012Metric, symbol Device:LED
- removed R1: 1.5k, Resistor_SMD:R_0402_1005Metric, symbol Device:R_Small
Changed lines of the file:
@@
 	1350 6400 1700 6400
-$Comp
-L Device:R_Small R1
-U 1 1 5C967669
-P 1700 5850
-F 0 "R1" H 1759 5896 50  0000 L CNN
-F 1 "1.5k" H 1759 5805 50  0000 L CNN
-F 2 "Resistor_SMD:R_0402_1005Metric" H 1700 5850 50  0001 C CNN
-F 3 "~" H 1700 5850 50  0001 C CNN
-	1    1700 5850
-	1    0    0    -1
-$EndComp
 $Comp
 L power:+5V #PWR03
 U 1 1 5C9678E4
-P 1700 5650
-F 0 "#PWR03" H 1700 5500 50  0001 C CNN
-F 1 "+5V" H 1715 5823 50  0000 C CNN
-F 2 "" H 1700 5650 50  0001 C CNN
-F 3 "" H 1700 5650 50  0001 C CNN
-	1    1700 5650
-	1    0    0    -1
-$EndComp
-Wire Wire Line
-	1700 5650 1700 5700
-$Comp
-L Device:LED D1
-U 1 1 5C9A070B
-P 1700 6200
-F 0 "D1" V 1738 6082 50  0000 R CNN
-F 1 "RED" V 1647 6082 50  0000 R CNN
-F 2 "LED_SMD:LED_0805_2012Metric" H 1700 6200 50  0001 C CNN
-F 3 "~" H 1700 6200 50  0001 C CNN
-	1    1700 6200
-	0    -1   -1   0
-$EndComp
-Wire Wire Line
-	1700 6050 1700 5950
-Wire Wire Line
-	1700 6350 1700 6400
+P 2100 5650
+F 0 "#PWR03" H 2100 5500 50  0001 C CNN
+F 1 "+5V" H 2115 5823 50  0000 C CNN
+F 2 "" H 2100 5650 50  0001 C CNN
+F 3 "" H 2100 5650 50  0001 C CNN
+	1    2100 5650
+	1    0    0    -1
+$EndComp
 Connection ~ 1700 6400
 Wire Wire Line
@@
 Wire Wire Line
 	1700 7250 1800 7250
-Wire Wire Line
-	2100 5700 1700 5700
-Connection ~ 1700 5700
-Wire Wire Line
-	1700 5700 1700 5750
 $Comp
 L Device:R_Small R2
@@
 	1    0    0    -1
 $EndComp
-Wire Wire Line
-	2100 5750 2100 5700
 Wire Wire Line
 	2100 5950 2100 6650
@@
 	1    0    0    -1
 $EndComp
+Wire Wire Line
+	2100 5650 2100 5750
 $EndSCHEMATC

Commit message: hardware/mainboard: Small design tweaks
Signed-off-by: David Shah <dave@ds0.me>
Parts:
- added TP10: 2.5V, TestPoint:TestPoint_THTPad_1.5x1.5mm_Drill0.7mm, symbol Connector:TestPoint
- added TP11: 1.35V, TestPoint:TestPoint_THTPad_1.5x1.5mm_Drill0.7mm, symbol Connector:TestPoint
- added TP12: 1.8V, TestPoint:TestPoint_THTPad_1.5x1.5mm_Drill0.7mm, symbol Connector:TestPoint
- added TP3: 1.2VA, TestPoint:TestPoint_THTPad_1.5x1.5mm_Drill0.7mm, symbol Connector:TestPoint
- added TP4: 1.2V, TestPoint:TestPoint_THTPad_1.5x1.5mm_Drill0.7mm, symbol Connector:TestPoint
- added TP5: 5V, TestPoint:TestPoint_THTPad_1.5x1.5mm_Drill0.7mm, symbol Connector:TestPoint
- added TP6, TP7: GND, TestPoint:TestPoint_THTPad_1.5x1.5mm_Drill0.7mm, symbol Connector:TestPoint
- added TP8: 1.2VT, TestPoint:TestPoint_THTPad_1.5x1.5mm_Drill0.7mm, symbol Connector:TestPoint
- added TP9: 3.3V, TestPoint:TestPoint_THTPad_1.5x1.5mm_Drill0.7mm, symbol Connector:TestPoint
Connections:
- net +1V2: now also TP4.1
- net +1V2A: now also TP3.1
- net +1V2T: now also TP8.1
- net +1V35: now also TP11.1
- net +1V8: now also TP12.1
- net +2V5: now also TP10.1
- net +3V3: now also TP9.1
- net +5V: now also TP5.1
- net GND: now also TP6.1, TP7.1
Changed lines of the file:
@@
 Connection ~ 8050 2200
 Wire Wire Line
-	8500 3050 8500 3350
+	8500 3050 8500 3200
 Wire Wire Line
 	8500 3350 8050 3350
@@
 Wire Wire Line
 	2100 5650 2100 5750
+$Comp
+L Connector:TestPoint TP9
+U 1 1 5C127F56
+P 13900 1650
+F 0 "TP9" H 13958 1770 50  0000 L CNN
+F 1 "3.3V" H 13958 1679 50  0000 L CNN
+F 2 "TestPoint:TestPoint_THTPad_1.5x1.5mm_Drill0.7mm" H 14100 1650 50  0001 C CNN
+F 3 "~" H 14100 1650 50  0001 C CNN
+	1    13900 1650
+	1    0    0    -1
+$EndComp
+Wire Wire Line
+	13900 1650 13900 1750
+Connection ~ 13900 1750
+$Comp
+L Connector:TestPoint TP10
+U 1 1 5C15E0E3
+P 13900 3100
+F 0 "TP10" H 13958 3220 50  0000 L CNN
+F 1 "2.5V" H 13958 3129 50  0000 L CNN
+F 2 "TestPoint:TestPoint_THTPad_1.5x1.5mm_Drill0.7mm" H 14100 3100 50  0001 C CNN
+F 3 "~" H 14100 3100 50  0001 C CNN
+	1    13900 3100
+	1    0    0    -1
+$EndComp
+Wire Wire Line
+	13900 3100 13900 3250
+Connection ~ 13900 3250
+$Comp
+L Connector:TestPoint TP12
+U 1 1 5C1949EC
+P 13950 4650
+F 0 "TP12" H 14008 4770 50  0000 L CNN
+F 1 "1.8V" H 14008 4679 50  0000 L CNN
+F 2 "TestPoint:TestPoint_THTPad_1.5x1.5mm_Drill0.7mm" H 14150 4650 50  0001 C CNN
+F 3 "~" H 14150 4650 50  0001 C CNN
+	1    13950 4650
+	1    0    0    -1
+$EndComp
+Wire Wire Line
+	13950 4650 13950 4800
+Connection ~ 13950 4800
+$Comp
+L Connector:TestPoint TP11
+U 1 1 5C1CB463
+P 13900 6100
+F 0 "TP11" H 13958 6220 50  0000 L CNN
+F 1 "1.35V" H 13958 6129 50  0000 L CNN
+F 2 "TestPoint:TestPoint_THTPad_1.5x1.5mm_Drill0.7mm" H 14100 6100 50  0001 C CNN
+F 3 "~" H 14100 6100 50  0001 C CNN
+	1    13900 6100
+	1    0    0    -1
+$EndComp
+Wire Wire Line
+	13900 6100 13900 6250
+Connection ~ 13900 6250
+$Comp
+L Connector:TestPoint TP3
+U 1 1 5C2061D6
+P 5550 9450
+F 0 "TP3" H 5608 9570 50  0000 L CNN
+F 1 "1.2VA" H 5608 9479 50  0000 L CNN
+F 2 "TestPoint:TestPoint_THTPad_1.5x1.5mm_Drill0.7mm" H 5750 9450 50  0001 C CNN
+F 3 "~" H 5750 9450 50  0001 C CNN
+	1    5550 9450
+	1    0    0    -1
+$EndComp
+Wire Wire Line
+	5550 9450 5550 9650
+Connection ~ 5550 9650
+$Comp
+L Connector:TestPoint TP8
+U 1 1 5C23D719
+P 10300 9500
+F 0 "TP8" H 10358 9620 50  0000 L CNN
+F 1 "1.2VT" H 10358 9529 50  0000 L CNN
+F 2 "TestPoint:TestPoint_THTPad_1.5x1.5mm_Drill0.7mm" H 10500 9500 50  0001 C CNN
+F 3 "~" H 10500 9500 50  0001 C CNN
+	1    10300 9500
+	1    0    0    -1
+$EndComp
+Wire Wire Line
+	10300 9500 10300 9700
+Connection ~ 10300 9700
+$Comp
+L Connector:TestPoint TP4
+U 1 1 5C274F6C
+P 8650 6050
+F 0 "TP4" H 8708 6170 50  0000 L CNN
+F 1 "1.2V" H 8708 6079 50  0000 L CNN
+F 2 "TestPoint:TestPoint_THTPad_1.5x1.5mm_Drill0.7mm" H 8850 6050 50  0001 C CNN
+F 3 "~" H 8850 6050 50  0001 C CNN
+	1    8650 6050
+	1    0    0    -1
+$EndComp
+Wire Wire Line
+	8650 6050 8650 6200
+Connection ~ 8650 6200
+$Comp
+L Connector:TestPoint TP5
+U 1 1 5C2ACBFC
+P 8800 2200
+F 0 "TP5" V 8754 2388 50  0000 L CNN
+F 1 "5V" V 8845 2388 50  0000 L CNN
+F 2 "TestPoint:TestPoint_THTPad_1.5x1.5mm_Drill0.7mm" H 9000 2200 50  0001 C CNN
+F 3 "~" H 9000 2200 50  0001 C CNN
+	1    8800 2200
+	0    1    1    0
+$EndComp
+Wire Wire Line
+	8800 2200 8500 2200
+$Comp
+L Connector:TestPoint TP6
+U 1 1 5C2E8C62
+P 8850 3200
+F 0 "TP6" V 8804 3387 50  0000 L CNN
+F 1 "GND" V 8895 3387 50  0000 L CNN
+F 2 "TestPoint:TestPoint_THTPad_1.5x1.5mm_Drill0.7mm" H 9050 3200 50  0001 C CNN
+F 3 "~" H 9050 3200 50  0001 C CNN
+	1    8850 3200
+	0    1    1    0
+$EndComp
+$Comp
+L Connector:TestPoint TP7
+U 1 1 5C2E908C
+P 8850 3350
+F 0 "TP7" V 8804 3537 50  0000 L CNN
+F 1 "GND" V 8895 3537 50  0000 L CNN
+F 2 "TestPoint:TestPoint_THTPad_1.5x1.5mm_Drill0.7mm" H 9050 3350 50  0001 C CNN
+F 3 "~" H 9050 3350 50  0001 C CNN
+	1    8850 3350
+	0    1    1    0
+$EndComp
+Wire Wire Line
+	8500 3350 8850 3350
+Connection ~ 8500 3350
+Wire Wire Line
+	8850 3200 8500 3200
+Connection ~ 8500 3200
+Wire Wire Line
+	8500 3200 8500 3350
 $EndSCHEMATC

Commit message: hardware/mainboard: DRC fixes
Signed-off-by: David Shah <dave@ds0.me>
Parts:
- TP4, TP6: footprint TestPoint:TestPoint_THTPad_1.5x1.5mm_Drill0.7mm -> TestPoint:TestPoint_Pad_1.5x1.5mm
Changed lines of the file:
@@
 F 0 "TP4" H 8708 6170 50  0000 L CNN
 F 1 "1.2V" H 8708 6079 50  0000 L CNN
-F 2 "TestPoint:TestPoint_THTPad_1.5x1.5mm_Drill0.7mm" H 8850 6050 50  0001 C CNN
+F 2 "TestPoint:TestPoint_Pad_1.5x1.5mm" H 8850 6050 50  0001 C CNN
 F 3 "~" H 8850 6050 50  0001 C CNN
 	1    8650 6050
@@
 F 0 "TP6" V 8804 3387 50  0000 L CNN
 F 1 "GND" V 8895 3387 50  0000 L CNN
-F 2 "TestPoint:TestPoint_THTPad_1.5x1.5mm_Drill0.7mm" H 9050 3200 50  0001 C CNN
+F 2 "TestPoint:TestPoint_Pad_1.5x1.5mm" H 9050 3200 50  0001 C CNN
 F 3 "~" H 9050 3200 50  0001 C CNN
 	1    8850 3200

Commit message: hardware/mainboard: BoM fixes, add USB power option
Signed-off-by: David Shah <dave@ds0.me>
Parts:
- added J?: PWR, Connector_PinHeader_2.54mm:PinHeader_1x03_P2.54mm_Vertical, symbol Connector_Generic:Conn_01x03
Connections:
- net +5V: now also J?.2 (Pin_2); no longer C13.1, L2.2, R12.1
- new net: C13.1, J?.1 (Pin_1), L2.2, R12.1
- new net USB_5V: J?.3 (Pin_3)
Other:
- moved on the sheet: C13, R12, R13, TP5, TP6, TP7
Changed lines of the file:
@@
 EESchema Schematic File Version 4
 LIBS:ecp5_mainboard-cache
-EELAYER 26 0
+EELAYER 29 0
 EELAYER END
 $Descr A3 16535 11693
@@
 Wire Wire Line
 	5050 3350 4550 3350
-$Comp
-L Device:L L2
-U 1 1 5B5E85F4
-P 7500 2200
-F 0 "L2" V 7690 2200 50  0000 C CNN
-F 1 "3.3µH/XAL6030-332" V 7599 2200 50  0000 C CNN
-F 2 "Custom Parts:L_CoilCraft_XAL60xx" H 7500 2200 50  0001 C CNN
-F 3 "~" H 7500 2200 50  0001 C CNN
-	1    7500 2200
-	0    -1   -1   0
-$EndComp
-Wire Wire Line
-	7350 2200 7150 2200
 Wire Wire Line
 	7150 2200 7150 2550
@@
 L Device:R_Small R12
 U 1 1 5B5EBCCF
-P 8050 2450
-F 0 "R12" H 8109 2496 50  0000 L CNN
-F 1 "54.9k" H 8109 2405 50  0000 L CNN
-F 2 "Resistor_SMD:R_0402_1005Metric" H 8050 2450 50  0001 C CNN
-F 3 "~" H 8050 2450 50  0001 C CNN
-	1    8050 2450
-	1    0    0    -1
-$EndComp
-Wire Wire Line
-	8050 2350 8050 2200
-Wire Wire Line
-	8050 2550 8050 2950
-Wire Wire Line
-	8050 2950 6850 2950
+P 8300 2450
+F 0 "R12" H 8359 2496 50  0000 L CNN
+F 1 "54.9k" H 8359 2405 50  0000 L CNN
+F 2 "Resistor_SMD:R_0402_1005Metric" H 8300 2450 50  0001 C CNN
+F 3 "~" H 8300 2450 50  0001 C CNN
+	1    8300 2450
+	1    0    0    -1
+$EndComp
+Wire Wire Line
+	8300 2350 8300 2200
+Wire Wire Line
+	8300 2550 8300 2950
+Wire Wire Line
+	8300 2950 6850 2950
 $Comp
 L Device:R_Small R13
 U 1 1 5B5ED622
-P 8050 3150
-F 0 "R13" H 8109 3196 50  0000 L CNN
-F 1 "10k" H 8109 3105 50  0000 L CNN
-F 2 "Resistor_SMD:R_0402_1005Metric" H 8050 3150 50  0001 C CNN
-F 3 "~" H 8050 3150 50  0001 C CNN
-	1    8050 3150
-	1    0    0    -1
-$EndComp
-Wire Wire Line
-	8050 3050 8050 2950
-Connection ~ 8050 2950
-Wire Wire Line
-	5350 3350 8050 3350
-Wire Wire Line
-	8050 3350 8050 3250
+P 8300 3150
+F 0 "R13" H 8359 3196 50  0000 L CNN
+F 1 "10k" H 8359 3105 50  0000 L CNN
+F 2 "Resistor_SMD:R_0402_1005Metric" H 8300 3150 50  0001 C CNN
+F 3 "~" H 8300 3150 50  0001 C CNN
+	1    8300 3150
+	1    0    0    -1
+$EndComp
+Wire Wire Line
+	8300 3050 8300 2950
+Connection ~ 8300 2950
+Wire Wire Line
+	5350 3350 8300 3350
+Wire Wire Line
+	8300 3350 8300 3250
 $Comp
 L Device:C_Small C13
 U 1 1 5B5F0113
-P 8500 2950
-F 0 "C13" H 8592 2996 50  0000 L CNN
-F 1 "47µ" H 8592 2905 50  0000 L CNN
-F 2 "Capacitor_SMD:C_1210_3225Metric" H 8500 2950 50  0001 C CNN
-F 3 "~" H 8500 2950 50  0001 C CNN
-	1    8500 2950
-	1    0    0    -1
-$EndComp
-Wire Wire Line
-	8500 2200 8050 2200
-Connection ~ 8050 2200
-Wire Wire Line
-	8500 3050 8500 3200
-Wire Wire Line
-	8500 3350 8050 3350
+P 8750 2950
+F 0 "C13" H 8842 2996 50  0000 L CNN
+F 1 "47µ" H 8842 2905 50  0000 L CNN
+F 2 "Capacitor_SMD:C_1210_3225Metric" H 8750 2950 50  0001 C CNN
+F 3 "~" H 8750 2950 50  0001 C CNN
+	1    8750 2950
+	1    0    0    -1
+$EndComp
+Wire Wire Line
+	8750 2200 8300 2200
+Connection ~ 8300 2200
+Wire Wire Line
+	8750 3050 8750 3200
+Wire Wire Line
+	8750 3350 8300 3350
 $Comp
 L power:+5V #PWR022
 U 1 1 5B5F2065
-P 8050 2150
-F 0 "#PWR022" H 8050 2000 50  0001 C CNN
-F 1 "+5V" H 8065 2323 50  0000 C CNN
-F 2 "" H 8050 2150 50  0001 C CNN
-F 3 "" H 8050 2150 50  0001 C CNN
-	1    8050 2150
-	1    0    0    -1
-$EndComp
-Wire Wire Line
-	8050 2150 8050 2200
+P 9450 2400
+F 0 "#PWR022" H 9450 2250 50  0001 C CNN
+F 1 "+5V" H 9465 2573 50  0000 C CNN
+F 2 "" H 9450 2400 50  0001 C CNN
+F 3 "" H 9450 2400 50  0001 C CNN
+	1    9450 2400
+	0    1    1    0
+$EndComp
 Text Notes 1800 2950 0    50   ~ 0
 12V/2.5A\ninput
@@
 Connection ~ 5050 2400
 Wire Wire Line
-	7650 2200 8050 2200
-Wire Wire Line
 	11850 1750 12000 1750
 $Comp
@@
 	1    0    0    -1
 $EndComp
-Connection ~ 8050 3350
+Connection ~ 8300 3350
 Connection ~ 5350 3350
 Text Label 2150 6400 0    50   ~ 0
@@
 	5400 6100 5300 6100
 Connection ~ 5300 6100
-Wire Wire Line
-	8500 2200 8500 2850
 $Comp
 L power:PWR_FLAG #FLG05
@@
 Wire Wire Line
 	3200 3350 3300 3350
-$Comp
-L power:PWR_FLAG #FLG0101
-U 1 1 61A6AF75
-P 8500 2150
-F 0 "#FLG0101" H 8500 2225 50  0001 C CNN
-F 1 "PWR_FLAG" H 8500 2324 50  0000 C CNN
-F 2 "" H 8500 2150 50  0001 C CNN
-F 3 "~" H 8500 2150 50  0001 C CNN
-	1    8500 2150
-	1    0    0    -1
-$EndComp
-Wire Wire Line
-	8500 2150 8500 2200
-Connection ~ 8500 2200
 Wire Wire Line
 	3050 2750 3050 3350
@@
 Connection ~ 8650 6200
 $Comp
+L Connector:TestPoint TP6
+U 1 1 5C2E8C62
+P 9100 3200
+F 0 "TP6" V 9054 3387 50  0000 L CNN
+F 1 "GND" V 9145 3387 50  0000 L CNN
+F 2 "TestPoint:TestPoint_Pad_1.5x1.5mm" H 9300 3200 50  0001 C CNN
+F 3 "~" H 9300 3200 50  0001 C CNN
+	1    9100 3200
+	0    1    1    0
+$EndComp
+$Comp
+L Connector:TestPoint TP7
+U 1 1 5C2E908C
+P 9100 3350
+F 0 "TP7" V 9054 3537 50  0000 L CNN
+F 1 "GND" V 9145 3537 50  0000 L CNN
+F 2 "TestPoint:TestPoint_THTPad_1.5x1.5mm_Drill0.7mm" H 9300 3350 50  0001 C CNN
+F 3 "~" H 9300 3350 50  0001 C CNN
+	1    9100 3350
+	0    1    1    0
+$EndComp
+Wire Wire Line
+	8750 3350 9100 3350
+Connection ~ 8750 3350
+Wire Wire Line
+	9100 3200 8750 3200
+Connection ~ 8750 3200
+Wire Wire Line
+	8750 3200 8750 3350
+Wire Wire Line
+	7650 2200 8300 2200
+Wire Wire Line
+	7350 2200 7150 2200
+$Comp
+L Device:L L2
+U 1 1 5B5E85F4
+P 7500 2200
+F 0 "L2" V 7690 2200 50  0000 C CNN
+F 1 "3.3µH/XAL6030-332" V 7599 2200 50  0000 C CNN
+F 2 "Custom Parts:L_CoilCraft_XAL60xx" H 7500 2200 50  0001 C CNN
+F 3 "~" H 7500 2200 50  0001 C CNN
+	1    7500 2200
+	0    -1   -1   0
+$EndComp
+$Comp
 L Connector:TestPoint TP5
 U 1 1 5C2ACBFC
-P 8800 2200
-F 0 "TP5" V 8754 2388 50  0000 L CNN
-F 1 "5V" V 8845 2388 50  0000 L CNN
-F 2 "TestPoint:TestPoint_THTPad_1.5x1.5mm_Drill0.7mm" H 9000 2200 50  0001 C CNN
-F 3 "~" H 9000 2200 50  0001 C CNN
-	1    8800 2200
+P 9350 2200
+F 0 "TP5" V 9304 2388 50  0000 L CNN
+F 1 "5V" V 9395 2388 50  0000 L CNN
+F 2 "TestPoint:TestPoint_THTPad_1.5x1.5mm_Drill0.7mm" H 9550 2200 50  0001 C CNN
+F 3 "~" H 9550 2200 50  0001 C CNN
+	1    9350 2200
 	0    1    1    0
 $EndComp
 Wire Wire Line
-	8800 2200 8500 2200
-$Comp
-L Connector:TestPoint TP6
-U 1 1 5C2E8C62
-P 8850 3200
-F 0 "TP6" V 8804 3387 50  0000 L CNN
-F 1 "GND" V 8895 3387 50  0000 L CNN
-F 2 "TestPoint:TestPoint_Pad_1.5x1.5mm" H 9050 3200 50  0001 C CNN
-F 3 "~" H 9050 3200 50  0001 C CNN
-	1    8850 3200
+	8750 2200 8750 2850
+$Comp
+L Connector_Generic:Conn_01x03 J?
+U 1 1 5CE8562B
+P 9000 1800
+F 0 "J?" V 8964 1612 50  0000 R CNN
+F 1 "PWR" V 8873 1612 50  0000 R CNN
+F 2 "Connector_PinHeader_2.54mm:PinHeader_1x03_P2.54mm_Vertical" H 9000 1800 50  0001 C CNN
+F 3 "~" H 9000 1800 50  0001 C CNN
+	1    9000 1800
+	0    -1   -1   0
+$EndComp
+Wire Wire Line
+	9000 2000 9000 2200
+Wire Wire Line
+	8900 2000 8900 2200
+Wire Wire Line
+	8900 2200 8750 2200
+Connection ~ 8750 2200
+Wire Wire Line
+	9100 2000 9100 2050
+Text GLabel 9150 2050 2    50   Input ~ 0
+USB_5V
+Wire Wire Line
+	9100 2050 9150 2050
+Wire Wire Line
+	9000 2200 9350 2200
+Wire Wire Line
+	9450 2400 9000 2400
+Wire Wire Line
+	9000 2400 9000 2200
+Connection ~ 9000 2200
+$Comp
+L power:PWR_FLAG #FLG?
+U 1 1 5D0278A5
+P 9150 2550
+F 0 "#FLG?" H 9150 2625 50  0001 C CNN
+F 1 "PWR_FLAG" V 9150 2678 50  0000 L CNN
+F 2 "" H 9150 2550 50  0001 C CNN
+F 3 "~" H 9150 2550 50  0001 C CNN
+	1    9150 2550
 	0    1    1    0
 $EndComp
-$Comp
-L Connector:TestPoint TP7
-U 1 1 5C2E908C
-P 8850 3350
-F 0 "TP7" V 8804 3537 50  0000 L CNN
-F 1 "GND" V 8895 3537 50  0000 L CNN
-F 2 "TestPoint:TestPoint_THTPad_1.5x1.5mm_Drill0.7mm" H 9050 3350 50  0001 C CNN
-F 3 "~" H 9050 3350 50  0001 C CNN
-	1    8850 3350
-	0    1    1    0
-$EndComp
-Wire Wire Line
-	8500 3350 8850 3350
-Connection ~ 8500 3350
-Wire Wire Line
-	8850 3200 8500 3200
-Connection ~ 8500 3200
-Wire Wire Line
-	8500 3200 8500 3350
+Wire Wire Line
+	9150 2550 9000 2550
+Wire Wire Line
+	9000 2550 9000 2400
+Connection ~ 9000 2400
 $EndSCHEMATC

Commit message: hardware/mainboard: Switch debug/power connector from micro-B to C
Signed-off-by: David Shah <dave@ds0.me>
Parts:
- gave numbers to parts that had none: 1
Changed lines of the file:
@@
 	8750 2200 8750 2850
 $Comp
-L Connector_Generic:Conn_01x03 J?
+L Connector_Generic:Conn_01x03 J15
 U 1 1 5CE8562B
 P 9000 1800
-F 0 "J?" V 8964 1612 50  0000 R CNN
+F 0 "J15" V 8964 1612 50  0000 R CNN
 F 1 "PWR" V 8873 1612 50  0000 R CNN
 F 2 "Connector_PinHeader_2.54mm:PinHeader_1x03_P2.54mm_Vertical" H 9000 1800 50  0001 C CNN
@@
 Connection ~ 9000 2200
 $Comp
-L power:PWR_FLAG #FLG?
+L power:PWR_FLAG #FLG0101
 U 1 1 5D0278A5
 P 9150 2550
-F 0 "#FLG?" H 9150 2625 50  0001 C CNN
+F 0 "#FLG0101" H 9150 2625 50  0001 C CNN
 F 1 "PWR_FLAG" V 9150 2678 50  0000 L CNN
 F 2 "" H 9150 2550 50  0001 C CNN
