File: hardware/ecp5_mainboard/fpga_pwr.sch (KiCad schematic (older format))
At the start: 62 parts

Commit message: ecp5_mainboard: Run ERC and fix issues
Signed-off-by: David Shah <davey1576@gmail.com>
Parts:
- L301, L302, L303, L304, L305: renamed from L?; value Ferrite_Bead -> 100R@100MHz
- gave numbers to parts that had none: 57
