File: hardware/ecp5_mainboard/debug.sch (KiCad schematic (older format))
At the start: 34 parts

Commit message: hardware/mainboard: Re-annotate and fix ERC
Signed-off-by: David Shah <dave@ds0.me>
Parts:
- gave numbers to parts that had none: 34
Connections:
- no-connect marks 17 -> 23

Commit message: hardware/mainboard: Assign some footprints
Signed-off-by: David Shah <dave@ds0.me>
Parts:
- C87, C88, C91, C92, C94, C95, C97, C98: footprint (none) -> Capacitor_SMD:C_0402_1005Metric
- C89, C90, C93, C96: footprint (none) -> Capacitor_SMD:C_0603_1608Metric
- D12: footprint (none) -> LED_SMD:LED_0805_2012Metric
- L12, L13: footprint (none) -> Inductor_SMD:L_0603_1608Metric
- R34, R35, R36, R37, R38, R39, R40, R41, R46: footprint (none) -> Resistor_SMD:R_0402_1005Metric
- R42, R43, R44, R45: footprint (none) -> Resistor_SMD:R_0805_2012Metric
- RN2, RN3: footprint (none) -> Resistor_SMD:R_Array_Convex_4x0402
- U12: footprint (none) -> Package_TO_SOT_SMD:SOT-23-6
- U13: footprint (none) -> Package_QFP:LQFP-64_10x10mm_P0.5mm
Changed lines of the file:
@@
 F 0 "U13" H 8200 4000 50  0000 C CNN
 F 1 "FT2232H" H 8200 3900 50  0000 C CNN
-F 2 "" H 8200 3950 50  0001 C CNN
+F 2 "Package_QFP:LQFP-64_10x10mm_P0.5mm" H 8200 3950 50  0001 C CNN
 F 3 "http://www.ftdichip.com/Products/ICs/FT2232H.html" H 8200 3950 50  0001 C CNN
 	1    8200 3950
@@
 F 0 "R34" V 4900 3850 50  0000 C CNN
 F 1 "0R" V 5000 3850 50  0000 C CNN
-F 2 "" H 5000 3850 50  0001 C CNN
+F 2 "Resistor_SMD:R_0402_1005Metric" H 5000 3850 50  0001 C CNN
 F 3 "~" H 5000 3850 50  0001 C CNN
 	1    5000 3850
@@
 F 0 "R35" V 4900 4050 50  0000 C CNN
 F 1 "0R" V 5000 4050 50  0000 C CNN
-F 2 "" H 5000 4050 50  0001 C CNN
+F 2 "Resistor_SMD:R_0402_1005Metric" H 5000 4050 50  0001 C CNN
 F 3 "~" H 5000 4050 50  0001 C CNN
 	1    5000 4050
@@
 F 0 "R40" V 6650 3550 50  0000 C CNN
 F 1 "10k" V 6750 3550 50  0000 C CNN
-F 2 "" H 6750 3550 50  0001 C CNN
+F 2 "Resistor_SMD:R_0402_1005Metric" H 6750 3550 50  0001 C CNN
 F 3 "~" H 6750 3550 50  0001 C CNN
 	1    6750 3550
@@
 F 0 "R39" V 6650 3350 50  0000 C CNN
 F 1 "12k" V 6750 3350 50  0000 C CNN
-F 2 "" H 6750 3350 50  0001 C CNN
+F 2 "Resistor_SMD:R_0402_1005Metric" H 6750 3350 50  0001 C CNN
 F 3 "~" H 6750 3350 50  0001 C CNN
 	1    6750 3350
@@
 F 0 "C96" H 8742 1246 50  0000 L CNN
 F 1 "4.7µ" H 8742 1155 50  0000 L CNN
-F 2 "" H 8650 1200 50  0001 C CNN
+F 2 "Capacitor_SMD:C_0603_1608Metric" H 8650 1200 50  0001 C CNN
 F 3 "~" H 8650 1200 50  0001 C CNN
 	1    8650 1200
@@
 F 0 "C97" H 9042 1246 50  0000 L CNN
 F 1 "470n" H 9042 1155 50  0000 L CNN
-F 2 "" H 8950 1200 50  0001 C CNN
+F 2 "Capacitor_SMD:C_0402_1005Metric" H 8950 1200 50  0001 C CNN
 F 3 "~" H 8950 1200 50  0001 C CNN
 	1    8950 1200
@@
 F 0 "C98" H 9392 1246 50  0000 L CNN
 F 1 "470n" H 9392 1155 50  0000 L CNN
-F 2 "" H 9300 1200 50  0001 C CNN
+F 2 "Capacitor_SMD:C_0402_1005Metric" H 9300 1200 50  0001 C CNN
 F 3 "~" H 9300 1200 50  0001 C CNN
 	1    9300 1200
@@
 F 0 "C95" H 7892 1246 50  0000 L CNN
 F 1 "470n" H 7892 1155 50  0000 L CNN
-F 2 "" H 7800 1200 50  0001 C CNN
+F 2 "Capacitor_SMD:C_0402_1005Metric" H 7800 1200 50  0001 C CNN
 F 3 "~" H 7800 1200 50  0001 C CNN
 	1    7800 1200
@@
 F 0 "C94" H 7592 1246 50  0000 L CNN
 F 1 "470n" H 7592 1155 50  0000 L CNN
-F 2 "" H 7500 1200 50  0001 C CNN
+F 2 "Capacitor_SMD:C_0402_1005Metric" H 7500 1200 50  0001 C CNN
 F 3 "~" H 7500 1200 50  0001 C CNN
 	1    7500 1200
@@
 F 0 "C93" H 7292 1246 50  0000 L CNN
 F 1 "4.7µ" H 7292 1155 50  0000 L CNN
-F 2 "" H 7200 1200 50  0001 C CNN
+F 2 "Capacitor_SMD:C_0603_1608Metric" H 7200 1200 50  0001 C CNN
 F 3 "~" H 7200 1200 50  0001 C CNN
 	1    7200 1200
@@
 F 0 "L13" V 5126 1500 50  0000 C CNN
 F 1 "Ferrite_Bead" V 5217 1500 50  0000 C CNN
-F 2 "" V 5330 1500 50  0001 C CNN
+F 2 "Inductor_SMD:L_0603_1608Metric" V 5330 1500 50  0001 C CNN
 F 3 "~" H 5400 1500 50  0001 C CNN
 	1    5400 1500
@@
 F 0 "L12" V 5076 1900 50  0000 C CNN
 F 1 "Ferrite_Bead" V 5167 1900 50  0000 C CNN
-F 2 "" V 5280 1900 50  0001 C CNN
+F 2 "Inductor_SMD:L_0603_1608Metric" V 5280 1900 50  0001 C CNN
 F 3 "~" H 5350 1900 50  0001 C CNN
 	1    5350 1900
@@
 F 0 "C89" H 5692 2146 50  0000 L CNN
 F 1 "4.7µ" H 5692 2055 50  0000 L CNN
-F 2 "" H 5600 2100 50  0001 C CNN
+F 2 "Capacitor_SMD:C_0603_1608Metric" H 5600 2100 50  0001 C CNN
 F 3 "~" H 5600 2100 50  0001 C CNN
 	1    5600 2100
@@
 F 0 "C90" H 5992 2146 50  0000 L CNN
 F 1 "4.7µ" H 5992 2055 50  0000 L CNN
-F 2 "" H 5900 2100 50  0001 C CNN
+F 2 "Capacitor_SMD:C_0603_1608Metric" H 5900 2100 50  0001 C CNN
 F 3 "~" H 5900 2100 50  0001 C CNN
 	1    5900 2100
@@
 F 0 "C91" H 6292 2146 50  0000 L CNN
 F 1 "470n" H 6292 2055 50  0000 L CNN
-F 2 "" H 6200 2100 50  0001 C CNN
+F 2 "Capacitor_SMD:C_0402_1005Metric" H 6200 2100 50  0001 C CNN
 F 3 "~" H 6200 2100 50  0001 C CNN
 	1    6200 2100
@@
 F 0 "C92" H 6592 2146 50  0000 L CNN
 F 1 "470n" H 6592 2055 50  0000 L CNN
-F 2 "" H 6500 2100 50  0001 C CNN
+F 2 "Capacitor_SMD:C_0402_1005Metric" H 6500 2100 50  0001 C CNN
 F 3 "~" H 6500 2100 50  0001 C CNN
 	1    6500 2100
@@
 F 0 "R36" V 5704 6550 50  0000 C CNN
 F 1 "22" V 5795 6550 50  0000 C CNN
-F 2 "" H 5900 6550 50  0001 C CNN
+F 2 "Resistor_SMD:R_0402_1005Metric" H 5900 6550 50  0001 C CNN
 F 3 "~" H 5900 6550 50  0001 C CNN
 	1    5900 6550
@@
 F 0 "R37" V 5704 6850 50  0000 C CNN
 F 1 "22" V 5795 6850 50  0000 C CNN
-F 2 "" H 5900 6850 50  0001 C CNN
+F 2 "Resistor_SMD:R_0402_1005Metric" H 5900 6850 50  0001 C CNN
 F 3 "~" H 5900 6850 50  0001 C CNN
 	1    5900 6850
@@
 F 0 "C88" V 4721 6150 50  0000 C CNN
 F 1 "100n" V 4812 6150 50  0000 C CNN
-F 2 "" H 4950 6150 50  0001 C CNN
+F 2 "Capacitor_SMD:C_0402_1005Metric" H 4950 6150 50  0001 C CNN
 F 3 "~" H 4950 6150 50  0001 C CNN
 	1    4950 6150
@@
 F 0 "U12" H 5150 5815 50  0000 C CNN
 F 1 "93AA46B_OT" H 5150 5724 50  0000 C CNN
-F 2 "" H 5150 5400 50  0001 C CNN
+F 2 "Package_TO_SOT_SMD:SOT-23-6" H 5150 5400 50  0001 C CNN
 F 3 "http://ww1.microchip.com/downloads/en/DeviceDoc/20001749K.pdf" H 5150 5400 50  0001 C CNN
 	1    5150 5400
@@
 F 0 "C87" H 4142 5446 50  0000 L CNN
 F 1 "470n" H 4142 5355 50  0000 L CNN
-F 2 "" H 4050 5400 50  0001 C CNN
+F 2 "Capacitor_SMD:C_0402_1005Metric" H 4050 5400 50  0001 C CNN
 F 3 "~" H 4050 5400 50  0001 C CNN
 	1    4050 5400
@@
 F 0 "R38" V 6350 5550 50  0000 C CNN
 F 1 "2.2k" V 6250 5550 50  0000 C CNN
-F 2 "" H 6250 5550 50  0001 C CNN
+F 2 "Resistor_SMD:R_0402_1005Metric" H 6250 5550 50  0001 C CNN
 F 3 "~" H 6250 5550 50  0001 C CNN
 	1    6250 5550
@@
 F 0 "RN2" V 4783 4750 50  0000 C CNN
 F 1 "10k" V 4874 4750 50  0000 C CNN
-F 2 "" V 5475 4750 50  0001 C CNN
+F 2 "Resistor_SMD:R_Array_Convex_4x0402" V 5475 4750 50  0001 C CNN
 F 3 "~" H 5200 4750 50  0001 C CNN
 	1    5200 4750
@@
 F 0 "R42" V 9650 2200 50  0000 C CNN
 F 1 "0R" V 9700 2050 50  0000 C CNN
-F 2 "" H 9700 2050 50  0001 C CNN
+F 2 "Resistor_SMD:R_0805_2012Metric" H 9700 2050 50  0001 C CNN
 F 3 "~" H 9700 2050 50  0001 C CNN
 	1    9700 2050
@@
 F 0 "R43" V 9650 2300 50  0000 C CNN
 F 1 "0R" V 9700 2150 50  0000 C CNN
-F 2 "" H 9700 2150 50  0001 C CNN
+F 2 "Resistor_SMD:R_0805_2012Metric" H 9700 2150 50  0001 C CNN
 F 3 "~" H 9700 2150 50  0001 C CNN
 	1    9700 2150
@@
 F 0 "R44" V 9650 2400 50  0000 C CNN
 F 1 "0R" V 9700 2250 50  0000 C CNN
-F 2 "" H 9700 2250 50  0001 C CNN
+F 2 "Resistor_SMD:R_0805_2012Metric" H 9700 2250 50  0001 C CNN
 F 3 "~" H 9700 2250 50  0001 C CNN
 	1    9700 2250
@@
 F 0 "R45" V 9650 2500 50  0000 C CNN
 F 1 "0R" V 9700 2350 50  0000 C CNN
-F 2 "" H 9700 2350 50  0001 C CNN
+F 2 "Resistor_SMD:R_0805_2012Metric" H 9700 2350 50  0001 C CNN
 F 3 "~" H 9700 2350 50  0001 C CNN
 	1    9700 2350
@@
 F 0 "D12" H 10091 2916 50  0000 C CNN
 F 1 "GREEN" H 10091 2825 50  0000 C CNN
-F 2 "" H 10100 2700 50  0001 C CNN
+F 2 "LED_SMD:LED_0805_2012Metric" H 10100 2700 50  0001 C CNN
 F 3 "~" H 10100 2700 50  0001 C CNN
 	1    10100 2700
@@
 F 0 "R46" V 10304 2700 50  0000 C CNN
 F 1 "1.5k" V 10395 2700 50  0000 C CNN
-F 2 "" H 10500 2700 50  0001 C CNN
+F 2 "Resistor_SMD:R_0402_1005Metric" H 10500 2700 50  0001 C CNN
 F 3 "~" H 10500 2700 50  0001 C CNN
 	1    10500 2700
@@
 F 0 "R41" V 9650 2050 50  0000 C CNN
 F 1 "10k" V 9700 1900 50  0000 C CNN
-F 2 "" H 9700 1900 50  0001 C CNN
+F 2 "Resistor_SMD:R_0402_1005Metric" H 9700 1900 50  0001 C CNN
 F 3 "~" H 9700 1900 50  0001 C CNN
 	1    9700 1900
@@
 F 0 "RN3" V 9733 5700 50  0000 C CNN
 F 1 "R_Pack04" V 9824 5700 50  0000 C CNN
-F 2 "" V 10425 5700 50  0001 C CNN
+F 2 "Resistor_SMD:R_Array_Convex_4x0402" V 10425 5700 50  0001 C CNN
 F 3 "~" H 10150 5700 50  0001 C CNN
 	1    10150 5700

Commit message: hardware/mainboard: Assign more footprints
Signed-off-by: David Shah <dave@ds0.me>
Parts:
- J2: footprint (none) -> Connector_USB:USB_Micro-B_Molex-105017-0001
Changed lines of the file:
@@
 F 0 "J2" H 3355 4317 50  0000 C CNN
 F 1 "USB_B_Micro" H 3355 4226 50  0000 C CNN
-F 2 "" H 3450 3800 50  0001 C CNN
+F 2 "Connector_USB:USB_Micro-B_Molex-105017-0001" H 3450 3800 50  0001 C CNN
 F 3 "~" H 3450 3800 50  0001 C CNN
 	1    3300 3850
