File: hardware/ecp5_mainboard/debug.sch (KiCad schematic (older format))
At the start: 34 parts, among them J2 USB_B_Micro, U12 93AA46B_OT, U13 FT2232H, X1 XO32

Commit message: hardware/mainboard: BoM fixes, add USB power option
Signed-off-by: David Shah <dave@ds0.me>
Parts:
- RN3: value R_Pack04 -> 10k
- X1: value XO32 -> 12MHz
Connections:
- net USB_5V: now reaches J2.1 (VBUS)
- no-connect marks 23 -> 22
Changed lines of the file:
@@
 EESchema Schematic File Version 4
 LIBS:ecp5_mainboard-cache
-EELAYER 26 0
+EELAYER 29 0
 EELAYER END
 $Descr A4 11693 8268
@@
 P 5200 6550
 F 0 "X1" H 5541 6596 50  0000 L CNN
-F 1 "XO32" H 5541 6505 50  0000 L CNN
+F 1 "12MHz" H 5541 6505 50  0000 L CNN
 F 2 "Oscillator:Oscillator_SMD_EuroQuartz_XO32-4Pin_3.2x2.5mm" H 5900 6200 50  0001 C CNN
 F 3 "http://cdn-reichelt.de/documents/datenblatt/B400/XO32.pdf" H 5100 6550 50  0001 C CNN
@@
 P 10150 5700
 F 0 "RN3" V 9733 5700 50  0000 C CNN
-F 1 "R_Pack04" V 9824 5700 50  0000 C CNN
+F 1 "10k" V 9824 5700 50  0000 C CNN
 F 2 "Resistor_SMD:R_Array_Convex_4x0402" V 10425 5700 50  0001 C CNN
 F 3 "~" H 10150 5700 50  0001 C CNN
@@
 Wire Wire Line
 	3300 4350 3300 4250
-NoConn ~ 3600 3650
 NoConn ~ 9400 5250
 NoConn ~ 9400 5350
@@
 NoConn ~ 9400 2650
 NoConn ~ 9400 2750
+Wire Wire Line
+	4150 3500 3900 3500
+Wire Wire Line
+	3900 3500 3900 3650
+Wire Wire Line
+	3900 3650 3600 3650
+Text GLabel 4150 3500 2    50   Output ~ 0
+USB_5V
 $EndSCHEMATC

Commit message: hardware/mainboard: Switch debug/power connector from micro-B to C
Signed-off-by: David Shah <dave@ds0.me>
Parts:
- removed J2: USB_B_Micro, Connector_USB:USB_Micro-B_Molex-105017-0001, symbol Connector:USB_B_Micro
- added J?: USB_C_Receptacle, Connector_USB:USB_C_Receptacle_Amphenol_12401610E4-2A, symbol Connector:USB_C_Receptacle
Connections:
- net GND: now also J?.A1 (GND), J?.A12 (GND), J?.B1 (GND), J?.B12 (GND), J?.S1 (SHIELD)
- net PORT_D+: now also J?.A6 (D+), J?.B6 (D+)
- net PORT_D-: now also J?.A7 (D-), J?.B7 (D-)
- net USB_5V: now also J?.A4 (VBUS), J?.A9 (VBUS), J?.B4 (VBUS), J?.B9 (VBUS)
- no-connect marks 22 -> 33
Changed lines of the file:
@@
 Wire Wire Line
 	10500 5700 10500 5800
+Text Label 3900 4050 0    50   ~ 0
+PORT_D+
+Text Label 3800 3850 0    50   ~ 0
+PORT_D-
 $Comp
-L Connector:USB_B_Micro J2
-U 1 1 61582E96
-P 3300 3850
-F 0 "J2" H 3355 4317 50  0000 C CNN
-F 1 "USB_B_Micro" H 3355 4226 50  0000 C CNN
-F 2 "Connector_USB:USB_Micro-B_Molex-105017-0001" H 3450 3800 50  0001 C CNN
-F 3 "~" H 3450 3800 50  0001 C CNN
-	1    3300 3850
+L power:GND #PWR068
+U 1 1 615FD047
+P 2450 6050
+F 0 "#PWR068" H 2450 5800 50  0001 C CNN
+F 1 "GND" H 2455 5877 50  0000 C CNN
+F 2 "" H 2450 6050 50  0001 C CNN
+F 3 "" H 2450 6050 50  0001 C CNN
+	1    2450 6050
 	1    0    0    -1
 $EndComp
 Wire Wire Line
-	3600 3850 4350 3850
+	2450 6050 2450 5950
 Wire Wire Line
-	4350 3850 4550 4050
+	2450 5950 2300 5950
 Wire Wire Line
-	4900 4050 4550 4050
-Wire Wire Line
-	4900 3850 4450 3850
-Wire Wire Line
-	4450 3850 4350 3950
-Wire Wire Line
-	4350 3950 3600 3950
-Text Label 3700 3850 0    50   ~ 0
-PORT_D+
-Text Label 3700 3950 0    50   ~ 0
-PORT_D-
-NoConn ~ 3600 4050
-$Comp
-L power:GND #PWR068
-U 1 1 615FD047
-P 3300 4450
-F 0 "#PWR068" H 3300 4200 50  0001 C CNN
-F 1 "GND" H 3305 4277 50  0000 C CNN
-F 2 "" H 3300 4450 50  0001 C CNN
-F 3 "" H 3300 4450 50  0001 C CNN
-	1    3300 4450
-	1    0    0    -1
-$EndComp
-Wire Wire Line
-	3300 4450 3300 4350
-Wire Wire Line
-	3300 4350 3200 4350
-Wire Wire Line
-	3200 4350 3200 4250
-Connection ~ 3300 4350
-Wire Wire Line
-	3300 4350 3300 4250
+	2300 5950 2300 5850
 NoConn ~ 9400 5250
 NoConn ~ 9400 5350
@@
 NoConn ~ 9400 2650
 NoConn ~ 9400 2750
+Text GLabel 3400 3250 2    50   Output ~ 0
+USB_5V
+$Comp
+L Connector:USB_C_Receptacle J?
+U 1 1 5D1382FA
+P 2600 4250
+F 0 "J?" H 2707 5517 50  0000 C CNN
+F 1 "USB_C_Receptacle" H 2707 5426 50  0000 C CNN
+F 2 "Connector_USB:USB_C_Receptacle_Amphenol_12401610E4-2A" H 2750 4250 50  0001 C CNN
+F 3 "https://www.usb.org/sites/default/files/documents/usb_type-c.zip" H 2750 4250 50  0001 C CNN
+	1    2600 4250
+	1    0    0    -1
+$EndComp
 Wire Wire Line
-	4150 3500 3900 3500
+	3200 3850 3300 3850
 Wire Wire Line
-	3900 3500 3900 3650
+	3200 3750 3300 3750
 Wire Wire Line
-	3900 3650 3600 3650
-Text GLabel 4150 3500 2    50   Output ~ 0
-USB_5V
+	3300 3750 3300 3850
+Connection ~ 3300 3850
+Wire Wire Line
+	3300 3850 4900 3850
+Wire Wire Line
+	3200 4050 3300 4050
+Wire Wire Line
+	3200 3950 3300 3950
+Wire Wire Line
+	3300 3950 3300 4050
+Connection ~ 3300 4050
+Wire Wire Line
+	3300 4050 4900 4050
+Wire Wire Line
+	3200 3250 3400 3250
+Wire Wire Line
+	2600 5850 2600 5950
+Wire Wire Line
+	2600 5950 2450 5950
+Connection ~ 2450 5950
+NoConn ~ 3200 5450
+NoConn ~ 3200 5550
+NoConn ~ 3200 5250
+NoConn ~ 3200 5150
+NoConn ~ 3200 4950
+NoConn ~ 3200 4850
+NoConn ~ 3200 4650
+NoConn ~ 3200 4550
+NoConn ~ 3200 4350
+NoConn ~ 3200 4250
+NoConn ~ 3200 3450
+NoConn ~ 3200 3550
 $EndSCHEMATC

Commit message: hardware/mainboard: RefDes silkscreen improvements
Signed-off-by: David Shah <dave@ds0.me>
Parts:
- gave numbers to parts that had none: 1
Changed lines of the file:
@@
 USB_5V
 $Comp
-L Connector:USB_C_Receptacle J?
+L Connector:USB_C_Receptacle J2
 U 1 1 5D1382FA
 P 2600 4250
-F 0 "J?" H 2707 5517 50  0000 C CNN
+F 0 "J2" H 2707 5517 50  0000 C CNN
 F 1 "USB_C_Receptacle" H 2707 5426 50  0000 C CNN
 F 2 "Connector_USB:USB_C_Receptacle_Amphenol_12401610E4-2A" H 2750 4250 50  0001 C CNN
