File: hardware/ecp5_mainboard/usbc_dp.sch (KiCad schematic (older format))
At the start: 1 part

Commit message: ecp5_mainboard: Starting USB-C and DP schematics
Signed-off-by: David Shah <davey1576@gmail.com>
Parts:
- added C?: 1µ, symbol Device:C_Small
- added C? (x7): 100n, symbol Device:C_Small
- added C?: 10n, symbol Device:C_Small
- added C? (x6): 470n, symbol Device:C_Small
- added C?: 4.7µ, symbol Device:C_Small
- added C? (x2): 12p, symbol Device:C_Small
- added C?: 47µ, symbol Device:CP_Small
- added DA? (x2): TPD4E02B04, symbol eco_interface:TPD4E02B04
- added DA?: TPD4E05U06, symbol eco_interface:TPD4E05U06
- added J?: USB_C_Receptacle, symbol Connector:USB_C_Receptacle
- added J? (x2): SMA/DNP, symbol Connector:Conn_Coaxial
- added L?: L_Core_Ferrite, symbol Device:L_Core_Ferrite
- added P?: miniDP_sink, symbol eco_connectors:miniDP_sink
- added P?: miniDP_source, symbol eco_connectors:miniDP_source
- added R?: 2.2, symbol Device:R_Small
- added R? (x2): 100, symbol Device:R_Small
- added R? (x5): 10k, symbol Device:R_Small
- added R?: 22, symbol Device:R_Small
- added U?: 5P49V6965, symbol eco_glue:5P49V6965
- added U?: USB3300-EZK, Package_DFN_QFN:QFN-32-1EP_5x5mm_P0.5mm_EP3.45x3.45mm, symbol Interface_USB:USB3300-EZK
- added U? (x2): CBTL02043A, symbol eco_glue:CBTL02043A
- added U?: TPS2041B, Package_TO_SOT_SMD:SOT-23-5, symbol Power_Management:TPS2041B
- added Y?: 25MHz, symbol Device:Crystal_GND24
Connections:
- net labels added: +1V8, +3.3V, +3V3, +5V, 1V8C, 1V8CA, CLKIN+, CLKIN-, CLKINC+, CLKINC-, DP_RX0+, DP_RX0-, DP_RX1+, DP_RX1-, DP_TX0+, DP_TX0-, DP_TX1+, DP_TX1-, GND, HS_RX_SEL, HS_TX_SEL, I2C0_SCL, I2C0_SDA, REFCLK0+, REFCLK0-, REFCLK1, RX0+, RX0-, RX1+, RX1-, TX0+, TX0-, TX1+, TX1-, USBC_CC1, USBC_CC2, USBC_C_TX1+, USBC_C_TX1-, USBC_C_TX2+, USBC_C_TX2-, USBC_D+, USBC_D-, USBC_PWR~EN, USBC_RX0+, USBC_RX0-, USBC_RX1+, USBC_RX1-, USBC_RX2+, USBC_RX2-, USBC_SBU1, USBC_SBU2, USBC_TX0+, USBC_TX0-, USBC_TX1+, USBC_TX1-, USBC_VBUS, XIN, XOUT
- wire segments 2 -> 293
- no-connect marks 0 -> 5
Other:
- note added: "I²C Address 0xD4\n"
- moved on the sheet: U?L

Commit message: ecp5_mainboard: Working on USBC/DP section
Signed-off-by: David Shah <davey1576@gmail.com>
Parts:
- removed U?: USB3300-EZK, Package_DFN_QFN:QFN-32-1EP_5x5mm_P0.5mm_EP3.45x3.45mm, symbol Interface_USB:USB3300-EZK
- added C? (x8): 100n, symbol Device:C_Small
- added C? (x4): 10n, symbol Device:C_Small
- added C? (x12): 470n, symbol Device:C_Small
- added C?: 22µ, symbol Device:C_Small
- added C?: 4.7µ, symbol Device:C_Small
- added D? (x2): GREEN, symbol Device:LED
- added D?: RED, symbol Device:LED
- added D?: RED, symbol Device:LED_Small
- added DA? (x2): TPD4E05U06, symbol eco_interface:TPD4E05U06
- added DA? (x2): TPD4E02B04, symbol eco_interface:TPD4E02B04
- added L? (x2): 60R/1A, symbol Device:Ferrite_Bead_Small
- added R? (x7): 10k, symbol Device:R_Small
- added R? (x3): 1k, symbol Device:R_Small
- added R? (x2): 1.5k, symbol Device:R_Small
- added R? (x4): 51, symbol Device:R_Small
- added R?: 2.49k, symbol Device:R_Small
- added U?: TPS2041B, Package_TO_SOT_SMD:SOT-23-5, symbol Power_Management:TPS2041B
- added U? (x2): SN65MLVD200A, symbol eco_interface:SN65MLVD200A
Connections:
- net labels added: AUX_Vtt, DPC_TX0+, DPC_TX0-, DPC_TX1+, DPC_TX1-, DPRX_AUX+, DPRX_AUX-, DPRX_AUX_EN, DPRX_AUX_RX, DPRX_AUX_TX, DPRX_HPD, DPTX_AUX+, DPTX_AUX-, DPTX_AUX_EN, DPTX_AUX_RX, DPTX_AUX_TX, DPTX_HPD, DP_3V3, DP_PWR~EN, DP_~OC, RX_3V3, RX_AUXT+, RX_AUXT-, TX_3V3, TX_AUXT+, TX_AUXT-
- wire segments 293 -> 596
- no-connect marks 5 -> 16
Other:
- moved on the sheet: C?, DA?, R?, U?, U?L
