File: hardware/ecp5_mainboard/ecp5_mainboard.sch (KiCad schematic (older format))
At the start: 0 parts

Commit message: hardware/mainboard: Major spec change; remove USBC/DP; add PCIe and refclk
Signed-off-by: David Shah <dave@ds0.me>
Changed lines of the file:
@@
 $EndSheet
 $Sheet
-S 1000 3500 2400 1000
-U 5B642DC1
-F0 "USB-C + DisplayPort" 50
-F1 "usbc_dp.sch" 50
+S 1000 3450 2400 800
+U 5C060E84
+F0 "PCIe + SATA" 50
+F1 "serdes.sch" 50
 $EndSheet
 $EndSCHEMATC
