File: hardware/ecp5_mainboard/ecp5_mainboard.sch (KiCad schematic (older format))
At the start: 0 parts

Commit message: hardware/mainboard: Connect DDR3 IO to FPGA IO
Signed-off-by: David Shah <dave@ds0.me>
Changed lines of the file:
@@
 $Descr A4 11693 8268
 encoding utf-8
-Sheet 1 8
+Sheet 1 9
 Title ""
 Date ""
@@
 F1 "ddr3.sch" 50
 $EndSheet
+$Sheet
+S 4500 3500 2400 1700
+U 61FAF948
+F0 "FPGA IO" 50
+F1 "fpga_io.sch" 50
+$EndSheet
 $EndSCHEMATC
