File: hardware/ecp5_mainboard/serdes.sch (KiCad schematic (older format))
At the start: 27 parts

Commit message: hardware/mainboard: Add SATA and SATA REFCLK
Signed-off-by: David Shah <dave@ds0.me>
Parts:
- added C? (x4): 100n, symbol Device:C_Small
- added C?: 470n, symbol Device:C_Small
- added DA? (x4): TPD4E02B04, symbol eco_interface:TPD4E02B04
- added FB?: 200R@100MHz, symbol Device:Ferrite_Bead_Small
- added P? (x2): SATA, symbol eco_connectors:SATA
- added R? (x2): 0R, symbol Device:R_Small
- added R? (x2): DNP, symbol Device:R_Small
- added TP? (x2): DCU1_CLK+, symbol Connector:TestPoint
- added U?: ECP5UM5G_85_CABGA756, symbol ECP5UM5G:ECP5UM5G_85_CABGA756
- added U?: XL_XO_LVDS, symbol eco_glue:XL_XO_LVDS
Connections:
- net DCU0_REFCLK+: now also U?.AM14 (REFCLKP_D0)
- net DCU0_REFCLK-: now also U?.AM15 (REFCLKN_D0)
- net DCU0_RX0+: now also DA?.1 (IO1), DA?.10
- net DCU0_RX0-: now also DA?.2 (IO2), DA?.9
- net DCU0_RX1+: now also DA?.4 (IO3), DA?.7
- net DCU0_RX1-: now also DA?.5 (IO4), DA?.6
- net GND: now also C?.2, DA?.3 (GND), DA?.3 (GND), DA?.3 (GND), DA?.3 (GND), DA?.8, DA?.8, DA?.8, DA?.8, P?.1 (GND), P?.1 (GND), P?.4 (GND), P?.4 (GND), P?.7 (GND), P?.7 (GND), U?.3 (GND)
- net PCIe_HSI0+: now also DA?.1 (IO1), DA?.10
- net PCIe_HSI0-: now also DA?.2 (IO2), DA?.9
- net PCIe_HSI1+: now also DA?.4 (IO3), DA?.7
- net PCIe_HSI1-: now also DA?.5 (IO4), DA?.6
- net CLKAUXO-: now reaches U?.13 (OUT3-)
- net CLKAUXO-: now also R?.2
- net CLKAUXO+: now reaches U?.14 (OUT3+)
- net CLKAUXO+: now also R?.2
- new net: C?.1, FB?.1, U?.6 (Vdd)
- new net +3V3: FB?.2
- new net CLK150M+: R?.2, U?.4 (OUT+)
- new net CLK150M-: R?.2, U?.5 (OUT-)
- new net DCU1_REFCLK+: R?.1, R?.1, TP?.1, U?.AM23 (REFCLKP_D1)
- new net DCU1_REFCLK-: R?.1, R?.1, TP?.1, U?.AM24 (REFCLKN_D1)
- new net DCU1_RX0+: DA?.5 (IO4), DA?.6, P?.6 (B+/RX+), U?.AM17 (HDRXP0_D1CH0)
- new net DCU1_RX0-: DA?.4 (IO3), DA?.7, P?.5 (B-/RX-), U?.AM18 (HDRXN0_D1CH0)
- new net DCU1_RX1+: DA?.5 (IO4), DA?.6, P?.6 (B+/RX+), U?.AK21 (HDTXP0_D1CH1)
- new net DCU1_RX1-: DA?.4 (IO3), DA?.7, P?.5 (B-/RX-), U?.AK22 (HDTXN0_D1CH1)
- new net DCU1_TX0+: C?.2, U?.AK18 (HDTXP0_D1CH0)
- new net DCU1_TX0-: C?.2, U?.AK19 (HDTXN0_D1CH0)
- new net DCU1_TX1+: C?.2, U?.AM20 (HDRXP0_D1CH1)
- new net DCU1_TX1-: C?.2, U?.AM21 (HDRXN0_D1CH1)
- new net SATA0_A+: C?.1, DA?.1 (IO1), DA?.10, P?.2 (A+/TX+)
- new net SATA0_A-: C?.1, DA?.2 (IO2), DA?.9, P?.3 (A-/TX-)
- new net SATA1_A+: C?.1, DA?.1 (IO1), DA?.10, P?.2 (A+/TX+)
- new net SATA1_A-: C?.1, DA?.2 (IO2), DA?.9, P?.3 (A-/TX-)
