File: hardware/ecp5_mainboard/serdes.sch (KiCad schematic (older format))
At the start: 47 parts

Commit message: hardware/mainboard: Connecting more FPGA IO
Signed-off-by: David Shah <dave@ds0.me>
Parts:
- added C?: 10µ, symbol Device:C_Small
- added C?: 470n, symbol Device:C_Small
- added FB?: 200R@100MHz, symbol Device:Ferrite_Bead_Small
- added R?: 1k, symbol Device:R_Small
Connections:
- net +1V8: now also FB?.2; no longer FB?.2
- net +3V3: now also FB?.2
- net 1V8_C: now also C?.1, C?.1, FB?.1; no longer C?.1, C?.1, C?.1, C?.1, C?.1, FB?.1, R?.2, U?.10 (VddO4), U?.18 (VddO2), U?.22 (VddD), U?.23 (VddO0)
- net GND: now also C?.2, C?.2
- net ~PERST: now also R?.1; no longer P?.A11 (~PERST)
- net 1V8_CA renamed 3V3_CA
- new net: P?.A11 (~PERST), R?.2
- new net 3V3_C: C?.1, C?.1, C?.1, C?.1, C?.1, FB?.1, R?.2, U?.10 (VddO4), U?.18 (VddO2), U?.22 (VddD), U?.23 (VddO0)
Changed lines of the file:
@@
 NoConn ~ 1500 3650
 NoConn ~ 1500 3550
-Wire Wire Line
-	3300 2250 3700 2250
-Text GLabel 3700 2250 2    50   Output ~ 0
+Text GLabel 4300 2250 2    50   Output ~ 0
 ~PERST
 Text Label 4050 2550 2    50   ~ 0
@@
 	11800 3550 12550 3550
 $Comp
-L power:+1V8 #PWR?
-U 1 1 5C237E7D
-P 9500 2150
-F 0 "#PWR?" H 9500 2000 50  0001 C CNN
-F 1 "+1V8" H 9515 2323 50  0000 C CNN
-F 2 "" H 9500 2150 50  0001 C CNN
-F 3 "" H 9500 2150 50  0001 C CNN
-	1    9500 2150
-	1    0    0    -1
-$EndComp
-$Comp
 L Device:Ferrite_Bead_Small FB?
 U 1 1 5C238099
@@
 	9850 2950 9850 3050
 Text Label 10250 2600 0    50   ~ 0
-1V8_C
+3V3_C
 Text Label 12100 2600 0    50   ~ 0
-1V8_CA
+3V3_CA
 $Comp
 L power:PWR_FLAG #FLG?
@@
 	12550 2850 12350 2850
 Text Label 12350 2750 0    50   ~ 0
-1V8_C
+3V3_C
 Text Label 12350 2850 0    50   ~ 0
-1V8_C
+3V3_C
 $Comp
 L Device:C_Small C?
@@
 Wire Wire Line
 	11850 3750 12000 3750
-Text Label 14850 2650 2    50   ~ 0
-1V8_C
 Wire Wire Line
 	14850 2650 14550 2650
@@
 	15300 2850 14550 2850
 Text Label 14850 3150 2    50   ~ 0
-1V8_C
+3V3_C
 Wire Wire Line
 	14850 3150 14550 3150
@@
 	14850 3650 14550 3650
 Text Label 14850 4150 2    50   ~ 0
-1V8_C
+3V3_C
 Wire Wire Line
 	14850 4150 14550 4150
@@
 	12150 7850 12150 7750
 Connection ~ 12150 7750
+$Comp
+L Device:R_Small R?
+U 1 1 62339B3D
+P 3850 2250
+F 0 "R?" V 3654 2250 50  0000 C CNN
+F 1 "1k" V 3745 2250 50  0000 C CNN
+F 2 "" H 3850 2250 50  0001 C CNN
+F 3 "~" H 3850 2250 50  0001 C CNN
+	1    3850 2250
+	0    1    1    0
+$EndComp
+Wire Wire Line
+	3750 2250 3300 2250
+Wire Wire Line
+	3950 2250 4300 2250
+$Comp
+L power:+3V3 #PWR?
+U 1 1 62375601
+P 9500 2150
+F 0 "#PWR?" H 9500 2000 50  0001 C CNN
+F 1 "+3V3" H 9515 2323 50  0000 C CNN
+F 2 "" H 9500 2150 50  0001 C CNN
+F 3 "" H 9500 2150 50  0001 C CNN
+	1    9500 2150
+	1    0    0    -1
+$EndComp
+$Comp
+L Device:Ferrite_Bead_Small FB?
+U 1 1 6237B8C5
+P 8350 2400
+F 0 "FB?" H 8250 2354 50  0000 R CNN
+F 1 "200R@100MHz" H 8250 2445 50  0000 R CNN
+F 2 "" V 8280 2400 50  0001 C CNN
+F 3 "~" H 8350 2400 50  0001 C CNN
+	1    8350 2400
+	-1   0    0    1
+$EndComp
+$Comp
+L power:+1V8 #PWR?
+U 1 1 62397E98
+P 8350 2150
+F 0 "#PWR?" H 8350 2000 50  0001 C CNN
+F 1 "+1V8" H 8365 2323 50  0000 C CNN
+F 2 "" H 8350 2150 50  0001 C CNN
+F 3 "" H 8350 2150 50  0001 C CNN
+	1    8350 2150
+	1    0    0    -1
+$EndComp
+Wire Wire Line
+	8350 2150 8350 2300
+Text Label 8450 2600 0    50   ~ 0
+1V8_C
+Wire Wire Line
+	8350 2600 8350 2500
+$Comp
+L power:PWR_FLAG #FLG?
+U 1 1 623D1167
+P 8050 2150
+F 0 "#FLG?" H 8050 2225 50  0001 C CNN
+F 1 "PWR_FLAG" H 8050 2324 50  0000 C CNN
+F 2 "" H 8050 2150 50  0001 C CNN
+F 3 "~" H 8050 2150 50  0001 C CNN
+	1    8050 2150
+	1    0    0    -1
+$EndComp
+Wire Wire Line
+	8050 2150 8050 2600
+Wire Wire Line
+	8050 2600 8350 2600
+Connection ~ 8350 2600
+$Comp
+L Device:C_Small C?
+U 1 1 623EE239
+P 8350 2750
+F 0 "C?" H 8442 2796 50  0000 L CNN
+F 1 "10µ" H 8442 2705 50  0000 L CNN
+F 2 "" H 8350 2750 50  0001 C CNN
+F 3 "~" H 8350 2750 50  0001 C CNN
+	1    8350 2750
+	1    0    0    -1
+$EndComp
+Wire Wire Line
+	8350 2650 8350 2600
+$Comp
+L Device:C_Small C?
+U 1 1 6240B6D8
+P 8750 2750
+F 0 "C?" H 8842 2796 50  0000 L CNN
+F 1 "470n" H 8842 2705 50  0000 L CNN
+F 2 "" H 8750 2750 50  0001 C CNN
+F 3 "~" H 8750 2750 50  0001 C CNN
+	1    8750 2750
+	1    0    0    -1
+$EndComp
+Wire Wire Line
+	8750 2650 8750 2600
+Wire Wire Line
+	8750 2600 8350 2600
+Wire Wire Line
+	8750 2850 8750 2950
+Wire Wire Line
+	8750 2950 8350 2950
+Wire Wire Line
+	8350 2950 8350 2850
+$Comp
+L power:GND #PWR?
+U 1 1 6246401D
+P 8750 3050
+F 0 "#PWR?" H 8750 2800 50  0001 C CNN
+F 1 "GND" H 8755 2877 50  0000 C CNN
+F 2 "" H 8750 3050 50  0001 C CNN
+F 3 "" H 8750 3050 50  0001 C CNN
+	1    8750 3050
+	1    0    0    -1
+$EndComp
+Wire Wire Line
+	8750 3050 8750 2950
+Connection ~ 8750 2950
+Text Label 14850 2650 2    50   ~ 0
+1V8_C
 $EndSCHEMATC

Commit message: hardware/mainboard: Re-annotate and fix ERC
Signed-off-by: David Shah <dave@ds0.me>
Parts:
- gave numbers to parts that had none: 50
Other:
- moved on the sheet: FB3

Commit message: hardware/mainboard: Assign some footprints
Signed-off-by: David Shah <dave@ds0.me>
Parts:
- C100, C101, C102, C103, C104, C105, C106, C108, C110, C111, C112, C113, C114, C115, C116, C117, C118, C99: footprint (none) -> Capacitor_SMD:C_0402_1005Metric
- C107, C109: footprint (none) -> Capacitor_SMD:C_0805_2012Metric
- D13: footprint (none) -> LED_SMD:LED_0805_2012Metric
- FB1, FB2, FB3: footprint (none) -> Inductor_SMD:L_0603_1608Metric
- R47, R48, R49, R50, R51, R52, R57, R58: footprint (none) -> Resistor_SMD:R_0402_1005Metric
- R53, R54, R55, R56: footprint (none) -> Resistor_SMD:R_0805_2012Metric
- U16: footprint (none) -> Package_DFN_QFN:QFN-24-1EP_4x4mm_P0.5mm_EP2.7x2.7mm
Changed lines of the file:
@@
 F 0 "C103" V 4550 2850 50  0000 C CNN
 F 1 "100n" V 4150 2850 50  0000 C CNN
-F 2 "" H 4350 2850 50  0001 C CNN
+F 2 "Capacitor_SMD:C_0402_1005Metric" H 4350 2850 50  0001 C CNN
 F 3 "~" H 4350 2850 50  0001 C CNN
 	1    4350 2850
@@
 F 0 "C104" V 4550 2950 50  0000 C CNN
 F 1 "100n" V 4150 2950 50  0000 C CNN
-F 2 "" H 4350 2950 50  0001 C CNN
+F 2 "Capacitor_SMD:C_0402_1005Metric" H 4350 2950 50  0001 C CNN
 F 3 "~" H 4350 2950 50  0001 C CNN
 	1    4350 2950
@@
 F 0 "C105" V 4550 3350 50  0000 C CNN
 F 1 "100n" V 4150 3350 50  0000 C CNN
-F 2 "" H 4350 3350 50  0001 C CNN
+F 2 "Capacitor_SMD:C_0402_1005Metric" H 4350 3350 50  0001 C CNN
 F 3 "~" H 4350 3350 50  0001 C CNN
 	1    4350 3350
@@
 F 0 "C106" V 4550 3450 50  0000 C CNN
 F 1 "100n" V 4150 3450 50  0000 C CNN
-F 2 "" H 4350 3450 50  0001 C CNN
+F 2 "Capacitor_SMD:C_0402_1005Metric" H 4350 3450 50  0001 C CNN
 F 3 "~" H 4350 3450 50  0001 C CNN
 	1    4350 3450
@@
 F 0 "R48" V 4204 850 50  0000 C CNN
 F 1 "4.7k" V 4295 850 50  0000 C CNN
-F 2 "" H 4400 850 50  0001 C CNN
+F 2 "Resistor_SMD:R_0402_1005Metric" H 4400 850 50  0001 C CNN
 F 3 "~" H 4400 850 50  0001 C CNN
 	1    4400 850
@@
 F 0 "D13" H 4950 645 50  0000 C CNN
 F 1 "GREEN" H 4950 736 50  0000 C CNN
-F 2 "" V 4950 850 50  0001 C CNN
+F 2 "LED_SMD:LED_0805_2012Metric" V 4950 850 50  0001 C CNN
 F 3 "~" V 4950 850 50  0001 C CNN
 	1    4950 850
@@
 F 0 "U16" H 13550 4915 50  0000 C CNN
 F 1 "5P49V6965" H 13550 4824 50  0000 C CNN
-F 2 "" H 13550 3650 50  0001 C CNN
+F 2 "Package_DFN_QFN:QFN-24-1EP_4x4mm_P0.5mm_EP2.7x2.7mm" H 13550 3650 50  0001 C CNN
 F 3 "" H 13550 3650 50  0001 C CNN
 	1    13550 3650
@@
 F 0 "FB2" H 9400 2354 50  0000 R CNN
 F 1 "200R@100MHz" H 9400 2445 50  0000 R CNN
-F 2 "" V 9430 2400 50  0001 C CNN
+F 2 "Inductor_SMD:L_0603_1608Metric" V 9430 2400 50  0001 C CNN
 F 3 "~" H 9500 2400 50  0001 C CNN
 	1    9500 2400
@@
 F 0 "C109" H 9592 2796 50  0000 L CNN
 F 1 "10µ" H 9592 2705 50  0000 L CNN
-F 2 "" H 9500 2750 50  0001 C CNN
+F 2 "Capacitor_SMD:C_0805_2012Metric" H 9500 2750 50  0001 C CNN
 F 3 "~" H 9500 2750 50  0001 C CNN
 	1    9500 2750
@@
 F 0 "C110" H 9942 2796 50  0000 L CNN
 F 1 "470n" H 9942 2705 50  0000 L CNN
-F 2 "" H 9850 2750 50  0001 C CNN
+F 2 "Capacitor_SMD:C_0402_1005Metric" H 9850 2750 50  0001 C CNN
 F 3 "~" H 9850 2750 50  0001 C CNN
 	1    9850 2750
@@
 F 0 "C112" H 10292 2796 50  0000 L CNN
 F 1 "470n" H 10292 2705 50  0000 L CNN
-F 2 "" H 10200 2750 50  0001 C CNN
+F 2 "Capacitor_SMD:C_0402_1005Metric" H 10200 2750 50  0001 C CNN
 F 3 "~" H 10200 2750 50  0001 C CNN
 	1    10200 2750
@@
 F 0 "C113" H 10642 2796 50  0000 L CNN
 F 1 "470n" H 10642 2705 50  0000 L CNN
-F 2 "" H 10550 2750 50  0001 C CNN
+F 2 "Capacitor_SMD:C_0402_1005Metric" H 10550 2750 50  0001 C CNN
 F 3 "~" H 10550 2750 50  0001 C CNN
 	1    10550 2750
@@
 F 0 "C114" H 10992 2796 50  0000 L CNN
 F 1 "470n" H 10992 2705 50  0000 L CNN
-F 2 "" H 10900 2750 50  0001 C CNN
+F 2 "Capacitor_SMD:C_0402_1005Metric" H 10900 2750 50  0001 C CNN
 F 3 "~" H 10900 2750 50  0001 C CNN
 	1    10900 2750
@@
 F 0 "R52" V 11004 2600 50  0000 C CNN
 F 1 "2.2" V 11095 2600 50  0000 C CNN
-F 2 "" H 11200 2600 50  0001 C CNN
+F 2 "Resistor_SMD:R_0402_1005Metric" H 11200 2600 50  0001 C CNN
 F 3 "~" H 11200 2600 50  0001 C CNN
 	1    11200 2600
@@
 F 0 "C116" H 11492 2796 50  0000 L CNN
 F 1 "470n" H 11492 2705 50  0000 L CNN
-F 2 "" H 11400 2750 50  0001 C CNN
+F 2 "Capacitor_SMD:C_0402_1005Metric" H 11400 2750 50  0001 C CNN
 F 3 "~" H 11400 2750 50  0001 C CNN
 	1    11400 2750
@@
 F 0 "C118" H 11842 2796 50  0000 L CNN
 F 1 "100n" H 11842 2705 50  0000 L CNN
-F 2 "" H 11750 2750 50  0001 C CNN
+F 2 "Capacitor_SMD:C_0402_1005Metric" H 11750 2750 50  0001 C CNN
 F 3 "~" H 11750 2750 50  0001 C CNN
 	1    11750 2750
@@
 F 0 "C117" H 11492 3646 50  0000 L CNN
 F 1 "DNP" H 11492 3555 50  0000 L CNN
-F 2 "" H 11400 3600 50  0001 C CNN
+F 2 "Capacitor_SMD:C_0402_1005Metric" H 11400 3600 50  0001 C CNN
 F 3 "~" H 11400 3600 50  0001 C CNN
 	1    11400 3600
@@
 F 0 "C115" H 10808 3554 50  0000 R CNN
 F 1 "DNP" H 10808 3645 50  0000 R CNN
-F 2 "" H 10900 3600 50  0001 C CNN
+F 2 "Capacitor_SMD:C_0402_1005Metric" H 10900 3600 50  0001 C CNN
 F 3 "~" H 10900 3600 50  0001 C CNN
 	1    10900 3600
@@
 F 0 "R49" H 9059 3696 50  0000 L CNN
 F 1 "DNP" H 9059 3605 50  0000 L CNN
-F 2 "" H 9000 3650 50  0001 C CNN
+F 2 "Resistor_SMD:R_0402_1005Metric" H 9000 3650 50  0001 C CNN
 F 3 "~" H 9000 3650 50  0001 C CNN
 	1    9000 3650
@@
 F 0 "R50" H 10459 4246 50  0000 L CNN
 F 1 "2.2k" H 10459 4155 50  0000 L CNN
-F 2 "" H 10400 4200 50  0001 C CNN
+F 2 "Resistor_SMD:R_0402_1005Metric" H 10400 4200 50  0001 C CNN
 F 3 "~" H 10400 4200 50  0001 C CNN
 	1    10400 4200
@@
 F 0 "R51" H 10809 4246 50  0000 L CNN
 F 1 "2.2k" H 10809 4155 50  0000 L CNN
-F 2 "" H 10750 4200 50  0001 C CNN
+F 2 "Resistor_SMD:R_0402_1005Metric" H 10750 4200 50  0001 C CNN
 F 3 "~" H 10750 4200 50  0001 C CNN
 	1    10750 4200
@@
 F 0 "R57" V 11904 3750 50  0000 C CNN
 F 1 "10k" V 11995 3750 50  0000 C CNN
-F 2 "" H 12100 3750 50  0001 C CNN
+F 2 "Resistor_SMD:R_0402_1005Metric" H 12100 3750 50  0001 C CNN
 F 3 "~" H 12100 3750 50  0001 C CNN
 	1    12100 3750
@@
 F 0 "R58" V 14854 3250 50  0000 C CNN
 F 1 "0R" V 14945 3250 50  0000 C CNN
-F 2 "" H 15050 3250 50  0001 C CNN
+F 2 "Resistor_SMD:R_0402_1005Metric" H 15050 3250 50  0001 C CNN
 F 3 "~" H 15050 3250 50  0001 C CNN
 	1    15050 3250
@@
 F 0 "C99" V 3100 7250 50  0000 C CNN
 F 1 "100n" V 2700 7250 50  0000 C CNN
-F 2 "" H 2900 7250 50  0001 C CNN
+F 2 "Capacitor_SMD:C_0402_1005Metric" H 2900 7250 50  0001 C CNN
 F 3 "~" H 2900 7250 50  0001 C CNN
 	1    2900 7250
@@
 F 0 "C100" V 3100 7350 50  0000 C CNN
 F 1 "100n" V 2700 7350 50  0000 C CNN
-F 2 "" H 2900 7350 50  0001 C CNN
+F 2 "Capacitor_SMD:C_0402_1005Metric" H 2900 7350 50  0001 C CNN
 F 3 "~" H 2900 7350 50  0001 C CNN
 	1    2900 7350
@@
 F 0 "C101" V 3100 8350 50  0000 C CNN
 F 1 "100n" V 2700 8350 50  0000 C CNN
-F 2 "" H 2900 8350 50  0001 C CNN
+F 2 "Capacitor_SMD:C_0402_1005Metric" H 2900 8350 50  0001 C CNN
 F 3 "~" H 2900 8350 50  0001 C CNN
 	1    2900 8350
@@
 F 0 "C102" V 3100 8450 50  0000 C CNN
 F 1 "100n" V 2700 8450 50  0000 C CNN
-F 2 "" H 2900 8450 50  0001 C CNN
+F 2 "Capacitor_SMD:C_0402_1005Metric" H 2900 8450 50  0001 C CNN
 F 3 "~" H 2900 8450 50  0001 C CNN
 	1    2900 8450
@@
 F 0 "FB3" V 10487 7150 50  0000 C CNN
 F 1 "200R@100MHz" V 10396 7150 50  0000 C CNN
-F 2 "" V 10180 7150 50  0001 C CNN
+F 2 "Inductor_SMD:L_0603_1608Metric" V 10180 7150 50  0001 C CNN
 F 3 "~" H 10250 7150 50  0001 C CNN
 	1    10250 7150
@@
 F 0 "C111" H 10042 7446 50  0000 L CNN
 F 1 "470n" H 10042 7355 50  0000 L CNN
-F 2 "" H 9950 7400 50  0001 C CNN
+F 2 "Capacitor_SMD:C_0402_1005Metric" H 9950 7400 50  0001 C CNN
 F 3 "~" H 9950 7400 50  0001 C CNN
 	1    9950 7400
@@
 F 0 "R53" V 11750 7150 50  0000 C CNN
 F 1 "0R" V 11950 7150 50  0000 C CNN
-F 2 "" H 11950 7150 50  0001 C CNN
+F 2 "Resistor_SMD:R_0805_2012Metric" H 11950 7150 50  0001 C CNN
 F 3 "~" H 11950 7150 50  0001 C CNN
 	1    11950 7150
@@
 F 0 "R54" V 11750 7250 50  0000 C CNN
 F 1 "DNP" V 11950 7250 50  0000 C CNN
-F 2 "" H 11950 7250 50  0001 C CNN
+F 2 "Resistor_SMD:R_0805_2012Metric" H 11950 7250 50  0001 C CNN
 F 3 "~" H 11950 7250 50  0001 C CNN
 	1    11950 7250
@@
 F 0 "R55" V 11750 7650 50  0000 C CNN
 F 1 "0R" V 11950 7650 50  0000 C CNN
-F 2 "" H 11950 7650 50  0001 C CNN
+F 2 "Resistor_SMD:R_0805_2012Metric" H 11950 7650 50  0001 C CNN
 F 3 "~" H 11950 7650 50  0001 C CNN
 	1    11950 7650
@@
 F 0 "R56" V 11750 7750 50  0000 C CNN
 F 1 "DNP" V 11950 7750 50  0000 C CNN
-F 2 "" H 11950 7750 50  0001 C CNN
+F 2 "Resistor_SMD:R_0805_2012Metric" H 11950 7750 50  0001 C CNN
 F 3 "~" H 11950 7750 50  0001 C CNN
 	1    11950 7750
@@
 F 0 "R47" V 3654 2250 50  0000 C CNN
 F 1 "1k" V 3745 2250 50  0000 C CNN
-F 2 "" H 3850 2250 50  0001 C CNN
+F 2 "Resistor_SMD:R_0402_1005Metric" H 3850 2250 50  0001 C CNN
 F 3 "~" H 3850 2250 50  0001 C CNN
 	1    3850 2250
@@
 F 0 "FB1" H 8250 2354 50  0000 R CNN
 F 1 "200R@100MHz" H 8250 2445 50  0000 R CNN
-F 2 "" V 8280 2400 50  0001 C CNN
+F 2 "Inductor_SMD:L_0603_1608Metric" V 8280 2400 50  0001 C CNN
 F 3 "~" H 8350 2400 50  0001 C CNN
 	1    8350 2400
@@
 F 0 "C107" H 8442 2796 50  0000 L CNN
 F 1 "10µ" H 8442 2705 50  0000 L CNN
-F 2 "" H 8350 2750 50  0001 C CNN
+F 2 "Capacitor_SMD:C_0805_2012Metric" H 8350 2750 50  0001 C CNN
 F 3 "~" H 8350 2750 50  0001 C CNN
 	1    8350 2750
@@
 F 0 "C108" H 8842 2796 50  0000 L CNN
 F 1 "470n" H 8842 2705 50  0000 L CNN
-F 2 "" H 8750 2750 50  0001 C CNN
+F 2 "Capacitor_SMD:C_0402_1005Metric" H 8750 2750 50  0001 C CNN
 F 3 "~" H 8750 2750 50  0001 C CNN
 	1    8750 2750

Commit message: hardware/mainboard: Assign more footprints
Signed-off-by: David Shah <dave@ds0.me>
Parts:
- DA1, DA2, DA3, DA4: footprint (none) -> Custom Parts:USON10
- JP1: footprint (none) -> Connector_PinHeader_2.54mm:PinHeader_1x03_P2.54mm_Vertical
- P3: footprint (none) -> Custom Parts:PCIe_EDGE_x4
- TP1: footprint (none) -> TestPoint:TestPoint_Pad_1.5x1.5mm
- TP2: value DCU1_CLK+ -> DCU1_CLK-; footprint (none) -> TestPoint:TestPoint_Pad_1.5x1.5mm
- U15: footprint (none) -> Custom Parts:CABGA756_27x27mm_p0.8mm
Changed lines of the file:
@@
 F 0 "P3" H 2400 3715 50  0000 C CNN
 F 1 "PCIe_x4_EDGE" H 2400 3624 50  0000 C CNN
-F 2 "" H 2400 2400 50  0001 C CNN
+F 2 "Custom Parts:PCIe_EDGE_x4" H 2400 2400 50  0001 C CNN
 F 3 "" H 2400 2400 50  0001 C CNN
 	1    2400 2350
@@
 F 0 "JP1" V 1246 5586 50  0000 L CNN
 F 1 "PRSNT" V 1155 5586 50  0000 L CNN
-F 2 "" H 1200 5500 50  0001 C CNN
+F 2 "Connector_PinHeader_2.54mm:PinHeader_1x03_P2.54mm_Vertical" H 1200 5500 50  0001 C CNN
 F 3 "~" H 1200 5500 50  0001 C CNN
 	1    1200 5500
@@
 F 0 "U15" H 13931 403 60  0000 L CNN
 F 1 "ECP5UM5G_85_CABGA756" H 13931 297 60  0000 L CNN
-F 2 "" H 13000 800 50  0001 C CNN
+F 2 "Custom Parts:CABGA756_27x27mm_p0.8mm" H 13000 800 50  0001 C CNN
 F 3 "" H 13000 800 50  0001 C CNN
 F 4 "ECP5UM5G_85" H 13150 750 60  0001 R CNN "manf#"
@@
 F 0 "DA3" H 6800 3087 60  0000 C CNN
 F 1 "TPD4E02B04" H 6800 2981 60  0000 C CNN
-F 2 "" H 6800 2300 60  0001 C CNN
+F 2 "Custom Parts:USON10" H 6800 2300 60  0001 C CNN
 F 3 "" H 6800 2300 60  0001 C CNN
 	1    6800 2300
@@
 F 0 "DA4" H 6800 4687 60  0000 C CNN
 F 1 "TPD4E02B04" H 6800 4581 60  0000 C CNN
-F 2 "" H 6800 3900 60  0001 C CNN
+F 2 "Custom Parts:USON10" H 6800 3900 60  0001 C CNN
 F 3 "" H 6800 3900 60  0001 C CNN
 	1    6800 3900
@@
 F 0 "DA1" H 5150 7937 60  0000 C CNN
 F 1 "TPD4E02B04" H 5150 7831 60  0000 C CNN
-F 2 "" H 5150 7150 60  0001 C CNN
+F 2 "Custom Parts:USON10" H 5150 7150 60  0001 C CNN
 F 3 "" H 5150 7150 60  0001 C CNN
 	1    5150 7150
@@
 F 0 "DA2" H 5150 9537 60  0000 C CNN
 F 1 "TPD4E02B04" H 5150 9431 60  0000 C CNN
-F 2 "" H 5150 8750 60  0001 C CNN
+F 2 "Custom Parts:USON10" H 5150 8750 60  0001 C CNN
 F 3 "" H 5150 8750 60  0001 C CNN
 	1    5150 8750
@@
 F 0 "U15" H 13931 8503 60  0000 L CNN
 F 1 "ECP5UM5G_85_CABGA756" H 13931 8397 60  0000 L CNN
-F 2 "" H 13000 8900 50  0001 C CNN
+F 2 "Custom Parts:CABGA756_27x27mm_p0.8mm" H 13000 8900 50  0001 C CNN
 F 3 "" H 13000 8900 50  0001 C CNN
 F 4 "ECP5UM5G_85" H 13150 8850 60  0001 R CNN "manf#"
@@
 F 0 "TP1" V 12050 8050 50  0000 C CNN
 F 1 "DCU1_CLK+" V 12050 7750 50  0000 C CNN
-F 2 "" H 12250 7350 50  0001 C CNN
+F 2 "TestPoint:TestPoint_Pad_1.5x1.5mm" H 12250 7350 50  0001 C CNN
 F 3 "~" H 12250 7350 50  0001 C CNN
 	1    12050 7350
@@
 P 12050 7850
 F 0 "TP2" V 12050 8550 50  0000 C CNN
-F 1 "DCU1_CLK+" V 12050 8250 50  0000 C CNN
-F 2 "" H 12250 7850 50  0001 C CNN
+F 1 "DCU1_CLK-" V 12050 8250 50  0000 C CNN
+F 2 "TestPoint:TestPoint_Pad_1.5x1.5mm" H 12250 7850 50  0001 C CNN
 F 3 "~" H 12250 7850 50  0001 C CNN
 	1    12050 7850

Commit message: hardware: Add SATA connector footprint
Signed-off-by: David Shah <dave@ds0.me>
Connections:
- net GND: now also P1.S, P2.S
Changed lines of the file:
@@
 L power:GND #PWR087
 U 1 1 5C4AE0D7
-P 2250 9100
-F 0 "#PWR087" H 2250 8850 50  0001 C CNN
-F 1 "GND" H 2255 8927 50  0000 C CNN
-F 2 "" H 2250 9100 50  0001 C CNN
-F 3 "" H 2250 9100 50  0001 C CNN
-	1    2250 9100
+P 2250 9300
+F 0 "#PWR087" H 2250 9050 50  0001 C CNN
+F 1 "GND" H 2255 9127 50  0000 C CNN
+F 2 "" H 2250 9300 50  0001 C CNN
+F 3 "" H 2250 9300 50  0001 C CNN
+	1    2250 9300
 	-1   0    0    -1
 $EndComp
 Wire Wire Line
-	2250 9100 2250 8850
+	2250 9300 2250 9200
 Wire Wire Line
 	2250 7150 2100 7150
@@
 Connection ~ 2250 8250
 Wire Wire Line
-	2250 8250 2250 7750
+	2250 8250 2250 8050
 Wire Wire Line
 	2100 8550 2250 8550
@@
 Wire Wire Line
 	9950 6900 9950 7150
+Wire Wire Line
+	1650 7950 1650 8050
+Wire Wire Line
+	1650 8050 2250 8050
+Connection ~ 2250 8050
+Wire Wire Line
+	2250 8050 2250 7750
+Wire Wire Line
+	1650 9050 1650 9200
+Wire Wire Line
+	1650 9200 2250 9200
+Connection ~ 2250 9200
+Wire Wire Line
+	2250 9200 2250 8850
 $EndSCHEMATC

Commit message: hardware: Creating and assigning some misc footprints
Signed-off-by: David Shah <dave@ds0.me>
Parts:
- P1, P2: footprint (none) -> Custom Parts:Molex_SATA_047080-4001
- U14: value XL_XO_LVDS -> XUL535150.000JS6I8; footprint (none) -> Custom Parts:OSC_IDT_XU_5x3.2mm
Changed lines of the file:
@@
 F 0 "P1" H 1928 7496 50  0000 L CNN
 F 1 "SATA" H 1928 7405 50  0000 L CNN
-F 2 "" H 1650 7450 50  0001 C CNN
+F 2 "Custom Parts:Molex_SATA_047080-4001" H 1650 7450 50  0001 C CNN
 F 3 "" H 1650 7450 50  0001 C CNN
 	1    1650 7450
@@
 F 0 "P2" H 1928 8596 50  0000 L CNN
 F 1 "SATA" H 1928 8505 50  0000 L CNN
-F 2 "" H 1650 8550 50  0001 C CNN
+F 2 "Custom Parts:Molex_SATA_047080-4001" H 1650 8550 50  0001 C CNN
 F 3 "" H 1650 8550 50  0001 C CNN
 	1    1650 8550
@@
 P 8600 7350
 F 0 "U14" H 8600 7815 50  0000 C CNN
-F 1 "XL_XO_LVDS" H 8600 7724 50  0000 C CNN
-F 2 "" H 8600 7350 50  0001 C CNN
+F 1 " XUL535150.000JS6I8" H 8600 7724 50  0000 C CNN
+F 2 "Custom Parts:OSC_IDT_XU_5x3.2mm" H 8600 7350 50  0001 C CNN
 F 3 "" H 8600 7350 50  0001 C CNN
 	1    8600 7350

Commit message: hardware/mainboard: More footprint assignment, other small tweaks
Signed-off-by: David Shah <dave@ds0.me>
Parts:
- Y1: footprint (none) -> Custom Parts:Crystal_Epsom_TSX-3225
Changed lines of the file:
@@
 F 0 "Y1" H 11150 3718 50  0000 C CNN
 F 1 "25MHz" H 11150 3627 50  0000 C CNN
-F 2 "" H 11150 3450 50  0001 C CNN
+F 2 "Custom Parts:Crystal_Epsom_TSX-3225" H 11150 3450 50  0001 C CNN
 F 3 "~" H 11150 3450 50  0001 C CNN
 	1    11150 3450
