File: hardware/ecp5_mainboard/serdes.sch (KiCad schematic (older format))
At the start: 50 parts, among them P1 SATA, P2 SATA, P3 PCIe_x4_EDGE, U14 XUL535150.000JS6I8, U15 ECP5UM5G_85_CABGA756, U16 5P49V6965, Y1 25MHz

Commit message: hardware/mainboard: Switching from SATA to m.2 connector for second DCU
Signed-off-by: David Shah <dave@ds0.me>
Parts:
- removed C111: 470n, Capacitor_SMD:C_0402_1005Metric, symbol Device:C_Small
- removed FB3: 200R@100MHz, Inductor_SMD:L_0603_1608Metric, symbol Device:Ferrite_Bead_Small
- removed P1, P2: SATA, Custom Parts:Molex_SATA_047080-4001, symbol eco_connectors:SATA
- removed R53, R55: 0R, Resistor_SMD:R_0805_2012Metric, symbol Device:R_Small
- removed R54, R56: DNP, Resistor_SMD:R_0805_2012Metric, symbol Device:R_Small
- removed TP1: DCU1_CLK+, TestPoint:TestPoint_Pad_1.5x1.5mm, symbol Connector:TestPoint
- removed TP2: DCU1_CLK-, TestPoint:TestPoint_Pad_1.5x1.5mm, symbol Connector:TestPoint
- removed U14: XUL535150.000JS6I8, Custom Parts:OSC_IDT_XU_5x3.2mm, symbol eco_glue:XL_XO_LVDS
- added P?: M2_SOCKET_E, symbol eco_connectors:M2_SOCKET_E
- added R?: 10k, symbol Device:R_Small
- added U?: CBTL02043A, symbol eco_glue:CBTL02043A
Connections:
- net labels added: CLKREFO+, CLKREFO-, M2_CTS, M2_REFCLK+, M2_REFCLK-, M2_RTS, M2_RX0+, M2_RX0-, M2_RX1+, M2_RX1-, M2_SDIO_CLK, M2_SDIO_CMD, M2_SDIO_D0, M2_SDIO_D1, M2_SDIO_D2, M2_SDIO_D3, M2_TXD
- net labels removed: CLK150M+, CLK150M-, SATA0_A+, SATA0_A-, SATA1_A+, SATA1_A-
- wire segments 334 -> 347
- no-connect marks 25 -> 52
Other:
- moved on the sheet: C100, C101, C102, C99, DA1, DA2

Commit message: hardware/mainboard: Add and place M.2 connector footprint
Signed-off-by: David Shah <davey1576@gmail.com>
Parts:
- added C111: 470n, Capacitor_SMD:C_0402_1005Metric, symbol Device:C_Small
- added R53, R54: 10k, Resistor_SMD:R_0402_1005Metric, symbol Device:R_Small
- P1: renamed from P?; footprint (none) -> Custom Parts:2199230-4
- R1: renamed from R?; footprint (none) -> Resistor_SMD:R_0402_1005Metric
- U11: renamed from U?; footprint (none) -> Package_DFN_QFN:WQFN-20-1EP_2.5x4.5mm_P0.5mm_EP1x2.9mm
Connections:
- net +3V3: now also U11.1 (Vdd), U11.10 (Vdd), U11.6 (Vdd), C111.1
- net GND: now also P1.M, U11.11 (GND), U11.20 (GND), U11.21 (GND), U11.5 (GND), C111.2, R53.1, R54.2
- net at U11.2 (XSD): now also R54.1
- net M2_CLKSEL: now reaches U11.9 (SEL)
- net M2_CLKSEL: now also R53.2
Changed lines of the file:
@@
 1V8_C
 $Comp
-L eco_glue:CBTL02043A U?
+L eco_glue:CBTL02043A U11
 U 1 1 652CFC30
 P 13550 6500
-F 0 "U?" H 13550 7865 50  0000 C CNN
+F 0 "U11" H 13550 7865 50  0000 C CNN
 F 1 "CBTL02043A" H 13550 7774 50  0000 C CNN
-F 2 "" H 13575 6500 50  0001 C CNN
+F 2 "Package_DFN_QFN:WQFN-20-1EP_2.5x4.5mm_P0.5mm_EP1x2.9mm" H 13575 6500 50  0001 C CNN
 F 3 "" H 13575 6500 50  0001 C CNN
 	1    13550 6500
@@
 CLKREFO-
 $Comp
-L eco_connectors:M2_SOCKET_E P?
+L eco_connectors:M2_SOCKET_E P1
 U 1 1 655141E5
 P 8000 7500
-F 0 "P?" H 8000 8965 50  0000 C CNN
+F 0 "P1" H 8000 8965 50  0000 C CNN
 F 1 "M2_SOCKET_E" H 8000 8874 50  0000 C CNN
-F 2 "" H 8000 8050 50  0001 C CNN
+F 2 "Custom Parts:2199230-4" H 8000 8050 50  0001 C CNN
 F 3 "" H 8000 8050 50  0001 C CNN
 	1    8000 7500
@@
 	7000 6300 7000 6600
 $Comp
-L power:GND #PWR?
+L power:GND #PWR087
 U 1 1 655A5C9A
 P 7000 10000
-F 0 "#PWR?" H 7000 9750 50  0001 C CNN
+F 0 "#PWR087" H 7000 9750 50  0001 C CNN
 F 1 "GND" H 7005 9827 50  0000 C CNN
 F 2 "" H 7000 10000 50  0001 C CNN
@@
 	7000 9400 7000 9700
 $Comp
-L power:GND #PWR?
+L power:GND #PWR094
 U 1 1 657AD7C1
 P 9000 10000
-F 0 "#PWR?" H 9000 9750 50  0001 C CNN
+F 0 "#PWR094" H 9000 9750 50  0001 C CNN
 F 1 "GND" H 9005 9827 50  0000 C CNN
 F 2 "" H 9000 10000 50  0001 C CNN
@@
 	9100 9600 9100 9500
 $Comp
-L power:+3V3 #PWR?
+L power:+3V3 #PWR099
 U 1 1 657EF089
 P 9100 6000
-F 0 "#PWR?" H 9100 5850 50  0001 C CNN
+F 0 "#PWR099" H 9100 5850 50  0001 C CNN
 F 1 "+3V3" H 9115 6173 50  0000 C CNN
 F 2 "" H 9100 6000 50  0001 C CNN
@@
 	8900 8500 9250 8500
 $Comp
-L Device:R_Small R?
+L Device:R_Small R1
 U 1 1 65CACA89
 P 9350 8500
-F 0 "R?" V 9154 8500 50  0000 C CNN
+F 0 "R1" V 9154 8500 50  0000 C CNN
 F 1 "10k" V 9245 8500 50  0000 C CNN
-F 2 "" H 9350 8500 50  0001 C CNN
+F 2 "Resistor_SMD:R_0402_1005Metric" H 9350 8500 50  0001 C CNN
 F 3 "~" H 9350 8500 50  0001 C CNN
 	1    9350 8500
@@
 $EndComp
 $Comp
-L power:+3V3 #PWR?
+L power:+3V3 #PWR0101
 U 1 1 65CACBDE
 P 9550 8500
-F 0 "#PWR?" H 9550 8350 50  0001 C CNN
+F 0 "#PWR0101" H 9550 8350 50  0001 C CNN
 F 1 "+3V3" V 9565 8628 50  0000 L CNN
 F 2 "" H 9550 8500 50  0001 C CNN
@@
 Wire Wire Line
 	8900 7700 9200 7700
+$Comp
+L power:GND #PWR0207
+U 1 1 5C78E250
+P 12700 7250
+F 0 "#PWR0207" H 12700 7000 50  0001 C CNN
+F 1 "GND" H 12705 7077 50  0000 C CNN
+F 2 "" H 12700 7250 50  0001 C CNN
+F 3 "" H 12700 7250 50  0001 C CNN
+	1    12700 7250
+	1    0    0    -1
+$EndComp
+Wire Wire Line
+	12850 6850 12700 6850
+Wire Wire Line
+	12700 6850 12700 6950
+Wire Wire Line
+	12850 6950 12700 6950
+Connection ~ 12700 6950
+Wire Wire Line
+	12700 6950 12700 7050
+Wire Wire Line
+	12700 7050 12850 7050
+Connection ~ 12700 7050
+Wire Wire Line
+	12700 7050 12700 7150
+$Comp
+L Device:R_Small R54
+U 1 1 5C83C987
+P 12650 6550
+F 0 "R54" V 12454 6550 50  0000 C CNN
+F 1 "10k" V 12545 6550 50  0000 C CNN
+F 2 "Resistor_SMD:R_0402_1005Metric" H 12650 6550 50  0001 C CNN
+F 3 "~" H 12650 6550 50  0001 C CNN
+	1    12650 6550
+	0    1    1    0
+$EndComp
+Wire Wire Line
+	12750 6550 12850 6550
+$Comp
+L power:GND #PWR0254
+U 1 1 5C8603EA
+P 12400 6550
+F 0 "#PWR0254" H 12400 6300 50  0001 C CNN
+F 1 "GND" V 12405 6422 50  0000 R CNN
+F 2 "" H 12400 6550 50  0001 C CNN
+F 3 "" H 12400 6550 50  0001 C CNN
+	1    12400 6550
+	0    1    1    0
+$EndComp
+Wire Wire Line
+	12550 6550 12400 6550
+Text GLabel 12150 6650 0    50   Input ~ 0
+M2_CLKSEL
+Wire Wire Line
+	12850 6650 12450 6650
+$Comp
+L Device:R_Small R53
+U 1 1 5C8F7D85
+P 12450 6850
+F 0 "R53" H 12391 6804 50  0000 R CNN
+F 1 "10k" H 12391 6895 50  0000 R CNN
+F 2 "Resistor_SMD:R_0402_1005Metric" H 12450 6850 50  0001 C CNN
+F 3 "~" H 12450 6850 50  0001 C CNN
+	1    12450 6850
+	-1   0    0    1
+$EndComp
+Wire Wire Line
+	12700 7050 12450 7050
+Wire Wire Line
+	12450 7050 12450 6950
+Wire Wire Line
+	12450 6750 12450 6650
+Connection ~ 12450 6650
+Wire Wire Line
+	12450 6650 12150 6650
+$Comp
+L power:+3V3 #PWR0255
+U 1 1 5C9FA52C
+P 12650 5250
+F 0 "#PWR0255" H 12650 5100 50  0001 C CNN
+F 1 "+3V3" H 12665 5423 50  0000 C CNN
+F 2 "" H 12650 5250 50  0001 C CNN
+F 3 "" H 12650 5250 50  0001 C CNN
+	1    12650 5250
+	1    0    0    -1
+$EndComp
+Wire Wire Line
+	12850 5500 12650 5500
+Wire Wire Line
+	12650 5500 12650 5400
+Wire Wire Line
+	12850 5400 12650 5400
+Connection ~ 12650 5400
+Wire Wire Line
+	12650 5400 12650 5300
+$Comp
+L Device:C_Small C111
+U 1 1 5CA4427D
+P 12400 5400
+F 0 "C111" V 12171 5400 50  0000 C CNN
+F 1 "470n" V 12262 5400 50  0000 C CNN
+F 2 "Capacitor_SMD:C_0402_1005Metric" H 12400 5400 50  0001 C CNN
+F 3 "~" H 12400 5400 50  0001 C CNN
+	1    12400 5400
+	0    1    1    0
+$EndComp
+Wire Wire Line
+	12500 5400 12650 5400
+$Comp
+L power:GND #PWR0256
+U 1 1 5CA69A18
+P 12100 5400
+F 0 "#PWR0256" H 12100 5150 50  0001 C CNN
+F 1 "GND" V 12105 5272 50  0000 R CNN
+F 2 "" H 12100 5400 50  0001 C CNN
+F 3 "" H 12100 5400 50  0001 C CNN
+	1    12100 5400
+	0    1    1    0
+$EndComp
+Wire Wire Line
+	12100 5400 12300 5400
+Wire Wire Line
+	12700 7150 12850 7150
+Connection ~ 12700 7150
+Wire Wire Line
+	12700 7150 12700 7250
+Wire Wire Line
+	12850 5300 12650 5300
+Connection ~ 12650 5300
+Wire Wire Line
+	12650 5300 12650 5250
+$Comp
+L power:GND #PWR0257
+U 1 1 5CC6769B
+P 8000 10100
+F 0 "#PWR0257" H 8000 9850 50  0001 C CNN
+F 1 "GND" H 8005 9927 50  0000 C CNN
+F 2 "" H 8000 10100 50  0001 C CNN
+F 3 "" H 8000 10100 50  0001 C CNN
+	1    8000 10100
+	1    0    0    -1
+$EndComp
+Wire Wire Line
+	8000 10100 8000 10000
 $EndSCHEMATC

Commit message: hardware/mainboard: Repositioning to fit in M.2
Signed-off-by: David Shah <davey1576@gmail.com>
Parts:
- added C?: 470n, Capacitor_SMD:C_0402_1005Metric, symbol Device:C_Small
Connections:
- net +3V3: now also C?.1
- net GND: now also C?.2
Other:
- moved on the sheet: C111
Changed lines of the file:
@@
 Wire Wire Line
 	12650 5500 12650 5400
-Wire Wire Line
-	12850 5400 12650 5400
-Connection ~ 12650 5400
-Wire Wire Line
-	12650 5400 12650 5300
+Connection ~ 12650 5300
 $Comp
 L Device:C_Small C111
 U 1 1 5CA4427D
-P 12400 5400
-F 0 "C111" V 12171 5400 50  0000 C CNN
-F 1 "470n" V 12262 5400 50  0000 C CNN
-F 2 "Capacitor_SMD:C_0402_1005Metric" H 12400 5400 50  0001 C CNN
-F 3 "~" H 12400 5400 50  0001 C CNN
-	1    12400 5400
+P 12450 5300
+F 0 "C111" V 12221 5300 50  0000 C CNN
+F 1 "470n" V 12312 5300 50  0000 C CNN
+F 2 "Capacitor_SMD:C_0402_1005Metric" H 12450 5300 50  0001 C CNN
+F 3 "~" H 12450 5300 50  0001 C CNN
+	1    12450 5300
 	0    1    1    0
 $EndComp
 Wire Wire Line
-	12500 5400 12650 5400
+	12550 5300 12650 5300
 $Comp
 L power:GND #PWR0256
 U 1 1 5CA69A18
-P 12100 5400
-F 0 "#PWR0256" H 12100 5150 50  0001 C CNN
-F 1 "GND" V 12105 5272 50  0000 R CNN
-F 2 "" H 12100 5400 50  0001 C CNN
-F 3 "" H 12100 5400 50  0001 C CNN
-	1    12100 5400
+P 11800 5300
+F 0 "#PWR0256" H 11800 5050 50  0001 C CNN
+F 1 "GND" V 11805 5172 50  0000 R CNN
+F 2 "" H 11800 5300 50  0001 C CNN
+F 3 "" H 11800 5300 50  0001 C CNN
+	1    11800 5300
 	0    1    1    0
 $EndComp
 Wire Wire Line
-	12100 5400 12300 5400
+	11800 5300 12200 5300
 Wire Wire Line
 	12700 7150 12850 7150
@@
 Wire Wire Line
 	12850 5300 12650 5300
-Connection ~ 12650 5300
 Wire Wire Line
 	12650 5300 12650 5250
@@
 Wire Wire Line
 	8000 10100 8000 10000
+Wire Wire Line
+	12650 5400 12850 5400
+Connection ~ 12650 5400
+Wire Wire Line
+	12650 5400 12650 5300
+$Comp
+L Device:C_Small C?
+U 1 1 5C836F58
+P 12450 5500
+F 0 "C?" V 12221 5500 50  0000 C CNN
+F 1 "470n" V 12312 5500 50  0000 C CNN
+F 2 "Capacitor_SMD:C_0402_1005Metric" H 12450 5500 50  0001 C CNN
+F 3 "~" H 12450 5500 50  0001 C CNN
+	1    12450 5500
+	0    1    1    0
+$EndComp
+Wire Wire Line
+	12550 5500 12650 5500
+Connection ~ 12650 5500
+Wire Wire Line
+	12350 5500 12200 5500
+Wire Wire Line
+	12200 5500 12200 5300
+Connection ~ 12200 5300
+Wire Wire Line
+	12200 5300 12350 5300
 $EndSCHEMATC

Commit message: hardware/mainboard: Tweak layout around M.2 and add standoffs for 30&42mm cards
Signed-off-by: David Shah <davey1576@gmail.com>
Parts:
- added J14, J8: 9774025151R, Custom Parts:9774025151R, symbol Connector:Conn_01x01_Male
- gave numbers to parts that had none: 1
Connections:
- net GND: now also J14.1 (Pin_1), J8.1 (Pin_1)
Other:
- note added: "M.2 standoffs"
Changed lines of the file:
@@
 	12650 5400 12650 5300
 $Comp
-L Device:C_Small C?
+L Device:C_Small C257
 U 1 1 5C836F58
 P 12450 5500
-F 0 "C?" V 12221 5500 50  0000 C CNN
+F 0 "C257" V 12221 5500 50  0000 C CNN
 F 1 "470n" V 12312 5500 50  0000 C CNN
 F 2 "Capacitor_SMD:C_0402_1005Metric" H 12450 5500 50  0001 C CNN
@@
 Wire Wire Line
 	12200 5300 12350 5300
+$Comp
+L power:GND #PWR0258
+U 1 1 5C702223
+P 6250 10750
+F 0 "#PWR0258" H 6250 10500 50  0001 C CNN
+F 1 "GND" H 6255 10577 50  0000 C CNN
+F 2 "" H 6250 10750 50  0001 C CNN
+F 3 "" H 6250 10750 50  0001 C CNN
+	1    6250 10750
+	0    1    1    0
+$EndComp
+$Comp
+L Connector:Conn_01x01_Male J8
+U 1 1 5C7023EB
+P 6600 10650
+F 0 "J8" H 6573 10580 50  0000 R CNN
+F 1 "9774025151R" H 6573 10671 50  0000 R CNN
+F 2 "Custom Parts:9774025151R" H 6600 10650 50  0001 C CNN
+F 3 "~" H 6600 10650 50  0001 C CNN
+	1    6600 10650
+	-1   0    0    1
+$EndComp
+Wire Wire Line
+	6250 10750 6300 10750
+Wire Wire Line
+	6300 10750 6300 10650
+Wire Wire Line
+	6300 10650 6400 10650
+$Comp
+L Connector:Conn_01x01_Male J14
+U 1 1 5C751C23
+P 6600 10850
+F 0 "J14" H 6573 10780 50  0000 R CNN
+F 1 "9774025151R" H 6573 10871 50  0000 R CNN
+F 2 "Custom Parts:9774025151R" H 6600 10850 50  0001 C CNN
+F 3 "~" H 6600 10850 50  0001 C CNN
+	1    6600 10850
+	-1   0    0    1
+$EndComp
+Wire Wire Line
+	6400 10850 6300 10850
+Wire Wire Line
+	6300 10850 6300 10750
+Connection ~ 6300 10750
+Text Notes 6300 11000 0    50   ~ 0
+M.2 standoffs
 $EndSCHEMATC

Commit message: hardware/mainboard: Clock & M.2 routing
Signed-off-by: David Shah <davey1576@gmail.com>
Connections:
- net M2_TXD: no longer P1.32 (UART_RXD)
- new net M2_RXD: P1.32 (UART_RXD)
Changed lines of the file:
@@
 M2_TXD
 Text GLabel 9200 7500 2    50   Output ~ 0
-M2_TXD
+M2_RXD
 Wire Wire Line
 	9200 7500 8900 7500

Commit message: hardware/mainboard: Misc routing
Signed-off-by: David Shah <davey1576@gmail.com>
Parts:
- added C259: 470n, Capacitor_SMD:C_0402_1005Metric, symbol Device:C_Small
Connections:
- net 1V8_C: now also C259.1
- net GND: now also C259.2
Changed lines of the file:
@@
 Text Notes 6300 11000 0    50   ~ 0
 M.2 standoffs
+$Comp
+L Device:C_Small C259
+U 1 1 5C9FD15E
+P 9100 2750
+F 0 "C259" H 9192 2796 50  0000 L CNN
+F 1 "470n" H 9192 2705 50  0000 L CNN
+F 2 "Capacitor_SMD:C_0402_1005Metric" H 9100 2750 50  0001 C CNN
+F 3 "~" H 9100 2750 50  0001 C CNN
+	1    9100 2750
+	1    0    0    -1
+$EndComp
+Wire Wire Line
+	8750 2600 9100 2600
+Wire Wire Line
+	9100 2600 9100 2650
+Connection ~ 8750 2600
+Wire Wire Line
+	9100 2850 9100 2950
+Wire Wire Line
+	9100 2950 8750 2950
 $EndSCHEMATC
