File: hardware/ecp5_mainboard/fpga_io.sch (KiCad schematic (older format))
At the start: 14 parts

Commit message: hardware/mainboard: Connecting more FPGA IO
Signed-off-by: David Shah <dave@ds0.me>
Parts:
- added C? (x8): 470n, symbol Device:C_Small
- added C? (x2): 4.7µ, symbol Device:C_Small
- added U? (x2): ECP5UM5G_85_CABGA756, symbol ECP5UM5G:ECP5UM5G_85_CABGA756
- added U?: XL_XO_LVDS, symbol eco_glue:XL_XO_LVDS
Connections:
- net CLK100+: now also U?.4 (OUT+), U?.B29 (PT121A); no longer U?.C28 (PR11A)
- net CLK100-: now also U?.5 (OUT-), U?.B30 (PT121B); no longer U?.D28 (PR11B)
- net GND: now also C?.2, C?.2, C?.2, C?.2, C?.2, C?.2, C?.2, C?.2, C?.2, C?.2, U?.3 (GND)
- new net +3V3: C?.1, C?.1, C?.1, C?.1, C?.1, C?.1, C?.1, C?.1, C?.1, C?.1, U?.6 (Vdd), U?.K12 (VCCIO0), U?.K14 (VCCIO0), U?.K15 (VCCIO0), U?.K16 (VCCIO0), U?.K17 (VCCIO1), U?.K18 (VCCIO1), U?.K19 (VCCIO1), U?.K21 (VCCIO1)
- new net CLK_SCL: U?.A22 (PT87A)
- new net CLK_SDA: U?.C22 (PT89A)
- new net DVI_CLK: U?.F8 (PT15A)
- new net DVI_D0: U?.F14 (PT45A)
- new net DVI_D1: U?.A13 (PT42B)
- new net DVI_D10: U?.A10 (PT31B)
- new net DVI_D11: U?.F11 (PT33A)
- new net DVI_D12: U?.B10 (PT31A)
- new net DVI_D13: U?.C10 (PT29B)
- new net DVI_D14: U?.E10 (PT27B)
- new net DVI_D15: U?.D10 (PT29A)
- new net DVI_D16: U?.F10 (PT27A)
- new net DVI_D17: U?.A9 (PT24B)
- new net DVI_D18: U?.D9 (PT22B)
- new net DVI_D19: U?.C9 (PT24A)
- new net DVI_D2: U?.D13 (PT40B)
- new net DVI_D20: U?.F9 (PT22A)
- new net DVI_D21: U?.A8 (PT20B)
- new net DVI_D22: U?.C8 (PT18B)
- new net DVI_D23: U?.B8 (PT20A)
- new net DVI_D3: U?.C13 (PT42A)
- new net DVI_D4: U?.F13 (PT40A)
- new net DVI_D5: U?.A11 (PT38B)
- new net DVI_D6: U?.C11 (PT36B)
- new net DVI_D7: U?.B11 (PT38A)
- new net DVI_D8: U?.D11 (PT36A)
- new net DVI_D9: U?.E11 (PT33B)
- new net DVI_DE: U?.D8 (PT18A)
- new net DVI_HSYNC: U?.A7 (PT13B)
- new net DVI_SCL: U?.C7 (PT11B)
- new net DVI_SDA: U?.B7 (PT13A)
- new net DVI_VSYNC: U?.E8 (PT15B)
- new net ETH_INT_N: U?.B14 (PT49A)
- new net ETH_MDC: U?.D17 (PT65B)
- new net ETH_MDIO: U?.B17 (PT63B)
- new net ETH_~RESET: U?.C14 (PT47B)
- new net FABRIC_REFCLK: U?.E17 (PT69A)
- new net LED0: U?.A5 (PT9B)
- new net LED1: U?.D7 (PT11A)
- new net LED10: U?.A28 (PT116A)
- new net LED11: U?.C26 (PT114A)
- new net LED2: U?.A4 (PT9A)
- new net LED3: U?.A3 (PT6B)
- new net LED4: U?.B4 (PT4B)
- new net LED5: U?.A2 (PT6A)
- new net LED6: U?.B3 (PT4A)
- new net LED7: U?.A30 (PT119A)
- new net LED8: U?.A29 (PT116B)
- new net LED9: U?.D26 (PT114B)
- new net PCIe_~WAKE: U?.A23 (PT94A)
- new net RGMII_REF_CLK: U?.A17 (PT63A)
- new net RGMII_RXD0: U?.C15 (PT54A)
- new net RGMII_RXD1: U?.D15 (PT51B)
- new net RGMII_RXD2: U?.A14 (PT49B)
- new net RGMII_RXD3: U?.F15 (PT51A)
- new net RGMII_RX_CLK: U?.C17 (PT65A)
- new net RGMII_RX_DV: U?.F16 (PT56A)
- new net RGMII_TXD0: U?.A16 (PT60B)
- new net RGMII_TXD1: U?.C16 (PT58B)
- new net RGMII_TXD2: U?.B16 (PT60A)
- new net RGMII_TXD3: U?.D16 (PT58A)
- new net RGMII_TX_CLK: U?.E16 (PT56B)
- new net RGMII_TX_EN: U?.A15 (PT54B)
- new net ULPI_CLKO: U?.A18 (PT71A)
- new net ULPI_D0: U?.F18 (PT74B)
- new net ULPI_D1: U?.B19 (PT76B)
- new net ULPI_D2: U?.C19 (PT78A)
- new net ULPI_D3: U?.E19 (PT80A)
- new net ULPI_D4: U?.D19 (PT78B)
- new net ULPI_D5: U?.F19 (PT80B)
- new net ULPI_D6: U?.A20 (PT83A)
- new net ULPI_D7: U?.D20 (PT85A)
- new net ULPI_DIR: U?.D18 (PT74A)
- new net ULPI_NXT: U?.A19 (PT76A)
- new net ULPI_RESET: U?.F17 (PT69B)
- new net ULPI_STP: U?.C18 (PT71B)
- new net ~PERST: U?.D22 (PT89B)
- no-connect marks 1 -> 3

Commit message: hardware/mainboard: Pin plan external IO FFCs
Signed-off-by: David Shah <dave@ds0.me>
Parts:
- added J?: EXT0, symbol Connector_Generic:Conn_01x40
- added J? (x3): EXT1, symbol Connector_Generic:Conn_01x40
- added U? (x2): ECP5UM5G_85_CABGA756, symbol ECP5UM5G:ECP5UM5G_85_CABGA756
Connections:
- net GND: now also J?.11 (Pin_11), J?.11 (Pin_11), J?.11 (Pin_11), J?.11 (Pin_11), J?.14 (Pin_14), J?.14 (Pin_14), J?.14 (Pin_14), J?.14 (Pin_14), J?.17 (Pin_17), J?.17 (Pin_17), J?.17 (Pin_17), J?.17 (Pin_17), J?.20 (Pin_20), J?.20 (Pin_20), J?.20 (Pin_20), J?.20 (Pin_20), J?.23 (Pin_23), J?.23 (Pin_23), J?.23 (Pin_23), J?.23 (Pin_23), J?.26 (Pin_26), J?.26 (Pin_26), J?.26 (Pin_26), J?.26 (Pin_26), J?.29 (Pin_29), J?.29 (Pin_29), J?.29 (Pin_29), J?.29 (Pin_29), J?.32 (Pin_32), J?.32 (Pin_32), J?.32 (Pin_32), J?.32 (Pin_32), J?.35 (Pin_35), J?.35 (Pin_35), J?.35 (Pin_35), J?.35 (Pin_35), J?.5 (Pin_5), J?.5 (Pin_5), J?.5 (Pin_5), J?.5 (Pin_5), J?.8 (Pin_8), J?.8 (Pin_8), J?.8 (Pin_8), J?.8 (Pin_8)
- new net EXT0_0+: J?.3 (Pin_3), U?.P5 (PL47A)
- new net EXT0_0-: J?.4 (Pin_4), U?.P4 (PL47B)
- new net EXT0_1+: J?.6 (Pin_6), U?.R7 (PL47C)
- new net EXT0_1-: J?.7 (Pin_7), U?.T7 (PL47D)
- new net EXT0_10+: J?.33 (Pin_33), U?.N1 (PL62A)
- new net EXT0_10-: J?.34 (Pin_34), U?.P1 (PL62B)
- new net EXT0_11+: J?.36 (Pin_36), U?.U2 (PL62C)
- new net EXT0_11-: J?.37 (Pin_37), U?.U3 (PL62D)
- new net EXT0_2+: J?.9 (Pin_9), U?.R6 (PL50A)
- new net EXT0_2-: J?.10 (Pin_10), U?.T6 (PL50B)
- new net EXT0_3+: J?.12 (Pin_12), U?.U6 (PL50C)
- new net EXT0_3-: J?.13 (Pin_13), U?.U7 (PL50D)
- new net EXT0_4+: J?.15 (Pin_15), U?.R4 (PL53A)
- new net EXT0_4-: J?.16 (Pin_16), U?.T5 (PL53B)
- new net EXT0_5+: J?.18 (Pin_18), U?.T4 (PL53C)
- new net EXT0_5-: J?.19 (Pin_19), U?.U5 (PL53D)
- new net EXT0_6+: J?.21 (Pin_21), U?.U4 (PL56A)
- new net EXT0_6-: J?.22 (Pin_22), U?.V4 (PL56B)
- new net EXT0_7+: J?.24 (Pin_24), U?.V6 (PL56C)
- new net EXT0_7-: J?.25 (Pin_25), U?.V7 (PL56D)
- new net EXT0_8+: J?.27 (Pin_27), U?.P2 (PL59A)
- new net EXT0_8-: J?.28 (Pin_28), U?.P3 (PL59B)
- new net EXT0_9+: J?.30 (Pin_30), U?.R3 (PL59C)
- new net EXT0_9-: J?.31 (Pin_31), U?.T3 (PL59D)
- new net EXT1_0+: J?.3 (Pin_3), U?.T1 (PL68A)
- new net EXT1_0-: J?.4 (Pin_4), U?.U1 (PL68B)
- new net EXT1_1+: J?.6 (Pin_6), U?.V1 (PL68C)
- new net EXT1_1-: J?.7 (Pin_7), U?.W1 (PL68D)
- new net EXT1_10+: J?.33 (Pin_33), U?.AB3 (PL83A)
- new net EXT1_10-: J?.34 (Pin_34), U?.AB4 (PL83B)
- new net EXT1_11+: J?.36 (Pin_36), U?.AC5 (PL83C)
- new net EXT1_11-: J?.37 (Pin_37), U?.AD4 (PL83D)
- new net EXT1_2+: J?.9 (Pin_9), U?.Y7 (PL71A)
- new net EXT1_2-: J?.10 (Pin_10), U?.Y6 (PL71B)
- new net EXT1_3+: J?.12 (Pin_12), U?.Y5 (PL71C)
- new net EXT1_3-: J?.13 (Pin_13), U?.W5 (PL71D)
- new net EXT1_4+: J?.15 (Pin_15), U?.Y4 (PL74A)
- new net EXT1_4-: J?.16 (Pin_16), U?.W4 (PL74B)
- new net EXT1_5+: J?.18 (Pin_18), U?.AB7 (PL74C)
- new net EXT1_5-: J?.19 (Pin_19), U?.AC6 (PL74D)
- new net EXT1_6+: J?.21 (Pin_21), U?.AB5 (PL77A)
- new net EXT1_6-: J?.22 (Pin_22), U?.AB6 (PL77B)
- new net EXT1_7+: J?.24 (Pin_24), U?.AC7 (PL77C)
- new net EXT1_7-: J?.25 (Pin_25), U?.AD7 (PL77D)
- new net EXT1_8+: J?.27 (Pin_27), U?.AD6 (PL80A)
- new net EXT1_8-: J?.28 (Pin_28), U?.AE6 (PL80B)
- new net EXT1_9+: J?.30 (Pin_30), U?.AE5 (PL80C)
- new net EXT1_9-: J?.31 (Pin_31), U?.AE4 (PL80D)
- new net EXT2_0+: J?.3 (Pin_3), U?.N6 (PL44A)
- new net EXT2_0-: J?.4 (Pin_4), U?.N7 (PL44B)
- new net EXT2_1+: J?.6 (Pin_6), U?.P6 (PL44C)
- new net EXT2_1-: J?.7 (Pin_7), U?.P7 (PL44D)
- new net EXT2_10+: J?.33 (Pin_33), U?.K2 (PL29A)
- new net EXT2_10-: J?.34 (Pin_34), U?.J1 (PL29B)
- new net EXT2_11+: J?.36 (Pin_36), U?.K1 (PL29C)
- new net EXT2_11-: J?.37 (Pin_37), U?.L1 (PL29D)
- new net EXT2_2+: J?.9 (Pin_9), U?.N3 (PL41A)
- new net EXT2_2-: J?.10 (Pin_10), U?.N4 (PL41B)
- new net EXT2_3+: J?.12 (Pin_12), U?.L7 (PL41C)
- new net EXT2_3-: J?.13 (Pin_13), U?.L6 (PL41D)
- new net EXT2_4+: J?.15 (Pin_15), U?.K6 (PL38A)
- new net EXT2_4-: J?.16 (Pin_16), U?.K7 (PL38B)
- new net EXT2_5+: J?.18 (Pin_18), U?.K5 (PL38C)
- new net EXT2_5-: J?.19 (Pin_19), U?.L4 (PL38D)
- new net EXT2_6+: J?.21 (Pin_21), U?.H6 (PL35A)
- new net EXT2_6-: J?.22 (Pin_22), U?.H5 (PL35B)
- new net EXT2_7+: J?.24 (Pin_24), U?.J7 (PL35C)
- new net EXT2_7-: J?.25 (Pin_25), U?.J6 (PL35D)
- new net EXT2_8+: J?.27 (Pin_27), U?.L2 (PL32A)
- new net EXT2_8-: J?.28 (Pin_28), U?.L3 (PL32B)
- new net EXT2_9+: J?.30 (Pin_30), U?.J4 (PL32C)
- new net EXT2_9-: J?.31 (Pin_31), U?.K4 (PL32D)
- new net EXT3_0+: J?.3 (Pin_3), U?.C5 (PL11A)
- new net EXT3_0-: J?.4 (Pin_4), U?.D5 (PL11B)
- new net EXT3_1+: J?.6 (Pin_6), U?.C4 (PL11C)
- new net EXT3_1-: J?.7 (Pin_7), U?.C3 (PL11D)
- new net EXT3_10+: J?.33 (Pin_33), U?.H2 (PL26A)
- new net EXT3_10-: J?.34 (Pin_34), U?.H3 (PL26B)
- new net EXT3_11+: J?.36 (Pin_36), U?.J3 (PL26C)
- new net EXT3_11-: J?.37 (Pin_37), U?.K3 (PL26D)
- new net EXT3_2+: J?.9 (Pin_9), U?.D4 (PL14A)
- new net EXT3_2-: J?.10 (Pin_10), U?.E4 (PL14B)
- new net EXT3_3+: J?.12 (Pin_12), U?.F4 (PL14C)
- new net EXT3_3-: J?.13 (Pin_13), U?.F5 (PL14D)
- new net EXT3_4+: J?.15 (Pin_15), U?.B1 (PL17A)
- new net EXT3_4-: J?.16 (Pin_16), U?.C2 (PL17B)
- new net EXT3_5+: J?.18 (Pin_18), U?.D3 (PL17C)
- new net EXT3_5-: J?.19 (Pin_19), U?.D2 (PL17D)
- new net EXT3_6+: J?.21 (Pin_21), U?.F3 (PL20A)
- new net EXT3_6-: J?.22 (Pin_22), U?.E3 (PL20B)
- new net EXT3_7+: J?.24 (Pin_24), U?.C1 (PL20C)
- new net EXT3_7-: J?.25 (Pin_25), U?.D1 (PL20D)
- new net EXT3_8+: J?.27 (Pin_27), U?.F2 (PL23A)
- new net EXT3_8-: J?.28 (Pin_28), U?.E1 (PL23B)
- new net EXT3_9+: J?.30 (Pin_30), U?.F1 (PL23C)
- new net EXT3_9-: J?.31 (Pin_31), U?.H1 (PL23D)
- new net VCCIO6: J?.1 (Pin_1), J?.1 (Pin_1), J?.2 (Pin_2), J?.2 (Pin_2), J?.39 (Pin_39), J?.39 (Pin_39), J?.40 (Pin_40), J?.40 (Pin_40)
- new net VCCIO7: J?.1 (Pin_1), J?.1 (Pin_1), J?.2 (Pin_2), J?.2 (Pin_2), J?.39 (Pin_39), J?.39 (Pin_39), J?.40 (Pin_40), J?.40 (Pin_40)
- no-connect marks 3 -> 7
Other:
- moved on the sheet: C?, U?, U?B, U?C, U?D, U?E

Commit message: hardware/mainboard: Add config, JTAG and boot flash
Signed-off-by: David Shah <dave@ds0.me>
Parts:
- added C? (x13): 470n, symbol Device:C_Small
- added C? (x6): 4.7µ, symbol Device:C_Small
- added C?: 100n, symbol Device:C_Small
- added D?: GREEN, symbol Device:LED
- added D?: RED, symbol Device:LED
- added JP?: CFG1, symbol Device:Jumper_NC_Small
- added Q?: BSH111BKR, Package_TO_SOT_SMD:SOT-23, symbol Transistor_FET:2N7002
- added R? (x2): 0R, symbol Device:R_Small
- added R? (x4): DNP, symbol Device:R_Small
- added R? (x3): 10k, symbol Device:R_Small
- added R? (x3): 1k, symbol Device:R_Small
- added R?: 22, symbol Device:R_Small
- added R?: 4.7k, symbol Device:R_Small
- added RN? (x2): 10k, symbol Device:R_Pack04
- added SW?: SW_Push, symbol Switch:SW_Push
- added U? (x3): ECP5UM5G_85_CABGA756, symbol ECP5UM5G:ECP5UM5G_85_CABGA756
- added U?: W25Q, symbol pkl_memory:W25Q
Connections:
- net +3V3: now also C?.1, C?.1, C?.1, C?.1, C?.1, JP?.1, R?.1, R?.1, R?.1, R?.1, R?.1, R?.1, R?.1, R?.2, R?.2, RN?.5 (R4.2), RN?.6 (R3.2), RN?.7 (R2.2), RN?.8 (R1.2), U?.8 (VCC), U?.AB10 (VCCIO8), U?.AB23 (VCCIO4), U?.AC10 (VCCIO8), U?.AC23 (VCCIO4)
- net GND: now also C?.2, C?.2, C?.2, C?.2, C?.2, C?.2, C?.2, C?.2, C?.2, C?.2, C?.2, C?.2, C?.2, C?.2, C?.2, C?.2, C?.2, C?.2, C?.2, C?.2, Q?.2 (S), RN?.2 (R2.1), RN?.3 (R3.1), RN?.4 (R4.1), SW?.1, U?.4 (GND)
- net VCCIO6: now also U?.AA10 (VCCIO6), U?.U10 (VCCIO6), U?.V10 (VCCIO6), U?.W10 (VCCIO6), C?.1, C?.1, C?.1, C?.1, C?.1, C?.1, C?.1, R?.1, R?.1, R?.1
- net VCCIO7: now also U?.M10 (VCCIO7), U?.P10 (VCCIO7), U?.R10 (VCCIO7), U?.T10 (VCCIO7), C?.1, C?.1, C?.1, C?.1, C?.1, C?.1, C?.1, R?.1, R?.1, R?.1
- new net: Q?.1 (G), R?.1
- new net: D?.1 (K), Q?.3 (D)
- new net: D?.2 (A), R?.2 (x2)
- new net +1V8: R?.2, R?.2
- new net +2V5: R?.2, R?.2
- new net CFG0: RN?.7 (R2.2), U?.AL4 (CFG_1)
- new net CFG1: JP?.2, RN?.6 (R3.2), U?.AK4 (CFG_2)
- new net CFG2: RN?.5 (R4.2), U?.AM4 (CFG_0)
- new net DONE: R?.2, R?.2, U?.AJ4 (DONE)
- new net FLASH_CLK: R?.2, U?.6 (CLK), U?.AM3 (CCLK)
- new net FLASH_D0: RN?.1 (R1.1), U?.5 (DI/IO0), U?.AK2 (PB11B)
- new net FLASH_D1: RN?.2 (R2.1), U?.2 (DO/IO1), U?.AJ2 (PB11A)
- new net FLASH_D2: RN?.3 (R3.1), U?.3 (~WP~/IO2), U?.AM2 (PB9B)
- new net FLASH_D3: RN?.4 (R4.1), U?.7 (~HLD~/~RST~/IO3), U?.AL1 (PB9A)
- new net FLASH_~CS: R?.2, U?.1 (~CS), U?.AJ3 (PB15A)
- new net JTAG_TCK: U?.AK5 (TCK)
- new net JTAG_TDI: U?.AJ5 (TDI)
- new net JTAG_TDO: U?.AG5 (TDO)
- new net JTAG_TMS: U?.AM5 (TMS)
- new net ~INIT: D?.1 (K), R?.2, U?.AG4 (INITN)
- new net ~PROGRAM: C?.1, R?.2, SW?.2, U?.AH4 (PROGRAMN)
- no-connect marks 7 -> 9

Commit message: hardware/mainboard: Connect FTDI and add quasi-dual-PMOD
Signed-off-by: David Shah <dave@ds0.me>
Parts:
- added J?: UART, symbol Connector_Generic:Conn_01x04
- added J?: JTAG, symbol Connector_Generic:Conn_01x06
- added J?: FLASH, symbol Connector_Generic:Conn_02x04_Odd_Even
- added J?: PMOD_01, symbol Connector_Generic:Conn_02x15_Odd_Even
Connections:
- net +3V3: now also J?.1 (Pin_1), J?.1 (Pin_1), J?.1 (Pin_1), J?.11 (Pin_11), J?.12 (Pin_12), J?.29 (Pin_29), J?.30 (Pin_30)
- net FLASH_CLK: now also J?.5 (Pin_5)
- net FLASH_D0: now also J?.2 (Pin_2)
- net FLASH_D1: now also J?.4 (Pin_4)
- net FLASH_D2: now also J?.6 (Pin_6)
- net FLASH_D3: now also J?.8 (Pin_8)
- net FLASH_~CS: now also J?.3 (Pin_3)
- net GND: now also J?.10 (Pin_10), J?.27 (Pin_27), J?.28 (Pin_28), J?.4 (Pin_4), J?.6 (Pin_6), J?.7 (Pin_7), J?.9 (Pin_9)
- net JTAG_TCK: now also J?.3 (Pin_3)
- net JTAG_TDI: now also J?.4 (Pin_4)
- net JTAG_TDO: now also J?.2 (Pin_2)
- net JTAG_TMS: now also J?.5 (Pin_5)
- net PMOD1_10: now reaches U?.D14 (PT47A)
- net PMOD1_10: now also J?.26 (Pin_26)
- net PMOD1_9: now reaches U?.E14 (PT45B)
- net PMOD1_9: now also J?.24 (Pin_24)
- net FTDI_~WR: now reaches U?.AG28 (PB110A)
- net FTDI_~SIWU: now reaches U?.AJ28 (PB112A)
- net FTDI_~TXE: now reaches U?.AJ31 (PB105B)
- net FTDI_D6: now reaches U?.AJ32 (PB101B)
- net FTDI_D3: now reaches U?.AK28 (PB98B)
- net FTDI_D4: now reaches U?.AK32 (PB101A)
- net FTDI_D1_RX: now reaches U?.AL28 (PB98A)
- net FTDI_D1_RX: now also J?.2 (Pin_2)
- net FTDI_D7: now reaches U?.AL30 (PB103B)
- net FTDI_~RD: now reaches U?.AL32 (PB107B)
- net FTDI_D0_TX: now reaches U?.AM28 (PB96A)
- net FTDI_D0_TX: now also J?.3 (Pin_3)
- net FTDI_D2: now reaches U?.AM29 (PB96B)
- net FTDI_D5: now reaches U?.AM30 (PB103A)
- net FTDI_~RXF: now reaches U?.AM31 (PB107A)
- net EXIO_1: now reaches U?.A24 (PT101A)
- net EXIO_1: now also J?.15 (Pin_15)
- net PMOD0_8: now reaches U?.A25 (PT105A)
- net PMOD0_8: now also J?.4 (Pin_4)
- net PMOD0_0: now reaches U?.A26 (PT112A)
- net PMOD0_0: now also J?.1 (Pin_1)
- net EXIO_5: now reaches U?.B22 (PT87B)
- net EXIO_5: now also J?.18 (Pin_18)
- net PMOD1_3: now reaches U?.B23 (PT94B)
- net PMOD1_3: now also J?.25 (Pin_25)
- net PMOD0_3: now reaches U?.B25 (PT105B)
- net PMOD0_3: now also J?.7 (Pin_7)
- net PMOD1_8: now reaches U?.C20 (PT83B)
- net PMOD1_8: now also J?.22 (Pin_22)
- net PMOD1_2: now reaches U?.C23 (PT96A)
- net PMOD1_2: now also J?.23 (Pin_23)
- net PMOD0_10: now reaches U?.C24 (PT101B)
- net PMOD0_10: now also J?.8 (Pin_8)
- net PMOD0_7: now reaches U?.C25 (PT107A)
- net PMOD0_7: now also J?.2 (Pin_2)
- net PMOD1_0: now reaches U?.D23 (PT96B)
- net PMOD1_0: now also J?.19 (Pin_19)
- net EXIO_0: now reaches U?.D24 (PT103A)
- net EXIO_0: now also J?.13 (Pin_13)
- net PMOD0_2: now reaches U?.D25 (PT107B)
- net PMOD0_2: now also J?.5 (Pin_5)
- net EXIO_4: now reaches U?.E22 (PT92A)
- net EXIO_4: now also J?.16 (Pin_16)
- net PMOD1_1: now reaches U?.E23 (PT98A)
- net PMOD1_1: now also J?.21 (Pin_21)
- net PMOD0_1: now reaches U?.E25 (PT110A)
- net PMOD0_1: now also J?.3 (Pin_3)
- net PMOD1_7: now reaches U?.F20 (PT85B)
- net PMOD1_7: now also J?.20 (Pin_20)
- net EXIO_3: now reaches U?.F22 (PT92B)
- net EXIO_3: now also J?.14 (Pin_14)
- net EXIO_2: now reaches U?.F23 (PT98B)
- net EXIO_2: now also J?.17 (Pin_17)
- net PMOD0_9: now reaches U?.F24 (PT103B)
- net PMOD0_9: now also J?.6 (Pin_6)
- net DDR3_Vtt_EN: now reaches U?.F25 (PT110B)

Commit message: hardware/mainboard: Re-annotate and fix ERC
Signed-off-by: David Shah <dave@ds0.me>
Parts:
- gave numbers to parts that had none: 74
Connections:
- net LED0: now also U15.AG29 (PB110B); no longer U15.A5 (PT9B)
- net LED1: now also U15.AH28 (PB112B); no longer U15.D7 (PT11A)
- net LED2: now also U15.AH30 (PB114A); no longer U15.A4 (PT9A)
- net LED3: now also U15.AK29 (PB116A); no longer U15.A3 (PT6B)
- net LED4: now also U15.AG30 (PB114B); no longer U15.B4 (PT4B)
- net LED5: now also U15.AK30 (PB116B); no longer U15.A2 (PT6A)
- net LED6: now also U15.AH32 (PB119A); no longer U15.B3 (PT4A)
- new net CLK_SD_OE: U15.A4 (PT9A)
- new net FPGA_12MHz: U15.B3 (PT4A)
- no-connect marks 9 -> 70

Commit message: hardware/mainboard: add microSD
Signed-off-by: David Shah <dave@ds0.me>
Parts:
- added R?: 22, symbol Device:R_Small
Connections:
- net USD_D0: now reaches U15.AG1 (PB4A)
- net USD_D2: now reaches U15.AH1 (PB4B)
- net USD_CMD: now reaches U15.AH3 (PB13B)
- net USD_D1: now reaches U15.AJ1 (PB6A)
- net USD_D3: now reaches U15.AK1 (PB6B)
- net at U15.AK3 (PB15B): now also R?.1
- new net USD_CLK: R?.2
- no-connect marks 70 -> 64
Changed lines of the file:
@@
 NoConn ~ 5600 8100
 NoConn ~ 5600 8200
-NoConn ~ 20650 4600
-NoConn ~ 20650 4700
-NoConn ~ 20650 4800
-NoConn ~ 20650 4900
 NoConn ~ 20650 5400
-NoConn ~ 20650 5600
-NoConn ~ 20650 5700
 NoConn ~ 20650 5800
 NoConn ~ 8100 11700
@@
 Wire Wire Line
 	11850 6900 11500 6900
+Text GLabel 20150 4600 0    50   BiDi ~ 0
+USD_D0
+Text GLabel 20150 4700 0    50   BiDi ~ 0
+USD_D1
+Text GLabel 20150 4800 0    50   BiDi ~ 0
+USD_D2
+Text GLabel 20150 4900 0    50   BiDi ~ 0
+USD_D3
+Text GLabel 20150 5600 0    50   BiDi ~ 0
+USD_CMD
+Text GLabel 20150 5700 0    50   Output ~ 0
+USD_CLK
+Wire Wire Line
+	20650 5600 20150 5600
+Wire Wire Line
+	20150 4900 20650 4900
+Wire Wire Line
+	20650 4800 20150 4800
+Wire Wire Line
+	20150 4700 20650 4700
+Wire Wire Line
+	20650 4600 20150 4600
+$Comp
+L Device:R_Small R?
+U 1 1 630CCB0A
+P 20400 5700
+F 0 "R?" V 20350 5800 50  0000 C CNN
+F 1 "22" V 20400 5700 50  0000 C CNN
+F 2 "" H 20400 5700 50  0001 C CNN
+F 3 "~" H 20400 5700 50  0001 C CNN
+	1    20400 5700
+	0    1    1    0
+$EndComp
+Wire Wire Line
+	20500 5700 20650 5700
+Wire Wire Line
+	20300 5700 20150 5700
 $EndSCHEMATC

Commit message: hardware/mainboard: Assign some footprints
Signed-off-by: David Shah <dave@ds0.me>
Parts:
- C213, C214, C215, C216, C217, C218, C224, C225, C226, C227, C229, C230, C231, C232, C234, C235, C236, C237, C238, C239, C241, C242, C244, C245, C246, C247, C248, C249, C251, C252, C253, C254: footprint (none) -> Capacitor_SMD:C_0402_1005Metric
- C219, C220, C221, C222, C223, C228, C233, C240, C243, C250: footprint (none) -> Capacitor_SMD:C_0603_1608Metric
- D26, D27: footprint (none) -> LED_SMD:LED_0805_2012Metric
- R82, R83, R84, R85, R86, R87: footprint (none) -> Resistor_SMD:R_0805_2012Metric
- R88, R89, R90, R91, R92, R93, R94, R95: footprint (none) -> Resistor_SMD:R_0402_1005Metric
- R97: renamed from R?; footprint (none) -> Resistor_SMD:R_0402_1005Metric
- RN22, RN23: footprint (none) -> Resistor_SMD:R_Array_Convex_4x0402
- U27: footprint (none) -> Package_SO:SO-8_5.3x6.2mm_P1.27mm

Commit message: hardware/mainboard: Assign more footprints
Signed-off-by: David Shah <dave@ds0.me>
Parts:
- J10: footprint (none) -> Connector_PinHeader_2.54mm:PinHeader_1x04_P2.54mm_Vertical
- J11: footprint (none) -> Connector_PinHeader_2.54mm:PinHeader_1x08_P2.54mm_Vertical
- J12: footprint (none) -> Connector_PinHeader_2.54mm:PinHeader_1x06_P2.54mm_Vertical
- J9: footprint (none) -> Connector_PinHeader_2.54mm:PinHeader_2x15_P2.54mm_Horizontal
- JP2: footprint (none) -> Connector_PinHeader_2.54mm:PinHeader_1x02_P2.54mm_Vertical
- SW6: footprint (none) -> Button_Switch_SMD:SW_SPST_B3S-1000
- U15: footprint (none) -> Custom Parts:CABGA756_27x27mm_p0.8mm
Changed lines of the file:
@@
 F 0 "U15" H 3481 -42 60  0000 L CNN
 F 1 "ECP5UM5G_85_CABGA756" H 3481 -148 60  0000 L CNN
-F 2 "" H 2350 1950 50  0001 C CNN
+F 2 "Custom Parts:CABGA756_27x27mm_p0.8mm" H 2350 1950 50  0001 C CNN
 F 3 "" H 2350 1950 50  0001 C CNN
 F 4 "ECP5UM5G_85" H 2500 1900 60  0001 R CNN "manf#"
@@
 F 0 "U15" H 6731 -892 60  0000 L CNN
 F 1 "ECP5UM5G_85_CABGA756" H 6731 -998 60  0000 L CNN
-F 2 "" H 5600 1900 50  0001 C CNN
+F 2 "Custom Parts:CABGA756_27x27mm_p0.8mm" H 5600 1900 50  0001 C CNN
 F 3 "" H 5600 1900 50  0001 C CNN
 F 4 "ECP5UM5G_85" H 5750 1850 60  0001 R CNN "manf#"
@@
 F 0 "U15" H 12981 -592 60  0000 L CNN
 F 1 "ECP5UM5G_85_CABGA756" H 12981 -698 60  0000 L CNN
-F 2 "" H 11850 1800 50  0001 C CNN
+F 2 "Custom Parts:CABGA756_27x27mm_p0.8mm" H 11850 1800 50  0001 C CNN
 F 3 "" H 11850 1800 50  0001 C CNN
 F 4 "ECP5UM5G_85" H 12000 1750 60  0001 R CNN "manf#"
@@
 F 0 "U15" H 16531 -192 60  0000 L CNN
 F 1 "ECP5UM5G_85_CABGA756" H 16531 -298 60  0000 L CNN
-F 2 "" H 15400 1800 50  0001 C CNN
+F 2 "Custom Parts:CABGA756_27x27mm_p0.8mm" H 15400 1800 50  0001 C CNN
 F 3 "" H 15400 1800 50  0001 C CNN
 F 4 "ECP5UM5G_85" H 15550 1750 60  0001 R CNN "manf#"
@@
 F 0 "U15" H 9231 6508 60  0000 L CNN
 F 1 "ECP5UM5G_85_CABGA756" H 9231 6402 60  0000 L CNN
-F 2 "" H 8100 9300 50  0001 C CNN
+F 2 "Custom Parts:CABGA756_27x27mm_p0.8mm" H 8100 9300 50  0001 C CNN
 F 3 "" H 8100 9300 50  0001 C CNN
 F 4 "ECP5UM5G_85" H 8250 9250 60  0001 R CNN "manf#"
@@
 F 0 "U15" H 13681 7308 60  0000 L CNN
 F 1 "ECP5UM5G_85_CABGA756" H 13681 7202 60  0000 L CNN
-F 2 "" H 12550 9300 50  0001 C CNN
+F 2 "Custom Parts:CABGA756_27x27mm_p0.8mm" H 12550 9300 50  0001 C CNN
 F 3 "" H 12550 9300 50  0001 C CNN
 F 4 "ECP5UM5G_85" H 12700 9250 60  0001 R CNN "manf#"
@@
 F 0 "U15" H 21781 2608 60  0000 L CNN
 F 1 "ECP5UM5G_85_CABGA756" H 21781 2502 60  0000 L CNN
-F 2 "" H 20650 4600 50  0001 C CNN
+F 2 "Custom Parts:CABGA756_27x27mm_p0.8mm" H 20650 4600 50  0001 C CNN
 F 3 "" H 20650 4600 50  0001 C CNN
 F 4 "ECP5UM5G_85" H 20800 4550 60  0001 R CNN "manf#"
@@
 F 0 "JP2" H 19400 6612 50  0000 C CNN
 F 1 "CFG1" H 19400 6521 50  0000 C CNN
-F 2 "" H 19400 6400 50  0001 C CNN
+F 2 "Connector_PinHeader_2.54mm:PinHeader_1x02_P2.54mm_Vertical" H 19400 6400 50  0001 C CNN
 F 3 "~" H 19400 6400 50  0001 C CNN
 	1    19400 6400
@@
 F 0 "SW6" V 22196 8448 50  0000 L CNN
 F 1 "SW_Push" V 22105 8448 50  0000 L CNN
-F 2 "" H 22150 8500 50  0001 C CNN
+F 2 "Button_Switch_SMD:SW_SPST_B3S-1000" H 22150 8500 50  0001 C CNN
 F 3 "" H 22150 8500 50  0001 C CNN
 	1    22150 8300
@@
 F 0 "U15" H 20700 12100 60  0000 L CNN
 F 1 "ECP5UM5G_85_CABGA756" H 20700 11950 60  0000 L CNN
-F 2 "" H 20100 12050 50  0001 C CNN
+F 2 "Custom Parts:CABGA756_27x27mm_p0.8mm" H 20100 12050 50  0001 C CNN
 F 3 "" H 20100 12050 50  0001 C CNN
 F 4 "ECP5UM5G_85" H 20250 12000 60  0001 R CNN "manf#"
@@
 F 0 "J10" H 15620 11617 50  0000 C CNN
 F 1 "UART" H 15620 11526 50  0000 C CNN
-F 2 "" H 15700 11300 50  0001 C CNN
+F 2 "Connector_PinHeader_2.54mm:PinHeader_1x04_P2.54mm_Vertical" H 15700 11300 50  0001 C CNN
 F 3 "~" H 15700 11300 50  0001 C CNN
 	1    15700 11300
@@
 F 0 "J12" H 20730 12792 50  0000 L CNN
 F 1 "JTAG" H 20730 12701 50  0000 L CNN
-F 2 "" H 20650 12800 50  0001 C CNN
+F 2 "Connector_PinHeader_2.54mm:PinHeader_1x06_P2.54mm_Vertical" H 20650 12800 50  0001 C CNN
 F 3 "~" H 20650 12800 50  0001 C CNN
 	1    20650 12800
@@
 F 0 "J11" H 19150 10667 50  0000 C CNN
 F 1 "FLASH" H 19150 10576 50  0000 C CNN
-F 2 "" H 19100 10350 50  0001 C CNN
+F 2 "Connector_PinHeader_2.54mm:PinHeader_1x08_P2.54mm_Vertical" H 19100 10350 50  0001 C CNN
 F 3 "~" H 19100 10350 50  0001 C CNN
 	1    19100 10350
@@
 F 0 "J9" H 15050 15417 50  0000 C CNN
 F 1 "PMOD_01" H 15050 15326 50  0000 C CNN
-F 2 "" H 15000 14500 50  0001 C CNN
+F 2 "Connector_PinHeader_2.54mm:PinHeader_2x15_P2.54mm_Horizontal" H 15000 14500 50  0001 C CNN
 F 3 "~" H 15000 14500 50  0001 C CNN
 	1    15000 14500
@@
 F 0 "U15" H 17100 11750 60  0000 L CNN
 F 1 "ECP5UM5G_85_CABGA756" H 17100 11600 60  0000 L CNN
-F 2 "" H 16500 11700 50  0001 C CNN
+F 2 "Custom Parts:CABGA756_27x27mm_p0.8mm" H 16500 11700 50  0001 C CNN
 F 3 "" H 16500 11700 50  0001 C CNN
 F 4 "ECP5UM5G_85" H 16650 11650 60  0001 R CNN "manf#"
