File: hardware/ecp5_mainboard/fpga_io.sch (KiCad schematic (older format))
At the start: 75 parts, among them J10 UART, J11 FLASH, J12 JTAG, J5 EXT0, J6 EXT1, J7 EXT1, J8 EXT1, J9 PMOD_01, Q9 BSH111BKR, SW6 SW_Push, U15 ECP5UM5G_85_CABGA756, U26 XL_XO_LVDS, U27 W25Q

Commit message: hardware: Creating and assigning some misc footprints
Signed-off-by: David Shah <dave@ds0.me>
Parts:
- U26: footprint (none) -> Custom Parts:OSC_IDT_XU_5x3.2mm
Changed lines of the file:
@@
 F 0 "U26" H 20150 1615 50  0000 C CNN
 F 1 "XL_XO_LVDS" H 20150 1524 50  0000 C CNN
-F 2 "" H 20150 1150 50  0001 C CNN
+F 2 "Custom Parts:OSC_IDT_XU_5x3.2mm" H 20150 1150 50  0001 C CNN
 F 3 "" H 20150 1150 50  0001 C CNN
 	1    20150 1150

Commit message: hardware/mainboard: All footprints assigned
Signed-off-by: David Shah <dave@ds0.me>
Parts:
- J5, J6: footprint (none) -> Custom Parts:TE_FPC_40pin_p0.5mm_4-1734839-0
- J7: value EXT1 -> EXT2; footprint (none) -> Custom Parts:TE_FPC_40pin_p0.5mm_4-1734839-0
- J8: value EXT1 -> EXT3; footprint (none) -> Custom Parts:TE_FPC_40pin_p0.5mm_4-1734839-0
Changed lines of the file:
@@
 F 0 "J5" H 1120 15817 50  0000 C CNN
 F 1 "EXT0" H 1120 15726 50  0000 C CNN
-F 2 "" H 1200 13700 50  0001 C CNN
+F 2 "Custom Parts:TE_FPC_40pin_p0.5mm_4-1734839-0" H 1200 13700 50  0001 C CNN
 F 3 "~" H 1200 13700 50  0001 C CNN
 	1    1200 13700
@@
 F 0 "J6" H 2320 15817 50  0000 C CNN
 F 1 "EXT1" H 2320 15726 50  0000 C CNN
-F 2 "" H 2400 13700 50  0001 C CNN
+F 2 "Custom Parts:TE_FPC_40pin_p0.5mm_4-1734839-0" H 2400 13700 50  0001 C CNN
 F 3 "~" H 2400 13700 50  0001 C CNN
 	1    2400 13700
@@
 P 3500 13700
 F 0 "J7" H 3420 15817 50  0000 C CNN
-F 1 "EXT1" H 3420 15726 50  0000 C CNN
-F 2 "" H 3500 13700 50  0001 C CNN
+F 1 "EXT2" H 3420 15726 50  0000 C CNN
+F 2 "Custom Parts:TE_FPC_40pin_p0.5mm_4-1734839-0" H 3500 13700 50  0001 C CNN
 F 3 "~" H 3500 13700 50  0001 C CNN
 	1    3500 13700
@@
 P 4550 13700
 F 0 "J8" H 4470 15817 50  0000 C CNN
-F 1 "EXT1" H 4470 15726 50  0000 C CNN
-F 2 "" H 4550 13700 50  0001 C CNN
+F 1 "EXT3" H 4470 15726 50  0000 C CNN
+F 2 "Custom Parts:TE_FPC_40pin_p0.5mm_4-1734839-0" H 4550 13700 50  0001 C CNN
 F 3 "~" H 4550 13700 50  0001 C CNN
 	1    4550 13700

Commit message: hardware/mainboard: All parts placed
Signed-off-by: David Shah <dave@ds0.me>
Parts:
- J11: footprint Connector_PinHeader_2.54mm:PinHeader_1x08_P2.54mm_Vertical -> Connector_PinHeader_2.54mm:PinHeader_2x04_P2.54mm_Vertical
Changed lines of the file:
@@
 F 0 "J11" H 19150 10667 50  0000 C CNN
 F 1 "FLASH" H 19150 10576 50  0000 C CNN
-F 2 "Connector_PinHeader_2.54mm:PinHeader_1x08_P2.54mm_Vertical" H 19100 10350 50  0001 C CNN
+F 2 "Connector_PinHeader_2.54mm:PinHeader_2x04_P2.54mm_Vertical" H 19100 10350 50  0001 C CNN
 F 3 "~" H 19100 10350 50  0001 C CNN
 	1    19100 10350

Commit message: hardware/mainboard: Tidying up
Signed-off-by: David Shah <dave@ds0.me>
Connections:
- net DDR3_DM0: no longer U15.K28 (PR38C)
- net DDR3_DQ0: no longer U15.P26 (PR44D)
- net DDR3_DQ1: no longer U15.N26 (PR44B)
- net DDR3_DQ2: no longer U15.P27 (PR44C)
- net DDR3_DQ3: no longer U15.N27 (PR44A)
- net DDR3_DQ4: no longer U15.L27 (PR41D)
- net DDR3_DQ5: no longer U15.L26 (PR41C)
- net DDR3_DQ6: no longer U15.L29 (PR38D)
- net DDR3_DQ7: no longer U15.K26 (PR38B)
Changed lines of the file:
@@
 Text GLabel 2150 2450 0    50   BiDi ~ 0
 DDR3_DQS0-
-Text GLabel 2150 1950 0    50   BiDi ~ 0
+Text GLabel -1250 1700 0    50   BiDi ~ 0
 DDR3_DQ0
-Text GLabel 2150 2050 0    50   BiDi ~ 0
+Text GLabel -1250 1800 0    50   BiDi ~ 0
 DDR3_DQ1
-Text GLabel 2150 2150 0    50   BiDi ~ 0
+Text GLabel -1250 1900 0    50   BiDi ~ 0
 DDR3_DQ2
-Text GLabel 2150 2250 0    50   BiDi ~ 0
+Text GLabel -1250 2000 0    50   BiDi ~ 0
 DDR3_DQ3
-Text GLabel 2150 2350 0    50   BiDi ~ 0
+Text GLabel -1250 2100 0    50   BiDi ~ 0
 DDR3_DQ4
-Text GLabel 2150 2550 0    50   BiDi ~ 0
+Text GLabel -1250 2600 0    50   BiDi ~ 0
 DDR3_DQ5
-Text GLabel 2150 2750 0    50   BiDi ~ 0
+Text GLabel -1250 2250 0    50   BiDi ~ 0
 DDR3_DQ6
-Text GLabel 2150 2850 0    50   BiDi ~ 0
+Text GLabel -1250 2350 0    50   BiDi ~ 0
 DDR3_DQ7
-Text GLabel 2150 2950 0    50   BiDi ~ 0
+Text GLabel -1250 2450 0    50   BiDi ~ 0
 DDR3_DM0
 Wire Wire Line
-	2150 1950 2350 1950
+	-1250 1700 -1050 1700
 Wire Wire Line
-	2150 2050 2350 2050
+	-1250 1800 -1050 1800
 Wire Wire Line
-	2150 2150 2350 2150
+	-1250 1900 -1050 1900
 Wire Wire Line
-	2150 2250 2350 2250
+	-1250 2000 -1050 2000
 Wire Wire Line
-	2150 2350 2350 2350
+	-1250 2100 -1050 2100
 Wire Wire Line
 	2150 2450 2350 2450
 Wire Wire Line
-	2150 2550 2350 2550
+	-1250 2600 -1050 2600
 Wire Wire Line
 	2150 2650 2350 2650
 Wire Wire Line
-	2150 2750 2350 2750
+	-1250 2250 -1050 2250
 Wire Wire Line
-	2150 2850 2350 2850
+	-1250 2350 -1050 2350
 Wire Wire Line
-	2150 2950 2350 2950
+	-1250 2450 -1050 2450
 Text GLabel 5400 1900 0    50   Input ~ 0
 DIP_SW0

Commit message: hardware/mainboard: Swapping DDR3 groups
Signed-off-by: David Shah <dave@ds0.me>
Connections:
- net DDR3_A0: now also U15.F31 (PR23A); no longer U15.W32 (PR68D)
- net DDR3_A1: now also U15.D32 (PR20D); no longer U15.U32 (PR68B)
- net DDR3_A10: now also U15.E29 (PR14B); no longer U15.U31 (PR62C)
- net DDR3_A11: now also U15.F29 (PR14C); no longer U15.N32 (PR62A)
- net DDR3_A12: now also U15.D29 (PR14A); no longer U15.T30 (PR59D)
- net DDR3_A13: now also U15.E32 (PR23B); no longer U15.Y28 (PR71C)
- net DDR3_A14: now also U15.F32 (PR23C); no longer U15.Y26 (PR71A)
- net DDR3_A2: now also U15.E30 (PR20B); no longer U15.V32 (PR68C)
- net DDR3_A3: now also U15.C32 (PR20C); no longer U15.T32 (PR68A)
- net DDR3_A4: now also U15.F30 (PR20A); no longer U15.Y30 (PR65D)
- net DDR3_A5: now also U15.D31 (PR17D); no longer U15.T31 (PR65B)
- net DDR3_A6: now also U15.C31 (PR17B); no longer U15.W30 (PR65C)
- net DDR3_A7: now also U15.D30 (PR17C); no longer U15.R32 (PR65A)
- net DDR3_A8: now also U15.B32 (PR17A); no longer U15.U30 (PR62D)
- net DDR3_A9: now also U15.F28 (PR14D); no longer U15.P32 (PR62B)
- net DDR3_BA0: now also U15.H32 (PR23D); no longer U15.Y27 (PR71B)
- net DDR3_BA1: now also U15.H31 (PR26A); no longer U15.W28 (PR71D)
- net DDR3_BA2: now also U15.J30 (PR26C); no longer U15.Y29 (PR74A)
- net DDR3_CAS: now also U15.K30 (PR26D); no longer U15.W29 (PR74B)
- net DDR3_CKE: now also U15.K32 (PR29C); no longer U15.AB28 (PR77A)
- net DDR3_CLK+: now also U15.L31 (PR32A); no longer U15.AD27 (PR80A)
- net DDR3_CLK-: now also U15.L30 (PR32B); no longer U15.AE27 (PR80B)
- net DDR3_CS: now also U15.K31 (PR29A); no longer U15.AC27 (PR74D)
- net DDR3_DM0: now also U15.U27 (PR50C)
- net DDR3_DM1: now also U15.K28 (PR38C); no longer U15.J30 (PR26C)
- net DDR3_DM2: now also U15.U31 (PR62C); no longer U15.F29 (PR14C)
- net DDR3_DM3: now also U15.Y26 (PR71A); no longer U15.R27 (PR50A)
- net DDR3_DQ0: now also U15.V26 (PR56D)
- net DDR3_DQ1: now also U15.R27 (PR50A)
- net DDR3_DQ10: now also U15.P27 (PR44C); no longer U15.J29 (PR32C)
- net DDR3_DQ11: now also U15.N27 (PR44A); no longer U15.L31 (PR32A)
- net DDR3_DQ12: now also U15.L27 (PR41D); no longer U15.L32 (PR29D)
- net DDR3_DQ13: now also U15.L26 (PR41C); no longer U15.K32 (PR29C)
- net DDR3_DQ14: now also U15.L29 (PR38D); no longer U15.K30 (PR26D)
- net DDR3_DQ15: now also U15.K26 (PR38B); no longer U15.H30 (PR26B)
- net DDR3_DQ16: now also U15.W32 (PR68D); no longer U15.D32 (PR20D)
- net DDR3_DQ17: now also U15.U32 (PR68B); no longer U15.E30 (PR20B)
- net DDR3_DQ18: now also U15.V32 (PR68C); no longer U15.C32 (PR20C)
- net DDR3_DQ19: now also U15.T32 (PR68A); no longer U15.F30 (PR20A)
- net DDR3_DQ2: now also U15.V27 (PR56C)
- net DDR3_DQ20: now also U15.Y30 (PR65D); no longer U15.D31 (PR17D)
- net DDR3_DQ21: now also U15.W30 (PR65C); no longer U15.D30 (PR17C)
- net DDR3_DQ22: now also U15.U30 (PR62D); no longer U15.F28 (PR14D)
- net DDR3_DQ23: now also U15.P32 (PR62B); no longer U15.E29 (PR14B)
- net DDR3_DQ24: now also U15.AC26 (PR77C); no longer U15.V26 (PR56D)
- net DDR3_DQ25: now also U15.AC27 (PR74D); no longer U15.V27 (PR56C)
- net DDR3_DQ26: now also U15.W29 (PR74B); no longer U15.U29 (PR56A)
- net DDR3_DQ27: now also U15.AB26 (PR74C); no longer U15.U28 (PR53D)
- net DDR3_DQ28: now also U15.Y29 (PR74A); no longer U15.T29 (PR53C)
- net DDR3_DQ29: now also U15.W28 (PR71D); no longer U15.U26 (PR50D)
- net DDR3_DQ3: now also U15.U29 (PR56A)
- net DDR3_DQ30: now also U15.Y27 (PR71B); no longer U15.T27 (PR50B)
- net DDR3_DQ31: now also U15.Y28 (PR71C); no longer U15.U27 (PR50C)
- net DDR3_DQ4: now also U15.U28 (PR53D)
- net DDR3_DQ5: now also U15.T29 (PR53C)
- net DDR3_DQ6: now also U15.U26 (PR50D)
- net DDR3_DQ7: now also U15.T27 (PR50B)
- net DDR3_DQ8: now also U15.P26 (PR44D); no longer U15.K29 (PR32D)
- net DDR3_DQ9: now also U15.N26 (PR44B); no longer U15.L30 (PR32B)
- net DDR3_DQS0+: now also U15.R29 (PR53A); no longer U15.N30 (PR41A)
- net DDR3_DQS0-: now also U15.T28 (PR53B); no longer U15.N29 (PR41B)
- net DDR3_DQS1+: now also U15.N30 (PR41A); no longer U15.K31 (PR29A)
- net DDR3_DQS1-: now also U15.N29 (PR41B); no longer U15.J32 (PR29B)
- net DDR3_DQS2+: now also U15.R32 (PR65A); no longer U15.B32 (PR17A)
- net DDR3_DQS2-: now also U15.T31 (PR65B); no longer U15.C31 (PR17B)
- net DDR3_DQS3+: now also U15.AB28 (PR77A); no longer U15.R29 (PR53A)
- net DDR3_DQS3-: now also U15.AB27 (PR77B); no longer U15.T28 (PR53B)
- net DDR3_ODT: now also U15.L32 (PR29D); no longer U15.AB27 (PR77B)
- net DDR3_RAS: now also U15.H30 (PR26B); no longer U15.AB26 (PR74C)
- net DDR3_RESET: now also U15.J29 (PR32C); no longer U15.AD26 (PR77D)
- net DDR3_WE: now also U15.J32 (PR29B); no longer U15.AC26 (PR77C)
- no-connect marks 64 -> 61

Commit message: hardware/mainboard: DDR3 Address routing
Signed-off-by: David Shah <dave@ds0.me>
Connections:
- net DDR3_A0: now also U15.E30 (PR20B); no longer U15.F31 (PR23A)
- net DDR3_A1: now also U15.F28 (PR14D); no longer U15.D32 (PR20D)
- net DDR3_A10: now also U15.H32 (PR23D); no longer U15.E29 (PR14B)
- net DDR3_A11: now also U15.F31 (PR23A); no longer U15.F29 (PR14C)
- net DDR3_A12: now also U15.F29 (PR14C); no longer U15.D29 (PR14A)
- net DDR3_A13: now also U15.B32 (PR17A); no longer U15.E32 (PR23B)
- net DDR3_A14: now also U15.D31 (PR17D); no longer U15.F32 (PR23C)
- net DDR3_A2: now also U15.C32 (PR20C); no longer U15.E30 (PR20B)
- net DDR3_A3: now also U15.E29 (PR14B); no longer U15.C32 (PR20C)
- net DDR3_A4: now also U15.F32 (PR23C); no longer U15.F30 (PR20A)
- net DDR3_A5: now also U15.D30 (PR17C); no longer U15.D31 (PR17D)
- net DDR3_A6: now also U15.E32 (PR23B); no longer U15.C31 (PR17B)
- net DDR3_A7: now also U15.D29 (PR14A); no longer U15.D30 (PR17C)
- net DDR3_A8: now also U15.D32 (PR20D); no longer U15.B32 (PR17A)
- net DDR3_A9: now also U15.C31 (PR17B); no longer U15.F28 (PR14D)
- net DDR3_BA0: now also U15.H31 (PR26A); no longer U15.H32 (PR23D)
- net DDR3_BA1: now also U15.H30 (PR26B); no longer U15.H31 (PR26A)
- net DDR3_CAS: now also U15.K31 (PR29A); no longer U15.K30 (PR26D)
- net DDR3_CS: now also U15.K29 (PR32D); no longer U15.K31 (PR29A)
- net DDR3_ODT: now also U15.J29 (PR32C); no longer U15.L32 (PR29D)
- net DDR3_RAS: now also U15.K30 (PR26D); no longer U15.H30 (PR26B)
- net DDR3_RESET: now also U15.L32 (PR29D); no longer U15.J29 (PR32C)
Changed lines of the file:
@@
 Wire Wire Line
 	5400 4300 5600 4300
+Text GLabel 2150 5250 0    50   Output ~ 0
+DDR3_A0
+Text GLabel 2150 5950 0    50   Output ~ 0
+DDR3_A1
+Text GLabel 2150 5350 0    50   Output ~ 0
+DDR3_A2
+Text GLabel 2150 6050 0    50   Output ~ 0
+DDR3_A3
+Text GLabel 2150 4950 0    50   Output ~ 0
+DDR3_A4
+Text GLabel 2150 5750 0    50   Output ~ 0
+DDR3_A5
+Text GLabel 2150 4850 0    50   Output ~ 0
+DDR3_A6
+Text GLabel 2150 6250 0    50   Output ~ 0
+DDR3_A7
+Text GLabel 2150 5150 0    50   Output ~ 0
+DDR3_A8
+Text GLabel 2150 5650 0    50   Output ~ 0
+DDR3_A9
+Text GLabel 2150 4750 0    50   Output ~ 0
+DDR3_A10
 Text GLabel 2150 5050 0    50   Output ~ 0
-DDR3_A0
-Text GLabel 2150 5150 0    50   Output ~ 0
-DDR3_A1
-Text GLabel 2150 5250 0    50   Output ~ 0
-DDR3_A2
-Text GLabel 2150 5350 0    50   Output ~ 0
-DDR3_A3
-Text GLabel 2150 5450 0    50   Output ~ 0
-DDR3_A4
+DDR3_A11
+Text GLabel 2150 6150 0    50   Output ~ 0
+DDR3_A12
+Text GLabel 2150 5850 0    50   Output ~ 0
+DDR3_A13
 Text GLabel 2150 5550 0    50   Output ~ 0
-DDR3_A5
-Text GLabel 2150 5650 0    50   Output ~ 0
-DDR3_A6
-Text GLabel 2150 5750 0    50   Output ~ 0
-DDR3_A7
-Text GLabel 2150 5850 0    50   Output ~ 0
-DDR3_A8
-Text GLabel 2150 5950 0    50   Output ~ 0
-DDR3_A9
-Text GLabel 2150 6050 0    50   Output ~ 0
-DDR3_A10
-Text GLabel 2150 6150 0    50   Output ~ 0
-DDR3_A11
-Text GLabel 2150 6250 0    50   Output ~ 0
-DDR3_A12
-Text GLabel 2150 4850 0    50   Output ~ 0
-DDR3_A13
-Text GLabel 2150 4950 0    50   Output ~ 0
 DDR3_A14
+Wire Wire Line
+	2150 5250 2350 5250
+Wire Wire Line
+	2150 5950 2350 5950
+Wire Wire Line
+	2150 5350 2350 5350
+Wire Wire Line
+	2150 6050 2350 6050
+Wire Wire Line
+	2150 4950 2350 4950
+Wire Wire Line
+	2150 5750 2350 5750
+Wire Wire Line
+	2150 4850 2350 4850
+Wire Wire Line
+	2150 6250 2350 6250
+Wire Wire Line
+	2150 5150 2350 5150
+Wire Wire Line
+	2150 5650 2350 5650
+Wire Wire Line
+	2150 4750 2350 4750
 Wire Wire Line
 	2150 5050 2350 5050
 Wire Wire Line
-	2150 5150 2350 5150
-Wire Wire Line
-	2150 5250 2350 5250
-Wire Wire Line
-	2150 5350 2350 5350
-Wire Wire Line
-	2150 5450 2350 5450
-Wire Wire Line
-	2150 5550 2350 5550
-Wire Wire Line
-	2150 5650 2350 5650
-Wire Wire Line
-	2150 5750 2350 5750
+	2150 6150 2350 6150
 Wire Wire Line
 	2150 5850 2350 5850
 Wire Wire Line
-	2150 5950 2350 5950
-Wire Wire Line
-	2150 6050 2350 6050
-Wire Wire Line
-	2150 6150 2350 6150
-Wire Wire Line
-	2150 6250 2350 6250
-Wire Wire Line
-	2150 4850 2350 4850
-Wire Wire Line
-	2150 4950 2350 4950
+	2150 5550 2350 5550
 NoConn ~ 5600 6600
-Text GLabel 2150 4750 0    50   Output ~ 0
+Text GLabel 2150 4650 0    50   Output ~ 0
 DDR3_BA0
-Text GLabel 2150 4650 0    50   Output ~ 0
+Text GLabel 2150 4450 0    50   Output ~ 0
 DDR3_BA1
 Text GLabel 2150 4550 0    50   Output ~ 0
 DDR3_BA2
-Text GLabel 2150 4450 0    50   Output ~ 0
+Text GLabel 2150 4350 0    50   Output ~ 0
 DDR3_RAS
-Text GLabel 2150 4350 0    50   Output ~ 0
+Text GLabel 2150 4250 0    50   Output ~ 0
 DDR3_CAS
 Text GLabel 2150 4150 0    50   Output ~ 0
@@
 Text GLabel 2150 4050 0    50   Output ~ 0
 DDR3_WE
+Text GLabel 2150 3750 0    50   Output ~ 0
+DDR3_ODT
 Text GLabel 2150 3950 0    50   Output ~ 0
-DDR3_ODT
-Text GLabel 2150 3750 0    50   Output ~ 0
 DDR3_RESET
-Text GLabel 2150 4250 0    50   Output ~ 0
+Text GLabel 2150 3550 0    50   Output ~ 0
 DDR3_CS
 Text GLabel 5400 5000 0    50   BiDi ~ 0
@@
 	5400 5000 5600 5000
 Wire Wire Line
+	2150 3950 2350 3950
+Wire Wire Line
 	2150 3750 2350 3750
-Wire Wire Line
-	2150 3950 2350 3950
 Wire Wire Line
 	2150 4050 2350 4050
@@
 	2150 4150 2350 4150
 Wire Wire Line
+	2150 3550 2350 3550
+Wire Wire Line
 	2150 4250 2350 4250
 Wire Wire Line
 	2150 4350 2350 4350
 Wire Wire Line
+	2150 4550 2350 4550
+Wire Wire Line
 	2150 4450 2350 4450
 Wire Wire Line
-	2150 4550 2350 4550
-Wire Wire Line
 	2150 4650 2350 4650
-Wire Wire Line
-	2150 4750 2350 4750
 Text GLabel 2150 3850 0    50   Output ~ 0
 DDR3_CLK+
