File: hardware/ecp5_mainboard/fpga_io.sch (KiCad schematic (older format))
At the start: 74 parts, among them J10 UART, J11 FLASH, J12 JTAG, J5 EXT0, J6 EXT1, J7 EXT2, J9 PMOD_01, Q9 BSH111BKR, SW6 SW_Push, U15 ECP5UM5G_85_CABGA756, U26 XL_XO_LVDS, U27 W25Q

Commit message: hardware/mainboard: Switching from SATA to m.2 connector for second DCU
Signed-off-by: David Shah <dave@ds0.me>
Connections:
- net M2_TXD: now reaches U15.K5 (PL38C)
- net M2_TXD: now also U15.P6 (PL44C)
- net M2_SDIO_CLK: now reaches U15.L4 (PL38D)
- net M2_SDIO_D2: now reaches U15.L6 (PL41D)
- net M2_SDIO_D0: now reaches U15.L7 (PL41C)
- net M2_SDIO_CMD: now reaches U15.N3 (PL41A)
- net M2_SDIO_D1: now reaches U15.N4 (PL41B)
- net M2_SDIO_D3: now reaches U15.N6 (PL44A)
- net M2_RTS: now reaches U15.N7 (PL44B)
- net M2_CTS: now reaches U15.P7 (PL44D)
Changed lines of the file:
@@
 Wire Bus Line
 	12350 2100 12550 2100
+Text GLabel 12150 13200 0    50   Input ~ 0
+M2_SDIO_CLK
+Text GLabel 12150 13300 0    50   BiDi ~ 0
+M2_SDIO_CMD
+Text GLabel 12150 13400 0    50   BiDi ~ 0
+M2_SDIO_D0
+Text GLabel 12150 13500 0    50   BiDi ~ 0
+M2_SDIO_D1
+Text GLabel 12150 13600 0    50   BiDi ~ 0
+M2_SDIO_D2
+Text GLabel 12150 13700 0    50   BiDi ~ 0
+M2_SDIO_D3
+Wire Wire Line
+	12150 13200 12550 13200
+Wire Wire Line
+	12150 13300 12550 13300
+Wire Wire Line
+	12150 13400 12550 13400
+Wire Wire Line
+	12150 13500 12550 13500
+Wire Wire Line
+	12150 13600 12550 13600
+Wire Wire Line
+	12150 13700 12550 13700
+Wire Wire Line
+	12550 13000 12250 13000
+Text GLabel 12250 13000 0    50   Input ~ 0
+M2_TXD
+Text GLabel 12250 13800 0    50   Output ~ 0
+M2_TXD
+Wire Wire Line
+	12250 13800 12550 13800
+Text GLabel 12250 13900 0    50   BiDi ~ 0
+M2_RTS
+Text GLabel 12250 14000 0    50   BiDi ~ 0
+M2_CTS
+Wire Wire Line
+	12250 13900 12550 13900
+Wire Wire Line
+	12550 14000 12250 14000
 $EndSCHEMATC

Commit message: hardware/mainboard: Add and place M.2 connector footprint
Signed-off-by: David Shah <davey1576@gmail.com>
Parts:
- U27: symbol pkl_memory:W25Q -> ecp5_mainboard-rescue:W25Q-pkl_memory
Changed lines of the file:
@@
 ~INIT
 $Comp
-L pkl_memory:W25Q U27
+L ecp5_mainboard-rescue:W25Q-pkl_memory U27
 U 1 1 60E46888
 P 20600 9650
+AR Path="/60E46888" Ref="U27"  Part="1"
+AR Path="/61FAF948/60E46888" Ref="U27"  Part="1"
 F 0 "U27" H 20600 10075 50  0000 C CNN
 F 1 "W25Q" H 20600 9984 50  0000 C CNN

Commit message: hardware/mainboard: Clock & M.2 routing
Signed-off-by: David Shah <davey1576@gmail.com>
Parts:
- added C258: 470n, Capacitor_SMD:C_0402_1005Metric, symbol Device:C_Small
- added FB3: 100R, Inductor_SMD:L_0603_1608Metric, symbol Device:Ferrite_Bead
Connections:
- net +3V3: now also FB3.1; no longer U26.6 (Vdd)
- net GND: now also C258.2
- net M2_TXD: no longer U15.K5 (PL38C)
- new net: C258.1, FB3.2, U26.6 (Vdd)
- new net M2_RXD: U15.K5 (PL38C)
Other:
- moved on the sheet: U26
Changed lines of the file:
@@
 L eco_glue:XL_XO_LVDS U26
 U 1 1 6249D25D
-P 20150 1150
-F 0 "U26" H 20150 1615 50  0000 C CNN
-F 1 "XL_XO_LVDS" H 20150 1524 50  0000 C CNN
-F 2 "Custom Parts:OSC_IDT_XU_5x3.2mm" H 20150 1150 50  0001 C CNN
-F 3 "" H 20150 1150 50  0001 C CNN
-	1    20150 1150
+P 20150 1400
+F 0 "U26" H 20150 1865 50  0000 C CNN
+F 1 "XL_XO_LVDS" H 20150 1774 50  0000 C CNN
+F 2 "Custom Parts:OSC_IDT_XU_5x3.2mm" H 20150 1400 50  0001 C CNN
+F 3 "" H 20150 1400 50  0001 C CNN
+	1    20150 1400
 	1    0    0    -1
 $EndComp
@@
 L power:GND #PWR0234
 U 1 1 6249D389
-P 19250 1500
-F 0 "#PWR0234" H 19250 1250 50  0001 C CNN
-F 1 "GND" H 19255 1327 50  0000 C CNN
-F 2 "" H 19250 1500 50  0001 C CNN
-F 3 "" H 19250 1500 50  0001 C CNN
-	1    19250 1500
+P 19250 1750
+F 0 "#PWR0234" H 19250 1500 50  0001 C CNN
+F 1 "GND" H 19255 1577 50  0000 C CNN
+F 2 "" H 19250 1750 50  0001 C CNN
+F 3 "" H 19250 1750 50  0001 C CNN
+	1    19250 1750
 	1    0    0    -1
 $EndComp
 Wire Wire Line
-	19250 1500 19250 1350
+	19250 1750 19250 1600
 Wire Wire Line
-	19250 1350 19450 1350
-NoConn ~ 19450 1150
-NoConn ~ 19450 950
+	19250 1600 19450 1600
+NoConn ~ 19450 1400
+NoConn ~ 19450 1200
 $Comp
 L power:+3V3 #PWR0240
 U 1 1 624F33B1
-P 21000 800
-F 0 "#PWR0240" H 21000 650 50  0001 C CNN
-F 1 "+3V3" H 21015 973 50  0000 C CNN
-F 2 "" H 21000 800 50  0001 C CNN
-F 3 "" H 21000 800 50  0001 C CNN
-	1    21000 800
-	1    0    0    -1
+P 22200 800
+F 0 "#PWR0240" H 22200 650 50  0001 C CNN
+F 1 "+3V3" H 22215 973 50  0000 C CNN
+F 2 "" H 22200 800 50  0001 C CNN
+F 3 "" H 22200 800 50  0001 C CNN
+	1    22200 800
+	0    1    1    0
 $EndComp
-Wire Wire Line
-	21000 800  21000 950
-Wire Wire Line
-	21000 950  20850 950
-Text Label 21800 1150 2    50   ~ 0
+Text Label 21800 1400 2    50   ~ 0
 CLK100-
 Wire Wire Line
-	21800 1150 20850 1150
-Text Label 21800 1350 2    50   ~ 0
+	21800 1400 20850 1400
+Text Label 21800 1600 2    50   ~ 0
 CLK100+
 Wire Wire Line
-	21800 1350 20850 1350
+	21800 1600 20850 1600
 Text GLabel 15050 4800 0    50   BiDi ~ 0
 CLK_SDA
@@
 	12550 13000 12250 13000
 Text GLabel 12250 13000 0    50   Input ~ 0
-M2_TXD
+M2_RXD
 Text GLabel 12250 13800 0    50   Output ~ 0
 M2_TXD
@@
 Wire Wire Line
 	12550 14000 12250 14000
+$Comp
+L Device:C_Small C258
+U 1 1 5C82DC49
+P 21500 1200
+F 0 "C258" H 21592 1246 50  0000 L CNN
+F 1 "470n" H 21592 1155 50  0000 L CNN
+F 2 "Capacitor_SMD:C_0402_1005Metric" H 21500 1200 50  0001 C CNN
+F 3 "~" H 21500 1200 50  0001 C CNN
+	1    21500 1200
+	0    -1   -1   0
+$EndComp
+$Comp
+L power:GND #PWR0259
+U 1 1 5C9E75A6
+P 21800 1200
+F 0 "#PWR0259" H 21800 950 50  0001 C CNN
+F 1 "GND" V 21805 1072 50  0000 R CNN
+F 2 "" H 21800 1200 50  0001 C CNN
+F 3 "" H 21800 1200 50  0001 C CNN
+	1    21800 1200
+	0    -1   -1   0
+$EndComp
+Wire Wire Line
+	21800 1200 21600 1200
+Wire Wire Line
+	20850 1200 21200 1200
+$Comp
+L Device:Ferrite_Bead FB3
+U 1 1 5CBA0958
+P 21900 800
+F 0 "FB3" V 21626 800 50  0000 C CNN
+F 1 "100R" V 21717 800 50  0000 C CNN
+F 2 "Inductor_SMD:L_0603_1608Metric" V 21830 800 50  0001 C CNN
+F 3 "~" H 21900 800 50  0001 C CNN
+	1    21900 800
+	0    1    1    0
+$EndComp
+Wire Wire Line
+	22050 800  22200 800
+Wire Wire Line
+	21750 800  21200 800
+Wire Wire Line
+	21200 800  21200 1200
+Connection ~ 21200 1200
+Wire Wire Line
+	21200 1200 21400 1200
+$Comp
+L power:PWR_FLAG #FLG0102
+U 1 1 5D1B2799
+P 21000 800
+F 0 "#FLG0102" H 21000 875 50  0001 C CNN
+F 1 "PWR_FLAG" V 21000 928 50  0000 L CNN
+F 2 "" H 21000 800 50  0001 C CNN
+F 3 "~" H 21000 800 50  0001 C CNN
+	1    21000 800
+	0    -1   -1   0
+$EndComp
+Wire Wire Line
+	21000 800  21200 800
+Connection ~ 21200 800
 $EndSCHEMATC

Commit message: hardware/mainboard: Misc routing
Signed-off-by: David Shah <davey1576@gmail.com>
Connections:
- net M2_SDIO_CMD: now also U15.K4 (PL32D); no longer U15.N3 (PL41A)
Changed lines of the file:
@@
 Text GLabel 12150 13200 0    50   Input ~ 0
 M2_SDIO_CLK
-Text GLabel 12150 13300 0    50   BiDi ~ 0
+Text GLabel 12150 12400 0    50   BiDi ~ 0
 M2_SDIO_CMD
 Text GLabel 12150 13400 0    50   BiDi ~ 0
@@
 	12150 13200 12550 13200
 Wire Wire Line
-	12150 13300 12550 13300
+	12150 12400 12550 12400
 Wire Wire Line
 	12150 13400 12550 13400
