File: hardware/ecp5_mainboard/ecp5_mainboard.kicad_pcb (KiCad board)
At the start: 2 copper layers, 158.1 x 111.2 mm, 1 part

Commit message: hardware.mainboard: Fixes from PCB import
Signed-off-by: David Shah <dave@ds0.me>
Parts:
- removed REF**: PCIe_EDGE_x4, Custom Parts:PCIe_EDGE_x4
- added C1: 1µ, Capacitor_SMD:C_0603_1608Metric, F.Cu at (276.1, 51.8)
- added C10: 1µ, Capacitor_SMD:C_0603_1608Metric, F.Cu at (275.1, 68.0)
- added C100: 100n, Capacitor_SMD:C_0402_1005Metric, F.Cu at (224.5, 26.6)
- added C101: 100n, Capacitor_SMD:C_0402_1005Metric, F.Cu at (216.6, 31.9)
- added C102: 100n, Capacitor_SMD:C_0402_1005Metric, F.Cu at (216.6, 32.9)
- added C103: 100n, Capacitor_SMD:C_0402_1005Metric, F.Cu at (244.8, 4.89)
- added C104: 100n, Capacitor_SMD:C_0402_1005Metric, F.Cu at (220.0, 29.9)
- added C105: 100n, Capacitor_SMD:C_0402_1005Metric, F.Cu at (246.5, 3.40)
- added C106: 100n, Capacitor_SMD:C_0402_1005Metric, F.Cu at (249.6, 0.90)
- added C107: 10µ, Capacitor_SMD:C_0805_2012Metric, F.Cu at (243.9, 3.42)
- added C108: 470n, Capacitor_SMD:C_0402_1005Metric, F.Cu at (227.9, 24.6)
- added C109: 10µ, Capacitor_SMD:C_0805_2012Metric, F.Cu at (238.7, 5.40)
- added C11: 180p, Capacitor_SMD:C_0402_1005Metric, F.Cu at (282.4, 68.4)
- added C110: 470n, Capacitor_SMD:C_0402_1005Metric, F.Cu at (248.5, 2.41)
- added C111: 470n, Capacitor_SMD:C_0402_1005Metric, F.Cu at (238.2, 11.3)
- added C112: 470n, Capacitor_SMD:C_0402_1005Metric, F.Cu at (244.8, 5.88)
- added C113: 470n, Capacitor_SMD:C_0402_1005Metric, F.Cu at (244.0, 7.86)
- added C114: 470n, Capacitor_SMD:C_0402_1005Metric, F.Cu at (218.5, 32.9)
- added C115: DNP, Capacitor_SMD:C_0402_1005Metric, F.Cu at (216.6, 34.8)
- added C116: 470n, Capacitor_SMD:C_0402_1005Metric, F.Cu at (240.1, 11.1)
- added C117: DNP, Capacitor_SMD:C_0402_1005Metric, F.Cu at (237.3, 13.3)
- added C118: 100n, Capacitor_SMD:C_0402_1005Metric, F.Cu at (218.5, 33.9)
- added C119: 10µ, Capacitor_SMD:C_0805_2012Metric, F.Cu at (263.7, 36.9)
- added C12: 750p, Capacitor_SMD:C_0402_1005Metric, F.Cu at (303.3, 51.3)
- added C120: 10µ, Capacitor_SMD:C_0805_2012Metric, F.Cu at (270.5, 36.7)
- added C121: 100p, Capacitor_SMD:C_0402_1005Metric, F.Cu at (303.2, 30.5)
- added C122: 470n, Capacitor_SMD:C_0402_1005Metric, F.Cu at (311.9, 23.6)
- added C123: 10µ, Capacitor_SMD:C_0805_2012Metric, F.Cu at (267.1, 36.7)
- added C124: 10µ, Capacitor_SMD:C_0805_2012Metric, F.Cu at (301.3, 24.0)
- added C125: 10µ, Capacitor_SMD:C_0805_2012Metric, F.Cu at (309.2, 23.1)
- added C126: 10n, Capacitor_SMD:C_0402_1005Metric, F.Cu at (307.5, 27.1)
- added C127: 10n, Capacitor_SMD:C_0402_1005Metric, F.Cu at (323.8, 10.5)
- added C128: 10n, Capacitor_SMD:C_0402_1005Metric, F.Cu at (318.7, 15.9)
- added C129: 10n, Capacitor_SMD:C_0402_1005Metric, F.Cu at (319.8, 14.3)
- added C13: 47µ, Capacitor_SMD:C_1210_3225Metric, F.Cu at (294.5, 42.9)
- added C130: 10n, Capacitor_SMD:C_0402_1005Metric, F.Cu at (323.8, 11.5)
- added C131: 10n, Capacitor_SMD:C_0402_1005Metric, F.Cu at (299.3, 34.7)
- added C132: 100n, Capacitor_SMD:C_0402_1005Metric, F.Cu at (316.8, 17.8)
- added C133: 100n, Capacitor_SMD:C_0402_1005Metric, F.Cu at (309.0, 24.6)
- added C134: 100n, Capacitor_SMD:C_0402_1005Metric, F.Cu at (321.9, 13.1)
- added C135: 100n, Capacitor_SMD:C_0402_1005Metric, F.Cu at (305.5, 29.5)
- added C136: 22p, Capacitor_SMD:C_0402_1005Metric, F.Cu at (309.0, 25.6)
- added C137: 100u, Capacitor_SMD:CP_Elec_6.3x5.8, F.Cu at (294.9, 26.6)
- added C138: 4.7µ, Capacitor_SMD:C_0603_1608Metric, F.Cu at (304.1, 25.7)
- added C139: 4.7µ, Capacitor_SMD:C_0603_1608Metric, F.Cu at (317.3, 14.6)
- added C14: 10µ, Capacitor_SMD:C_0805_2012Metric, F.Cu at (302.2, 47.9)
- added C140: 470n, Capacitor_SMD:C_0402_1005Metric, F.Cu at (301.4, 33.6)
- added C141: 100n, Capacitor_SMD:C_0402_1005Metric, F.Cu at (313.8, 22.6)
- added C142: 4.7µ, Capacitor_SMD:C_0603_1608Metric, F.Cu at (322.5, 4.81)
- added C143: 22p, Capacitor_SMD:C_0402_1005Metric, F.Cu at (305.1, 30.5)
- added C144: 10n, Capacitor_SMD:C_0402_1005Metric, F.Cu at (307.5, 28.1)
- added C145: 10n, Capacitor_SMD:C_0402_1005Metric, F.Cu at (301.2, 34.6)
- added C146: 10n, Capacitor_SMD:C_0402_1005Metric, F.Cu at (303.3, 31.5)
- added C147: 12p, Capacitor_SMD:C_0402_1005Metric, F.Cu at (321.9, 14.1)
- added C148: 10n, Capacitor_SMD:C_0402_1005Metric, F.Cu at (324.0, 7.57)
- added C149: 10n, Capacitor_SMD:C_0402_1005Metric, F.Cu at (299.3, 35.7)
- added C15: 10µ, Capacitor_SMD:C_0805_2012Metric, F.Cu at (288.1, 62.8)
- added C150: 10n, Capacitor_SMD:C_0402_1005Metric, F.Cu at (294.7, 37.0)
- added C151: 12p, Capacitor_SMD:C_0402_1005Metric, F.Cu at (305.6, 28.1)
- added C152: 10n, Capacitor_SMD:C_0402_1005Metric, F.Cu at (297.4, 35.7)
- added C153: 10n, Capacitor_SMD:C_0402_1005Metric, F.Cu at (321.9, 12.1)
- added C154: 10n, Capacitor_SMD:C_0402_1005Metric, F.Cu at (310.9, 25.6)
- added C155: 10n, Capacitor_SMD:C_0402_1005Metric, F.Cu at (299.3, 36.7)
- added C156: 470n, Capacitor_SMD:C_0402_1005Metric, F.Cu at (323.8, 12.5)
- added C157: 10n, Capacitor_SMD:C_0402_1005Metric, F.Cu at (318.7, 16.8)
- added C158: 10n, Capacitor_SMD:C_0402_1005Metric, F.Cu at (320.6, 15.3)
- added C159: 470n, Capacitor_SMD:C_0402_1005Metric, F.Cu at (310.9, 24.6)
- added C16: 10µ, Capacitor_SMD:C_0805_2012Metric, F.Cu at (298.7, 49.4)
- added C160: 10n, Capacitor_SMD:C_0402_1005Metric, F.Cu at (316.8, 18.8)
- added C161: 4.7µ, Capacitor_SMD:C_0603_1608Metric, F.Cu at (301.1, 28.7)
- added C162: 470n, Capacitor_SMD:C_0402_1005Metric, F.Cu at (313.8, 23.6)
- added C163: 470n, Capacitor_SMD:C_0402_1005Metric, F.Cu at (305.6, 27.1)
- added C164: 4.7µ, Capacitor_SMD:C_0603_1608Metric, F.Cu at (322.5, 6.32)
- added C165: 4.7µ, Capacitor_SMD:C_0603_1608Metric, F.Cu at (279.8, 36.7)
- added C166: 100n, Capacitor_SMD:C_0402_1005Metric, F.Cu at (303.6, 29.5)
- added C167: 100n, Capacitor_SMD:C_0402_1005Metric, F.Cu at (321.9, 11.1)
- added C168: 100n, Capacitor_SMD:C_0402_1005Metric, F.Cu at (297.4, 36.7)
- added C169: 100n, Capacitor_SMD:C_0402_1005Metric, F.Cu at (301.4, 31.6)
- added C17: 10µ, Capacitor_SMD:C_0805_2012Metric, F.Cu at (283.2, 65.0)
- added C170: 100n, Capacitor_SMD:C_0402_1005Metric, F.Cu at (301.4, 32.6)
- added C171: 100n, Capacitor_SMD:C_0402_1005Metric, F.Cu at (299.5, 33.2)
- added C172: 4.7µ, Capacitor_SMD:C_0603_1608Metric, F.Cu at (282.8, 36.7)
- added C173: 4.7µ, Capacitor_SMD:C_0603_1608Metric, F.Cu at (285.8, 36.7)
- added C174: 10µ, Capacitor_SMD:C_0805_2012Metric, F.Cu at (160.0, 147.3)
- added C175: 100n, Capacitor_SMD:C_0402_1005Metric, F.Cu at (154.9, 159.1)
- added C176: 10µ, Capacitor_SMD:C_0805_2012Metric, F.Cu at (140.4, 162.3)
- added C177: 10µ, Capacitor_SMD:C_0805_2012Metric, F.Cu at (133.6, 162.3)
- added C178: 10µ, Capacitor_SMD:C_0805_2012Metric, F.Cu at (137.0, 162.3)
- added C179: 100n, Capacitor_SMD:C_0402_1005Metric, F.Cu at (160.4, 153.3)
- added C18: 10µ, Capacitor_SMD:C_0805_2012Metric, F.Cu at (284.5, 62.9)
- added C180: 10µ, Capacitor_SMD:C_0805_2012Metric, F.Cu at (155.7, 151.6)
- added C181: 100n, Capacitor_SMD:C_0402_1005Metric, F.Cu at (162.3, 151.3)
- added C182: 10µ, Capacitor_SMD:C_0603_1608Metric, F.Cu at (143.6, 162.1)
- added C183: 4.7µ, Capacitor_SMD:C_0603_1608Metric, F.Cu at (146.6, 162.1)
- added C184: 4.7µ, Capacitor_SMD:C_0603_1608Metric, F.Cu at (155.5, 153.3)
- added C185: 470n, Capacitor_SMD:C_0402_1005Metric, F.Cu at (160.4, 152.3)
- added C186: 470n, Capacitor_SMD:C_0402_1005Metric, F.Cu at (156.8, 157.2)
- added C187: 470n, Capacitor_SMD:C_0402_1005Metric, F.Cu at (153.0, 161.8)
- added C188: 470n, Capacitor_SMD:C_0402_1005Metric, F.Cu at (151.1, 163.8)
- added C189: 470n, Capacitor_SMD:C_0402_1005Metric, F.Cu at (162.3, 152.3)
- added C19: 120p, Capacitor_SMD:C_0402_1005Metric, F.Cu at (286.3, 47.9)
- added C190: 470n, Capacitor_SMD:C_0402_1005Metric, F.Cu at (158.9, 156.2)
- added C191: 470n, Capacitor_SMD:C_0402_1005Metric, F.Cu at (154.9, 158.1)
- added C192: 470n, Capacitor_SMD:C_0402_1005Metric, F.Cu at (162.4, 149.3)
- added C193: 470n, Capacitor_SMD:C_0402_1005Metric, F.Cu at (160.4, 151.3)
- added C194: 470n, Capacitor_SMD:C_0402_1005Metric, F.Cu at (160.0, 154.3)
- added C195: 470n, Capacitor_SMD:C_0402_1005Metric, F.Cu at (154.9, 157.1)
- added C196: 470n, Capacitor_SMD:C_0402_1005Metric, F.Cu at (146.9, 163.3)
- added C197: 470n, Capacitor_SMD:C_0402_1005Metric, F.Cu at (151.1, 161.8)
- added C198: 470n, Capacitor_SMD:C_0402_1005Metric, F.Cu at (157.0, 156.2)
- added C199: 470n, Capacitor_SMD:C_0402_1005Metric, F.Cu at (162.4, 150.3)
- added C2: 100µF/25V, Capacitor_SMD:CP_Elec_6.3x5.8, F.Cu at (263.3, 62.6)
- added C20: 120p, Capacitor_SMD:C_0402_1005Metric, F.Cu at (304.8, 49.7)
- added C200: 470n, Capacitor_SMD:C_0402_1005Metric, F.Cu at (140.4, 163.8)
- added C201: 100n, Capacitor_SMD:C_0402_1005Metric, F.Cu at (144.9, 163.3)
- added C202: 100n, Capacitor_SMD:C_0402_1005Metric, F.Cu at (132.8, 163.8)
- added C203: 470n, Capacitor_SMD:C_0402_1005Metric, F.Cu at (138.5, 163.8)
- added C204: 470n, Capacitor_SMD:C_0402_1005Metric, F.Cu at (136.6, 163.8)
- added C205: 470n, Capacitor_SMD:C_0402_1005Metric, F.Cu at (134.7, 163.8)
- added C206: 470n, Capacitor_SMD:C_0402_1005Metric, F.Cu at (143.0, 163.3)
- added C207: 100n, Capacitor_SMD:C_0402_1005Metric, F.Cu at (156.8, 158.2)
- added C208: 100n, Capacitor_SMD:C_0402_1005Metric, F.Cu at (154.9, 160.1)
- added C209: 470n, Capacitor_SMD:C_0402_1005Metric, F.Cu at (158.7, 158.2)
- added C21: 120p, Capacitor_SMD:C_0402_1005Metric, F.Cu at (302.7, 52.3)
- added C210: 470n, Capacitor_SMD:C_0402_1005Metric, F.Cu at (160.8, 156.2)
- added C211: 470n, Capacitor_SMD:C_0402_1005Metric, F.Cu at (154.9, 161.1)
- added C212: 470n, Capacitor_SMD:C_0402_1005Metric, F.Cu at (161.9, 154.3)
- added C213: 100n, Capacitor_SMD:C_0402_1005Metric, F.Cu at (64.1, 154.6)
- added C214: 100n, Capacitor_SMD:C_0402_1005Metric, F.Cu at (62.2, 154.6)
- added C215: 470n, Capacitor_SMD:C_0402_1005Metric, F.Cu at (94.1, 138.7)
- added C216: 470n, Capacitor_SMD:C_0402_1005Metric, F.Cu at (96.0, 136.8)
- added C217: 470n, Capacitor_SMD:C_0402_1005Metric, F.Cu at (108.6, 123.6)
- added C218: 470n, Capacitor_SMD:C_0402_1005Metric, F.Cu at (87.3, 144.8)
- added C219: 4.7µ, Capacitor_SMD:C_0603_1608Metric, F.Cu at (77.5, 151.9)
- added C22: 120p, Capacitor_SMD:C_0402_1005Metric, F.Cu at (293.5, 61.8)
- added C220: 4.7µ, Capacitor_SMD:C_0603_1608Metric, F.Cu at (80.9, 149.9)
- added C221: 4.7µ, Capacitor_SMD:C_0603_1608Metric, F.Cu at (103.8, 124.3)
- added C222: 4.7µ, Capacitor_SMD:C_0603_1608Metric, F.Cu at (100.2, 130.9)
- added C223: 4.7µ, Capacitor_SMD:C_0603_1608Metric, F.Cu at (94.6, 135.5)
- added C224: 470n, Capacitor_SMD:C_0402_1005Metric, F.Cu at (90.7, 140.7)
- added C225: 470n, Capacitor_SMD:C_0402_1005Metric, F.Cu at (69.8, 154.6)
- added C226: 470n, Capacitor_SMD:C_0402_1005Metric, F.Cu at (58.4, 154.6)
- added C227: 470n, Capacitor_SMD:C_0402_1005Metric, F.Cu at (78.9, 153.6)
- added C228: 4.7µ, Capacitor_SMD:C_0603_1608Metric, F.Cu at (107.2, 122.4)
- added C229: 470n, Capacitor_SMD:C_0402_1005Metric, F.Cu at (86.3, 146.8)
- added C23: 10µ, Capacitor_SMD:C_0805_2012Metric, F.Cu at (305.6, 46.1)
- added C230: 470n, Capacitor_SMD:C_0402_1005Metric, F.Cu at (107.8, 124.6)
- added C231: 470n, Capacitor_SMD:C_0402_1005Metric, F.Cu at (104.8, 128.1)
- added C232: 470n, Capacitor_SMD:C_0402_1005Metric, F.Cu at (66.0, 154.6)
- added C233: 4.7µ, Capacitor_SMD:C_0603_1608Metric, F.Cu at (91.2, 139.4)
- added C234: 470n, Capacitor_SMD:C_0402_1005Metric, F.Cu at (109.7, 122.1)
- added C235: 470n, Capacitor_SMD:C_0402_1005Metric, F.Cu at (104.8, 127.1)
- added C236: 470n, Capacitor_SMD:C_0402_1005Metric, F.Cu at (84.1, 148.4)
- added C237: 470n, Capacitor_SMD:C_0402_1005Metric, F.Cu at (86.3, 145.8)
- added C238: 470n, Capacitor_SMD:C_0402_1005Metric, F.Cu at (113.0, 117.4)
- added C239: 470n, Capacitor_SMD:C_0402_1005Metric, F.Cu at (97.5, 134.3)
- added C24: 10µ, Capacitor_SMD:C_0805_2012Metric, F.Cu at (298.1, 53.5)
- added C240: 4.7µ, Capacitor_SMD:C_0603_1608Metric, F.Cu at (84.8, 144.6)
- added C241: 470n, Capacitor_SMD:C_0402_1005Metric, F.Cu at (99.6, 132.2)
- added C242: 470n, Capacitor_SMD:C_0402_1005Metric, F.Cu at (80.0, 152.6)
- added C243: 4.7µ, Capacitor_SMD:C_0603_1608Metric, F.Cu at (105.3, 125.8)
- added C244: 470n, Capacitor_SMD:C_0402_1005Metric, F.Cu at (90.7, 141.6)
- added C245: 470n, Capacitor_SMD:C_0402_1005Metric, F.Cu at (83.4, 149.3)
- added C246: 470n, Capacitor_SMD:C_0402_1005Metric, F.Cu at (106.7, 123.6)
- added C247: 470n, Capacitor_SMD:C_0402_1005Metric, F.Cu at (97.5, 133.3)
- added C248: 470n, Capacitor_SMD:C_0402_1005Metric, F.Cu at (77.0, 154.1)
- added C249: 470n, Capacitor_SMD:C_0402_1005Metric, F.Cu at (67.9, 154.6)
- added C25: 10µ, Capacitor_SMD:C_0805_2012Metric, F.Cu at (291.6, 59.3)
- added C250: 4.7µ, Capacitor_SMD:C_0603_1608Metric, F.Cu at (88.3, 141.0)
- added C251: 470n, Capacitor_SMD:C_0402_1005Metric, F.Cu at (116.4, 115.4)
- added C252: 470n, Capacitor_SMD:C_0402_1005Metric, F.Cu at (94.1, 136.8)
- added C253: 100n, Capacitor_SMD:C_0402_1005Metric, F.Cu at (94.1, 137.7)
- added C254: 470n, Capacitor_SMD:C_0402_1005Metric, F.Cu at (113.0, 118.4)
- added C255: 10µ, Capacitor_SMD:C_0805_2012Metric, F.Cu at (260.3, 36.7)
- added C26: 10µ, Capacitor_SMD:C_0805_2012Metric, F.Cu at (286.6, 64.8)
- added C27: 10µ, Capacitor_SMD:C_0805_2012Metric, F.Cu at (305.8, 42.2)
- added C28: 10µ, Capacitor_SMD:C_0805_2012Metric, F.Cu at (292.9, 57.3)
- added C29: 10µ, Capacitor_SMD:C_0805_2012Metric, F.Cu at (305.8, 44.2)
- added C3: 10µ, Capacitor_SMD:C_0805_2012Metric, F.Cu at (302.2, 49.9)
- added C30: 10µ, Capacitor_SMD:C_0805_2012Metric, F.Cu at (298.7, 51.4)
- added C31: 47µ, Capacitor_SMD:C_1210_3225Metric, F.Cu at (161.7, 122.0)
- added C32: 4.7µ, Capacitor_SMD:C_0603_1608Metric, F.Cu at (160.9, 128.9)
- added C33: 47µ, Capacitor_SMD:C_1210_3225Metric, F.Cu at (166.3, 116.5)
- added C34: 47µ, Capacitor_SMD:C_1210_3225Metric, F.Cu at (166.3, 119.7)
- added C35: 4.7µ, Capacitor_SMD:C_0603_1608Metric, F.Cu at (163.9, 125.9)
- added C36: 4.7µ, Capacitor_SMD:C_0603_1608Metric, F.Cu at (163.9, 124.3)
- added C37: 4.7µ, Capacitor_SMD:C_0603_1608Metric, F.Cu at (173.1, 118.8)
- added C38: 470n, Capacitor_SMD:C_0402_1005Metric, F.Cu at (160.4, 132.1)
- added C39: 470n, Capacitor_SMD:C_0402_1005Metric, F.Cu at (175.6, 117.9)
- added C4: 10µ, Capacitor_SMD:C_0805_2012Metric, F.Cu at (294.7, 53.6)
- added C40: 470n, Capacitor_SMD:C_0402_1005Metric, F.Cu at (168.3, 124.3)
- added C41: 470n, Capacitor_SMD:C_0402_1005Metric, F.Cu at (166.4, 123.3)
- added C42: 10n, Capacitor_SMD:C_0402_1005Metric, F.Cu at (160.4, 131.1)
- added C43: 10n, Capacitor_SMD:C_0402_1005Metric, F.Cu at (160.4, 133.1)
- added C44: 470n, Capacitor_SMD:C_0402_1005Metric, F.Cu at (169.1, 126.3)
- added C45: 470n, Capacitor_SMD:C_0402_1005Metric, F.Cu at (166.4, 124.3)
- added C46: 10n, Capacitor_SMD:C_0402_1005Metric, F.Cu at (165.3, 127.1)
- added C47: 10n, Capacitor_SMD:C_0402_1005Metric, F.Cu at (164.2, 131.1)
- added C48: 470n, Capacitor_SMD:C_0402_1005Metric, F.Cu at (162.3, 133.1)
- added C49: 1n, Capacitor_SMD:C_0402_1005Metric, F.Cu at (167.2, 128.3)
- added C5: 10µ, Capacitor_SMD:C_0805_2012Metric, F.Cu at (288.1, 60.8)
- added C50: 1n, Capacitor_SMD:C_0402_1005Metric, F.Cu at (160.4, 135.1)
- added C51: 470n, Capacitor_SMD:C_0402_1005Metric, F.Cu at (167.2, 127.3)
- added C52: 470n, Capacitor_SMD:C_0402_1005Metric, F.Cu at (163.4, 127.1)
- added C53: 470n, Capacitor_SMD:C_0402_1005Metric, F.Cu at (174.2, 116.9)
- added C54: 470n, Capacitor_SMD:C_0402_1005Metric, F.Cu at (163.4, 129.1)
- added C55: 470n, Capacitor_SMD:C_0402_1005Metric, F.Cu at (174.5, 120.1)
- added C56: 470n, Capacitor_SMD:C_0402_1005Metric, F.Cu at (164.2, 130.1)
- added C57: 470n, Capacitor_SMD:C_0402_1005Metric, F.Cu at (175.6, 118.9)
- added C58: 470n, Capacitor_SMD:C_0402_1005Metric, F.Cu at (160.4, 134.1)
- added C59: 1n, Capacitor_SMD:C_0402_1005Metric, F.Cu at (167.2, 126.3)
- added C6: 22µ/25V, Capacitor_SMD:C_1206_3216Metric, F.Cu at (260.9, 67.3)
- added C60: 1n, Capacitor_SMD:C_0402_1005Metric, F.Cu at (172.6, 120.1)
- added C61: 470n, Capacitor_SMD:C_0402_1005Metric, F.Cu at (177.2, 116.4)
- added C62: 10n, Capacitor_SMD:C_0402_1005Metric, F.Cu at (179.1, 115.4)
- added C63: 10n, Capacitor_SMD:C_0402_1005Metric, F.Cu at (165.3, 129.1)
- added C64: 470n, Capacitor_SMD:C_0402_1005Metric, F.Cu at (162.3, 132.1)
- added C65: 10n, Capacitor_SMD:C_0402_1005Metric, F.Cu at (170.2, 123.6)
- added C66: 10n, Capacitor_SMD:C_0402_1005Metric, F.Cu at (177.2, 115.4)
- added C67: 470n, Capacitor_SMD:C_0402_1005Metric, F.Cu at (170.2, 124.6)
- added C68: 100n, Capacitor_SMD:C_0402_1005Metric, F.Cu at (166.4, 125.3)
- added C69: 100n, Capacitor_SMD:C_0402_1005Metric, F.Cu at (162.3, 131.1)
- added C7: 100n, Capacitor_SMD:C_0402_1005Metric, F.Cu at (300.8, 52.8)
- added C70: 470n, Capacitor_SMD:C_0402_1005Metric, F.Cu at (171.0, 122.6)
- added C71: 470n, Capacitor_SMD:C_0402_1005Metric, F.Cu at (165.3, 128.1)
- added C72: 470n, Capacitor_SMD:C_0402_1005Metric, F.Cu at (172.9, 121.1)
- added C73: 470n, Capacitor_SMD:C_0402_1005Metric, F.Cu at (168.3, 123.3)
- added C74: 470n, Capacitor_SMD:C_0402_1005Metric, F.Cu at (172.9, 122.1)
- added C75: 470n, Capacitor_SMD:C_0402_1005Metric, F.Cu at (168.3, 125.3)
- added C76: 470n, Capacitor_SMD:C_0402_1005Metric, F.Cu at (160.4, 130.1)
- added C77: 470n, Capacitor_SMD:C_0402_1005Metric, F.Cu at (162.3, 130.1)
- added C78: 470n, Capacitor_SMD:C_0402_1005Metric, F.Cu at (163.4, 128.1)
- added C79: 470n, Capacitor_SMD:C_0402_1005Metric, F.Cu at (177.5, 117.4)
- added C8: 100n/25V, Capacitor_SMD:C_0805_2012Metric, F.Cu at (283.2, 66.9)
- added C80: 4.7µ, Capacitor_SMD:C_0603_1608Metric, F.Cu at (165.5, 122.1)
- added C81: 4.7µ, Capacitor_SMD:C_0603_1608Metric, F.Cu at (160.9, 127.4)
- added C82: 470n, Capacitor_SMD:C_0402_1005Metric, F.Cu at (171.0, 121.6)
- added C83: 47µ, Capacitor_SMD:C_1210_3225Metric, F.Cu at (170.9, 116.5)
- added C84: 47µ, Capacitor_SMD:C_1210_3225Metric, F.Cu at (161.7, 118.8)
- added C85: 4.7µ, Capacitor_SMD:C_0603_1608Metric, F.Cu at (160.9, 125.9)
- added C86: 47µ, Capacitor_SMD:C_1206_3216Metric, F.Cu at (161.7, 116.0)
- added C87: 470n, Capacitor_SMD:C_0402_1005Metric, F.Cu at (202.3, 129.5)
- added C88: 100n, Capacitor_SMD:C_0402_1005Metric, F.Cu at (209.5, 122.6)
- added C89: 4.7µ, Capacitor_SMD:C_0603_1608Metric, F.Cu at (208.6, 119.3)
- added C9: 1.8n, Capacitor_SMD:C_0402_1005Metric, F.Cu at (301.4, 51.3)
- added C90: 4.7µ, Capacitor_SMD:C_0603_1608Metric, F.Cu at (197.1, 128.6)
- added C91: 470n, Capacitor_SMD:C_0402_1005Metric, F.Cu at (206.6, 126.0)
- added C92: 470n, Capacitor_SMD:C_0402_1005Metric, F.Cu at (202.6, 128.5)
- added C93: 4.7µ, Capacitor_SMD:C_0603_1608Metric, F.Cu at (207.1, 121.8)
- added C94: 470n, Capacitor_SMD:C_0402_1005Metric, F.Cu at (206.6, 124.0)
- added C95: 470n, Capacitor_SMD:C_0402_1005Metric, F.Cu at (211.4, 121.6)
- added C96: 4.7µ, Capacitor_SMD:C_0603_1608Metric, F.Cu at (200.1, 128.3)
- added C97: 470n, Capacitor_SMD:C_0402_1005Metric, F.Cu at (204.7, 125.0)
- added C98: 470n, Capacitor_SMD:C_0402_1005Metric, F.Cu at (206.6, 125.0)
- added C99: 100n, Capacitor_SMD:C_0402_1005Metric, F.Cu at (244.0, 6.87)
- added D1: RED, LED_SMD:LED_0805_2012Metric, F.Cu at (289.5, 57.3)
- added D10: GREEN, LED_SMD:LED_0805_2012Metric, F.Cu at (295.3, 49.5)
- added D11: GREEN, LED_SMD:LED_0805_2012Metric, F.Cu at (284.7, 60.9)
- added D12: GREEN, LED_SMD:LED_0805_2012Metric, F.Cu at (187.1, 128.9)
- added D13: GREEN, LED_SMD:LED_0805_2012Metric, F.Cu at (243.9, 1.42)
- added D14: APHB1608QBDSYKC, Custom Parts:LED_Kingbright_APHB1608, F.Cu at (195.0, 149.0)
- added D15: APHB1608QBDSYKC, Custom Parts:LED_Kingbright_APHB1608, F.Cu at (197.0, 147.9)
- added D16: APHB1608QBDSYKC, Custom Parts:LED_Kingbright_APHB1608, F.Cu at (180.9, 161.7)
- added D17: APHB1608QBDSYKC, Custom Parts:LED_Kingbright_APHB1608, F.Cu at (195.0, 147.9)
- added D18: APHB1608QBDCGKC, Custom Parts:LED_Kingbright_APHB1608, F.Cu at (197.0, 146.8)
- added D19: APHB1608QBDCGKC, Custom Parts:LED_Kingbright_APHB1608, F.Cu at (195.0, 146.8)
- added D2: GREEN, LED_SMD:LED_0805_2012Metric, F.Cu at (279.8, 65.0)
- added D20: APHB1608QBDCGKC, Custom Parts:LED_Kingbright_APHB1608, F.Cu at (196.9, 150.1)
- added D21: APHB1608QBDCGKC, Custom Parts:LED_Kingbright_APHB1608, F.Cu at (192.9, 149.4)
- added D22: APHB1608CGKSURKC, Custom Parts:LED_Kingbright_APHB1608, F.Cu at (192.9, 151.2)
- added D23: APHB1608CGKSURKC, Custom Parts:LED_Kingbright_APHB1608, F.Cu at (190.9, 151.9)
- added D24: APHB1608CGKSURKC, Custom Parts:LED_Kingbright_APHB1608, F.Cu at (197.0, 149.0)
- added D25: APHB1608CGKSURKC, Custom Parts:LED_Kingbright_APHB1608, F.Cu at (194.9, 150.1)
- added D26: GREEN, LED_SMD:LED_0805_2012Metric, F.Cu at (113.8, 115.9)
- added D27: RED, LED_SMD:LED_0805_2012Metric, F.Cu at (81.4, 147.5)
- added D3: MBR15U60, Package_TO_SOT_SMD:TO-277B, F.Cu at (289.9, 45.2)
- added D4: GREEN, LED_SMD:LED_0805_2012Metric, F.Cu at (295.3, 51.5)
- added D5: GREEN, LED_SMD:LED_0805_2012Metric, F.Cu at (264.9, 67.2)
- added D6: GREEN, LED_SMD:LED_0805_2012Metric, F.Cu at (268.4, 67.8)
- added D7: GREEN, LED_SMD:LED_0805_2012Metric, F.Cu at (301.2, 45.9)
- added D8: GREEN, LED_SMD:LED_0805_2012Metric, F.Cu at (279.8, 67.1)
- added D9: GREEN, LED_SMD:LED_0805_2012Metric, F.Cu at (271.8, 67.8)
- added DA1: TPD4E02B04, Custom Parts:USON10, F.Cu at (241.7, 7.04)
- added DA2: TPD4E02B04, Custom Parts:USON10, F.Cu at (225.6, 24.8)
- added DA3: TPD4E02B04, Custom Parts:USON10, F.Cu at (234.7, 14.0)
- added DA4: TPD4E02B04, Custom Parts:USON10, F.Cu at (222.2, 26.8)
- added DA5: TPD4E02B04, Custom Parts:USON10, F.Cu at (300.9, 30.2)
- added DA6: TPD4E02B04, Custom Parts:USON10, F.Cu at (288.6, 36.6)
- added F1: 3A/DNF, Custom Parts:FuseHolder_SMD_Shurter_0031.7701.11, F.Cu at (281.1, 44.3)
- added F2: 3A, Custom Parts:FuseHolder_SMD_Shurter_0031.7701.11, F.Cu at (265.1, 56.0)
- added FB1: 200R@100MHz, Inductor_SMD:L_0603_1608Metric, F.Cu at (247.1, 1.16)
- added FB2: 200R@100MHz, Inductor_SMD:L_0603_1608Metric, F.Cu at (234.9, 12.6)
- added FB3: 200R@100MHz, Inductor_SMD:L_0603_1608Metric, F.Cu at (238.8, 9.08)
- added FB4: 100R, Inductor_SMD:L_0603_1608Metric, F.Cu at (276.7, 36.7)
- added FB5: 100R, Inductor_SMD:L_0603_1608Metric, F.Cu at (273.7, 37.2)
- added FB6: 100R, Inductor_SMD:L_0603_1608Metric, F.Cu at (301.1, 27.2)
- added FB7: 100R, Inductor_SMD:L_0603_1608Metric, F.Cu at (301.1, 25.7)
- added FB8: 100R, Inductor_SMD:L_0603_1608Metric, F.Cu at (298.0, 30.9)
- added FB9: 100R, Inductor_SMD:L_0603_1608Metric, F.Cu at (304.5, 23.8)
- added J1: 12V_EXT, Connector_BarrelJack:BarrelJack_Horizontal, F.Cu at (272.6, 46.1)
- added J10: UART, Connector_PinHeader_2.54mm:PinHeader_1x04_P2.54mm_Vertical, F.Cu at (100.5, 116.7)
- added J11: FLASH, Connector_PinHeader_2.54mm:PinHeader_1x08_P2.54mm_Vertical, F.Cu at (74.2, 134.6)
- added J12: JTAG, Connector_PinHeader_2.54mm:PinHeader_1x06_P2.54mm_Vertical, F.Cu at (77.8, 134.6)
- added J13: Micro_SD_Card, Connector_Card:microSD_HC_Hirose_DM3AT-SF-PEJM5, F.Cu at (299.6, 9.25)
- added J2: USB_B_Micro, Connector_USB:USB_Micro-B_Molex-105017-0001, F.Cu at (202.7, 117.4)
- added J3: HDMI_A, Custom Parts:Molex_HDMI_A_47151-0001, F.Cu at (282.2, 23.3)
- added J4: USB_A, Custom Parts:292303-7, F.Cu at (265.7, 27.4)
- added J5: EXT0, Custom Parts:TE_FPC_40pin_p0.5mm_4-1734839-0, F.Cu at (85.4, 124.4)
- added J6: EXT1, Custom Parts:TE_FPC_40pin_p0.5mm_4-1734839-0, F.Cu at (85.4, 115.4)
- added J7: EXT2, Custom Parts:TE_FPC_40pin_p0.5mm_4-1734839-0, F.Cu at (85.4, 119.9)
- added J8: EXT3, Custom Parts:TE_FPC_40pin_p0.5mm_4-1734839-0, F.Cu at (85.4, 128.9)
- added J9: PMOD_01, Connector_PinHeader_2.54mm:PinHeader_2x15_P2.54mm_Horizontal, F.Cu at (59.2, 116.7)
- added JP1: PRSNT, Connector_PinHeader_2.54mm:PinHeader_1x03_P2.54mm_Vertical, F.Cu at (235.2, 2.23)
- added JP2: CFG1, Connector_PinHeader_2.54mm:PinHeader_1x02_P2.54mm_Vertical, F.Cu at (81.5, 142.1)
- added L1: 800nH/XAL5030, Inductor_SMD:L_Coilcraft_XAL5030, F.Cu at (282.5, 50.3)
- added L10: 100R@100MHz, Inductor_SMD:L_0603_1608Metric, F.Cu at (170.1, 120.4)
- added L11: 100R@100MHz, Inductor_SMD:L_0603_1608Metric, F.Cu at (160.9, 124.3)
- added L12: Ferrite_Bead, Inductor_SMD:L_0603_1608Metric, F.Cu at (199.8, 126.8)
- added L13: Ferrite_Bead, Inductor_SMD:L_0603_1608Metric, F.Cu at (203.6, 123.7)
- added L2: 3.3µH/XAL6030-332, Custom Parts:L_CoilCraft_XAL60xx, F.Cu at (271.3, 63.4)
- added L3: 470n/IHLP1212, Inductor_SMD:L_Vishay_IHLP-1212, F.Cu at (287.8, 50.9)
- added L4: 470n/IHLP1212, Inductor_SMD:L_Vishay_IHLP-1212, F.Cu at (277.0, 61.9)
- added L5: 470n/IHLP1212, Inductor_SMD:L_Vishay_IHLP-1212, F.Cu at (281.9, 55.1)
- added L6: 470n/IHLP1212, Inductor_SMD:L_Vishay_IHLP-1212, F.Cu at (277.0, 49.2)
- added L7: 100R@100MHz, Inductor_SMD:L_0603_1608Metric, F.Cu at (170.1, 118.8)
- added L8: 100R@100MHz, Inductor_SMD:L_0603_1608Metric, F.Cu at (168.5, 122.1)
- added L9: 100R@100MHz, Inductor_SMD:L_0603_1608Metric, F.Cu at (174.7, 115.6)
- added P1: SATA, Custom Parts:Molex_SATA_047080-4001, F.Cu at (225.0, 13.3)
- added P2: SATA, Custom Parts:Molex_SATA_047080-4001, F.Cu at (225.0, 1.40)
- added P3: PCIe_x4_EDGE, Custom Parts:PCIe_EDGE_x4, F.Cu at (110.1, 108.1)
- added P4: JK0654219NL, Custom Parts:Pulse_MagJack_JK0654219NL, F.Cu at (284.8, 9.76)
- added Q1: BSH111BKR, Package_TO_SOT_SMD:SOT-23, F.Cu at (281.3, 58.7)
- added Q2: BC850, Package_TO_SOT_SMD:SOT-23, F.Cu at (281.1, 62.2)
- added Q3: BSH111BKR, Package_TO_SOT_SMD:SOT-23, F.Cu at (297.7, 46.7)
- added Q4: BC850, Package_TO_SOT_SMD:SOT-23, F.Cu at (291.9, 50.9)
- added Q5: BSH111BKR, Package_TO_SOT_SMD:SOT-23, F.Cu at (302.4, 43.0)
- added Q6: BSH111BKR, Package_TO_SOT_SMD:SOT-23, F.Cu at (276.3, 65.5)
- added Q7: BSH111BKR, Package_TO_SOT_SMD:SOT-23, F.Cu at (291.3, 54.5)
- added Q8: BSH111BKR, Package_TO_SOT_SMD:SOT-23, F.Cu at (286.0, 58.1)
- added Q9: BSH111BKR, Package_TO_SOT_SMD:SOT-23, F.Cu at (85.0, 142.0)
- added R1: 1.5k, Resistor_SMD:R_0402_1005Metric, F.Cu at (290.8, 62.9)
- added R10: 10k, Resistor_SMD:R_0402_1005Metric, F.Cu at (288.2, 68.4)
- added R11: 10k, Resistor_SMD:R_0402_1005Metric, F.Cu at (299.8, 56.0)
- added R12: 54.9k, Resistor_SMD:R_0402_1005Metric, F.Cu at (292.7, 62.9)
- added R13: 10k, Resistor_SMD:R_0402_1005Metric, F.Cu at (288.5, 66.4)
- added R14: 470k, Resistor_SMD:R_0402_1005Metric, F.Cu at (306.7, 49.7)
- added R15: 1k, Resistor_SMD:R_0402_1005Metric, F.Cu at (294.2, 59.8)
- added R16: 10k, Resistor_SMD:R_0402_1005Metric, F.Cu at (301.7, 54.8)
- added R17: 1k, Resistor_SMD:R_0402_1005Metric, F.Cu at (290.4, 66.4)
- added R18: 124k, Resistor_SMD:R_0402_1005Metric, F.Cu at (297.8, 58.1)
- added R19: 100k, Resistor_SMD:R_0402_1005Metric, F.Cu at (299.8, 57.0)
- added R2: 1.5k, Resistor_SMD:R_0402_1005Metric, F.Cu at (269.0, 59.5)
- added R20: 453k, Resistor_SMD:R_0402_1005Metric, F.Cu at (304.6, 52.3)
- added R21: 100k, Resistor_SMD:R_0402_1005Metric, F.Cu at (295.4, 61.8)
- added R22: 316k, Resistor_SMD:R_0402_1005Metric, F.Cu at (294.6, 62.8)
- added R23: 100k, Resistor_SMD:R_0402_1005Metric, F.Cu at (295.4, 60.8)
- added R24: 200k, Resistor_SMD:R_0402_1005Metric, F.Cu at (288.5, 67.4)
- added R25: 100k, Resistor_SMD:R_0402_1005Metric, F.Cu at (301.7, 55.8)
- added R26: 10k, Resistor_SMD:R_0402_1005Metric, F.Cu at (299.8, 55.0)
- added R27: 10k, Resistor_SMD:R_0402_1005Metric, F.Cu at (297.3, 60.8)
- added R28: 10k, Resistor_SMD:R_0402_1005Metric, F.Cu at (304.6, 53.3)
- added R29: 10k, Resistor_SMD:R_0402_1005Metric, F.Cu at (305.2, 50.7)
- added R3: 4.7k, Resistor_SMD:R_0402_1005Metric, F.Cu at (302.7, 53.3)
- added R30: 1k, Resistor_SMD:R_0402_1005Metric, F.Cu at (296.1, 59.8)
- added R31: 1k, Resistor_SMD:R_0402_1005Metric, F.Cu at (291.5, 63.9)
- added R32: 1k, Resistor_SMD:R_0402_1005Metric, F.Cu at (291.5, 64.9)
- added R33: 1k, Resistor_SMD:R_0402_1005Metric, F.Cu at (293.4, 63.9)
- added R34: 0R, Resistor_SMD:R_0402_1005Metric, F.Cu at (204.7, 126.0)
- added R35: 0R, Resistor_SMD:R_0402_1005Metric, F.Cu at (198.5, 129.8)
- added R36: 22, Resistor_SMD:R_0402_1005Metric, F.Cu at (206.5, 123.0)
- added R37: 22, Resistor_SMD:R_0402_1005Metric, F.Cu at (209.5, 121.6)
- added R38: 2.2k, Resistor_SMD:R_0402_1005Metric, F.Cu at (204.5, 127.5)
- added R39: 12k, Resistor_SMD:R_0402_1005Metric, F.Cu at (196.6, 129.8)
- added R4: 10, Resistor_SMD:R_0402_1005Metric, F.Cu at (288.7, 58.8)
- added R40: 10k, Resistor_SMD:R_0402_1005Metric, F.Cu at (208.1, 120.5)
- added R41: 10k, Resistor_SMD:R_0402_1005Metric, F.Cu at (200.4, 129.5)
- added R42: 0R, Resistor_SMD:R_0805_2012Metric, F.Cu at (190.5, 128.8)
- added R43: 0R, Resistor_SMD:R_0805_2012Metric, F.Cu at (200.0, 125.1)
- added R44: 0R, Resistor_SMD:R_0805_2012Metric, F.Cu at (193.9, 128.8)
- added R45: 0R, Resistor_SMD:R_0805_2012Metric, F.Cu at (203.8, 122.0)
- added R46: 1.5k, Resistor_SMD:R_0402_1005Metric, F.Cu at (202.6, 127.5)
- added R47: 1k, Resistor_SMD:R_0402_1005Metric, F.Cu at (240.1, 12.0)
- added R48: 4.7k, Resistor_SMD:R_0402_1005Metric, F.Cu at (216.6, 35.8)
- added R49: DNP, Resistor_SMD:R_0402_1005Metric, F.Cu at (238.2, 10.3)
- added R5: 47k, Resistor_SMD:R_0402_1005Metric, F.Cu at (293.5, 60.8)
- added R50: 2.2k, Resistor_SMD:R_0402_1005Metric, F.Cu at (246.6, 2.41)
- added R51: 2.2k, Resistor_SMD:R_0402_1005Metric, F.Cu at (237.3, 12.3)
- added R52: 2.2, Resistor_SMD:R_0402_1005Metric, F.Cu at (216.6, 33.9)
- added R53: 0R, Resistor_SMD:R_0805_2012Metric, F.Cu at (238.7, 7.35)
- added R54: DNP, Resistor_SMD:R_0805_2012Metric, F.Cu at (217.3, 30.4)
- added R55: 0R, Resistor_SMD:R_0805_2012Metric, F.Cu at (222.6, 25.1)
- added R56: DNP, Resistor_SMD:R_0805_2012Metric, F.Cu at (242.1, 5.40)
- added R57: 10k, Resistor_SMD:R_0402_1005Metric, F.Cu at (218.5, 31.9)
- added R58: 0R, Resistor_SMD:R_0402_1005Metric, F.Cu at (221.8, 28.2)
- added R59: 2.2k, Resistor_SMD:R_0402_1005Metric, F.Cu at (316.8, 15.9)
- added R6: 10k, Resistor_SMD:R_0402_1005Metric, F.Cu at (284.4, 68.4)
- added R60: 2.2k, Resistor_SMD:R_0402_1005Metric, F.Cu at (277.0, 22.2)
- added R61: 200k, Resistor_SMD:R_0402_1005Metric, F.Cu at (324.0, 9.55)
- added R62: 510, Resistor_SMD:R_0402_1005Metric, F.Cu at (316.8, 16.8)
- added R63: 1k, Resistor_SMD:R_0402_1005Metric, F.Cu at (275.1, 22.4)
- added R64: 1k, Resistor_SMD:R_0402_1005Metric, F.Cu at (297.4, 34.7)
- added R65: 1k, Resistor_SMD:R_0402_1005Metric, F.Cu at (290.9, 37.7)
- added R66: 1k, Resistor_SMD:R_0402_1005Metric, F.Cu at (303.3, 32.5)
- added R67: 2.2k, Resistor_SMD:R_0402_1005Metric, F.Cu at (280.8, 22.4)
- added R68: 2.2k, Resistor_SMD:R_0402_1005Metric, F.Cu at (282.8, 22.4)
- added R69: 10k, Resistor_SMD:R_0402_1005Metric, F.Cu at (284.7, 22.4)
- added R7: 1k, Resistor_SMD:R_0402_1005Metric, F.Cu at (297.8, 57.1)
- added R70: 10k, Resistor_SMD:R_0402_1005Metric, F.Cu at (278.9, 22.4)
- added R71: 12.1k, Resistor_SMD:R_0402_1005Metric, F.Cu at (321.9, 10.1)
- added R72: 1M, Resistor_SMD:R_0402_1005Metric, F.Cu at (292.8, 37.0)
- added R73: 1k, Resistor_SMD:R_0402_1005Metric, F.Cu at (299.5, 32.2)
- added R74: 120k, Resistor_SMD:R_0402_1005Metric, F.Cu at (324.0, 8.56)
- added R75: 51, Resistor_SMD:R_0402_1005Metric, F.Cu at (160.0, 155.2)
- added R76: 51, Resistor_SMD:R_0402_1005Metric, F.Cu at (158.7, 157.2)
- added R77: 10k, Resistor_SMD:R_0402_1005Metric, F.Cu at (156.8, 159.2)
- added R78: 10k, Resistor_SMD:R_0402_1005Metric, F.Cu at (153.0, 163.8)
- added R79: 10k, Resistor_SMD:R_0402_1005Metric, F.Cu at (162.3, 153.3)
- added R8: 10k, Resistor_SMD:R_0402_1005Metric, F.Cu at (286.3, 68.4)
- added R80: 240, Resistor_SMD:R_0402_1005Metric, F.Cu at (151.1, 162.8)
- added R81: 240, Resistor_SMD:R_0402_1005Metric, F.Cu at (153.0, 162.8)
- added R82: 0R, Resistor_SMD:R_0805_2012Metric, F.Cu at (91.4, 137.7)
- added R83: DNP, Resistor_SMD:R_0805_2012Metric, F.Cu at (104.0, 122.6)
- added R84: DNP, Resistor_SMD:R_0805_2012Metric, F.Cu at (94.8, 133.8)
- added R85: 0R, Resistor_SMD:R_0805_2012Metric, F.Cu at (77.7, 150.1)
- added R86: DNP, Resistor_SMD:R_0805_2012Metric, F.Cu at (91.4, 135.7)
- added R87: DNP, Resistor_SMD:R_0805_2012Metric, F.Cu at (91.4, 133.8)
- added R88: 4.7k, Resistor_SMD:R_0402_1005Metric, F.Cu at (97.1, 135.3)
- added R89: 1k, Resistor_SMD:R_0402_1005Metric, F.Cu at (113.0, 119.4)
- added R9: 4.7k, Resistor_SMD:R_0402_1005Metric, F.Cu at (300.8, 53.8)
- added R90: 10k, Resistor_SMD:R_0402_1005Metric, F.Cu at (116.4, 116.4)
- added R91: 22, Resistor_SMD:R_0402_1005Metric, F.Cu at (114.9, 117.4)
- added R92: 1k, Resistor_SMD:R_0402_1005Metric, F.Cu at (80.0, 151.6)
- added R93: 1k, Resistor_SMD:R_0402_1005Metric, F.Cu at (102.6, 130.6)
- added R94: 10k, Resistor_SMD:R_0402_1005Metric, F.Cu at (77.0, 153.1)
- added R95: 10k, Resistor_SMD:R_0402_1005Metric, F.Cu at (99.6, 133.1)
- added R96: 10k, Resistor_SMD:R_0402_1005Metric, F.Cu at (311.9, 22.6)
- added R97: 22, Resistor_SMD:R_0402_1005Metric, F.Cu at (60.3, 154.6)
- added RN1: 10k, Resistor_SMD:R_Array_Convex_4x0402, F.Cu at (295.6, 55.9)
- added RN10: 2.2k, Resistor_SMD:R_Array_Convex_4x0402, F.Cu at (168.7, 161.7)
- added RN11: 1k, Resistor_SMD:R_Array_Convex_4x0402, F.Cu at (176.9, 162.5)
- added RN12: 10k, Resistor_SMD:R_Array_Convex_4x0402, F.Cu at (193.1, 147.6)
- added RN13: 2.2k, Resistor_SMD:R_Array_Convex_4x0402, F.Cu at (191.0, 150.1)
- added RN14: 2.2k, Resistor_SMD:R_Array_Convex_4x0402, F.Cu at (174.9, 162.5)
- added RN15: 2.2k, Resistor_SMD:R_Array_Convex_4x0402, F.Cu at (179.0, 162.5)
- added RN16: 51, Resistor_SMD:R_Array_Convex_4x0402, F.Cu at (158.4, 151.9)
- added RN17: 51, Resistor_SMD:R_Array_Convex_4x0402, F.Cu at (160.4, 149.5)
- added RN18: 51, Resistor_SMD:R_Array_Convex_4x0402, F.Cu at (162.7, 147.6)
- added RN19: 51, Resistor_SMD:R_Array_Convex_4x0402, F.Cu at (155.0, 155.4)
- added RN2: 10k, Resistor_SMD:R_Array_Convex_4x0402, F.Cu at (202.7, 125.8)
- added RN20: 51, Resistor_SMD:R_Array_Convex_4x0402, F.Cu at (149.1, 162.6)
- added RN21: 51, Resistor_SMD:R_Array_Convex_4x0402, F.Cu at (158.0, 154.5)
- added RN22: 10k, Resistor_SMD:R_Array_Convex_4x0402, F.Cu at (84.3, 146.6)
- added RN23: 10k, Resistor_SMD:R_Array_Convex_4x0402, F.Cu at (87.8, 143.0)
- added RN24: 10k, Resistor_SMD:R_Array_Convex_4x0402, F.Cu at (322.0, 8.35)
- added RN3: R_Pack04, Resistor_SMD:R_Array_Convex_4x0402, F.Cu at (211.2, 119.8)
- added RN4: 10k, Resistor_SMD:R_Array_Convex_4x0402, F.Cu at (297.5, 33.0)
- added RN5: 10k, Resistor_SMD:R_Array_Convex_4x0402, F.Cu at (303.6, 27.8)
- added RN6: 10k, Resistor_SMD:R_Array_Convex_4x0402, F.Cu at (307.1, 25.4)
- added RN7: 1k, Resistor_SMD:R_Array_Convex_4x0402, F.Cu at (170.8, 161.7)
- added RN8: 10k, Resistor_SMD:R_Array_Convex_4x0402, F.Cu at (191.0, 147.6)
- added RN9: 10k, Resistor_SMD:R_Array_Convex_4x0402, F.Cu at (172.8, 161.7)
- added SW1: CHP-081TA, Custom Parts:DipSW_CHP-081TA, F.Cu at (173.8, 149.6)
- added SW2: SW_Push, Button_Switch_SMD:SW_SPST_B3S-1000, F.Cu at (192.8, 157.5)
- added SW3: SW_Push, Button_Switch_SMD:SW_SPST_B3S-1000, F.Cu at (182.8, 157.5)
- added SW4: SW_Push, Button_Switch_SMD:SW_SPST_B3S-1000, F.Cu at (185.0, 150.0)
- added SW5: SW_Push, Button_Switch_SMD:SW_SPST_B3S-1000, F.Cu at (172.7, 156.7)
- added SW6: SW_Push, Button_Switch_SMD:SW_SPST_B3S-1000, F.Cu at (84.7, 136.5)
- added TP1: DCU1_CLK+, TestPoint:TestPoint_Pad_1.5x1.5mm, F.Cu at (234.6, 16.3)
- added TP2: DCU1_CLK-, TestPoint:TestPoint_Pad_1.5x1.5mm, F.Cu at (241.7, 9.29)
- added U1: MAX811MEUS-T, Package_TO_SOT_SMD:SOT-143, F.Cu at (287.5, 54.5)
- added U10: TPS62823, Custom Parts:TI_VSON-HR_1.5x2mm_p0.5mm, F.Cu at (297.9, 55.6)
- added U12: 93AA46B_OT, Package_TO_SOT_SMD:SOT-23-6, F.Cu at (209.1, 116.7)
- added U13: FT2232H, Package_QFP:LQFP-64_10x10mm_P0.5mm, F.Cu at (191.8, 121.4)
- added U14: XUL535150.000JS6I8, Custom Parts:OSC_IDT_XU_5x3.2mm, F.Cu at (239.6, 2.15)
- added U15: ECP5UM5G_85_CABGA756, Custom Parts:CABGA756_27x27mm_p0.8mm, F.Cu at (145.6, 128.7)
- added U16: 5P49V6965, Package_DFN_QFN:QFN-24-1EP_4x4mm_P0.5mm_EP2.7x2.7mm, F.Cu at (218.2, 26.8)
- added U17: TPS2041B, Package_TO_SOT_SMD:SOT-23-5, F.Cu at (288.5, 20.9)
- added U18: PCA9306, Package_SO:VSSOP-8_2.3x2mm_P0.5mm, F.Cu at (276.4, 20.4)
- added U19: TFP410, Package_QFP:HTQFP-64-1EP_10x10mm_P0.5mm_EP8x8mm_Mask4.4x4.4mm_ThermalVias, F.Cu at (314.2, 7.13)
- added U2: LM3880, Package_TO_SOT_SMD:SOT-23-6, F.Cu at (294.1, 46.3)
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Other:
- outline, holes or cut-outs redrawn

Commit message: hardware/mainboard: Preliminary placement of some major components
Signed-off-by: David Shah <dave@ds0.me>
Parts:
- RN13, RN15, RN7, RN8: moved to B.Cu
- moved U19 259.5 mm to (69.0, 92.0), turned to 270 degrees
- moved R97 252.7 mm to (307.2, 100.8)
- moved C214 247.0 mm to (303.9, 103.5)
- moved C226 245.0 mm to (299.0, 108.5)
- moved U21 241.4 mm to (87.9, 108.6)
- moved P4 241.0 mm to (66.4, 111.6)
- moved J3 239.8 mm to (51.9, 90.4), turned to 270 degrees
- moved C249 238.2 mm to (300.9, 105.1)
- moved RN12 233.3 mm to (425.4, 126.5)
- moved C236 232.4 mm to (310.6, 96.8)
- moved C242 226.8 mm to (302.0, 106.0)
- moved U22 226.0 mm to (71.0, 74.0)
- moved U18 226.0 mm to (59.0, 82.0), turned to 180 degrees
- moved C237 225.8 mm to (307.2, 98.8)
- moved C219 225.3 mm to (298.0, 105.8)
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Other:
- outline, holes or cut-outs redrawn

Commit message: hardware/mainboard: Power related placement
Signed-off-by: David Shah <dave@ds0.me>
Parts:
- added C256: 47µ, Capacitor_SMD:C_1210_3225Metric, F.Cu at (191.0, 99.5)
- RN12, U13: moved to B.Cu
- moved U17 256.9 mm to (65.9, 82.0)
- moved C137 243.7 mm to (66.0, 65.0)
- moved RN12 239.0 mm to (196.8, 57.0), turned to 90 degrees
- moved C33 225.8 mm to (135.0, 86.5)
- moved C84 221.0 mm to (135.0, 90.0)
- moved C12 189.0 mm to (186.5, 98.5), turned to 270 degrees
- moved JP2 188.1 mm to (91.0, 88.0), turned to 270 degrees
- moved C11 187.4 mm to (183.5, 101.0), turned to 90 degrees
- moved L4 186.0 mm to (158.0, 110.5), turned to 90 degrees
- moved R11 180.6 mm to (188.0, 101.0), turned to 270 degrees
- moved R9 176.9 mm to (186.0, 103.0), turned to 180 degrees
- moved R14 175.8 mm to (186.5, 101.0), turned to 270 degrees
- moved R5 173.3 mm to (203.5, 100.0), turned to 180 degrees
- moved R10 171.8 mm to (188.0, 98.5), turned to 270 degrees
- moved C9 170.7 mm to (185.0, 101.0), turned to 90 degrees
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
Commit message: hardware/mainboard: Power circuitry placed
Signed-off-by: David Shah <dave@ds0.me>
Parts:
- removed D1: RED, LED_SMD:LED_0805_2012Metric
- removed R1: 1.5k, Resistor_SMD:R_0402_1005Metric
- moved R7 228.9 mm to (139.5, 117.0), turned to 270 degrees
- moved R6 220.7 mm to (141.0, 111.5)
- moved R17 214.4 mm to (146.5, 117.0), turned to 270 degrees
- moved D5 214.0 mm to (142.1, 118.0)
- moved Q2 212.6 mm to (141.0, 114.0), turned to 270 degrees
- moved Q4 210.2 mm to (148.0, 114.0), turned to 270 degrees
- moved R15 207.3 mm to (160.0, 117.0), turned to 90 degrees
- moved D6 205.1 mm to (156.0, 118.0)
- moved D7 203.2 mm to (149.1, 118.0)
- moved Q7 202.4 mm to (161.1, 114.0), turned to 270 degrees
- moved C5 199.6 mm to (174.0, 100.1), turned to 270 degrees
- moved R33 199.6 mm to (171.5, 117.0), turned to 270 degrees
- moved R16 190.0 mm to (148.0, 111.5)
- moved C27 189.7 mm to (192.5, 74.5), turned to 90 degrees
- moved R32 189.3 mm to (165.0, 117.0), turned to 270 degrees
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Other:
- board text added: "12V"
- board text added: "1V2"
- board text added: "1V2A"
- board text added: "1V2T"
- board text added: "1V35"
- board text added: "1V8"
- board text added: "2V5"
- board text added: "3V3"
- board text added: "5V0"

Commit message: hardware/mainboard: Change LEDs to larger Wurth 3528 LEDs
Signed-off-by: David Shah <dave@ds0.me>
Parts:
- D14, D15, D16, D17: value APHB1608QBDSYKC -> 150141YB73100; footprint Custom Parts:LED_Kingbright_APHB1608 -> Custom Parts:Wurth_BiLED_150141_3528
- D18, D19: value APHB1608QBDCGKC -> 150141YB73100; footprint Custom Parts:LED_Kingbright_APHB1608 -> Custom Parts:Wurth_BiLED_150141_3528
- D20, D21: value APHB1608QBDCGKC -> 150141RV73100; footprint Custom Parts:LED_Kingbright_APHB1608 -> Custom Parts:Wurth_BiLED_150141_3528
- D22, D23, D24, D25: value APHB1608CGKSURKC -> 150141RV73100; footprint Custom Parts:LED_Kingbright_APHB1608 -> Custom Parts:Wurth_BiLED_150141_3528
- RN11, RN7: value 1k -> 2.2k
- moved D19 25.9 mm to (209.0, 38.0)
- moved D24 19.6 mm to (209.0, 44.0)
- moved D18 17.1 mm to (203.0, 38.0)
- moved RN13 16.7 mm to (201.0, 40.0)
- moved RN15 11.0 mm to (194.0, 40.0)
- moved D20 10.6 mm to (179.0, 44.0)
- moved D23 10.6 mm to (197.0, 44.0)
- moved D25 10.6 mm to (203.0, 44.0)
- moved D21 7.65 mm to (185.0, 44.0)
- moved D22 7.65 mm to (191.0, 44.0)
- moved D14 4.74 mm to (179.0, 38.0)
- moved D17 4.74 mm to (197.0, 38.0)
- moved RN7 2.55 mm to (187.0, 40.0)
- moved D15 2.12 mm to (185.0, 38.0)
- moved D16 2.12 mm to (191.0, 38.0)
