File: hardware/ecp5_mainboard/ecp5_mainboard.kicad_pcb (KiCad board)
At the start: 2 copper layers, 158.1 x 111.2 mm, 498 parts, among them J1 12V_EXT, J10 UART, J11 FLASH, J12 JTAG, J13 Micro_SD_Card, J2 USB_B_Micro, J3 HDMI_A, J4 USB_A, J5 EXT0, J6 EXT1, J7 EXT2, J8 EXT3, J9 PMOD_01, P1 SATA, P2 SATA, P3 PCIe_x4_EDGE, P4 JK0654219NL, Q1 BSH111BKR, Q2 BC850, Q3 BSH111BKR, Q4 BC850, Q5 BSH111BKR, Q6 BSH111BKR, Q7 BSH111BKR, Q8 BSH111BKR, Q9 BSH111BKR, SW1 CHP-081TA, SW2 SW_Push, SW3 SW_Push, SW4 SW_Push, SW5 SW_Push, SW6 SW_Push, U1 MAX811MEUS-T, U10 TPS62823, U12 93AA46B_OT, U13 FT2232H, U14 XUL535150.000JS6I8, U15 ECP5UM5G_85_CABGA756, U16 5P49V6965, U17 TPS2041B, U18 PCA9306, U19 TFP410, U2 LM3880, U20 TPS2041B, U21 KSZ9031RNXCA, U22 USB3300-EZK, U23 AS4C256M16D3, U24 AS4C256M16D3, U25 TPS51200DRC, U26 XL_XO_LVDS, U27 W25Q, U3 TLV75712PDR, U4 TPS565208, U5 LM21212-2, U6 TLV75712PDR, U7 TPS62823, U8 TPS62823, U9 TPS62823, X1 XO32, Y1 25MHz, Y2 25MHz, Y3 24MHz

Commit message: hardware/mainboard: Complete 3D models, other footprint tweaks
Signed-off-by: David Shah <dave@ds0.me>
Parts:
- moved C18 1.00 mm to (215.0, 71.0)
- moved C22 1.00 mm to (209.5, 70.5)
- moved C26 1.00 mm to (207.5, 74.0)
- moved C30 1.00 mm to (205.5, 74.0)
- moved L6 1.00 mm to (211.0, 74.0)
- moved R24 1.00 mm to (209.5, 71.5)
- moved R25 1.00 mm to (209.5, 69.5)
- moved R29 1.00 mm to (215.0, 67.5)
- moved U10 1.00 mm to (212.0, 70.5)

Commit message: hardware/mainboard: Reduce refdes size to 0.8mm
Signed-off-by: David Shah <dave@ds0.me>
Parts:
- moved C15 0.50 mm to (201.5, 71.0)
- moved C19 0.50 mm to (196.0, 70.5)
- moved C23 0.50 mm to (194.5, 74.0)
- moved C27 0.50 mm to (192.5, 74.0)
- moved L3 0.50 mm to (198.0, 74.0)
- moved R18 0.50 mm to (196.0, 71.5)
- moved R19 0.50 mm to (196.0, 69.5)
- moved R28 0.50 mm to (201.5, 68.5)
- moved U7 0.50 mm to (198.5, 71.0)

Commit message: hardware/mainboard: Tidy up silkscreen
Signed-off-by: David Shah <dave@ds0.me>
Parts:
- moved C219 3.80 mm to (142.5, 74.5)
- moved C37 0.75 mm to (119.7, 86.7)
- moved C80 0.75 mm to (121.4, 86.7)
- moved C5 0.70 mm to (148.0, 100.9)
- turned RN17 to 0 degrees

Commit message: hardware/mainboard: Small design tweaks
Signed-off-by: David Shah <dave@ds0.me>
Parts:
- added TP10: 2.5V, TestPoint:TestPoint_THTPad_1.5x1.5mm_Drill0.7mm, F.Cu at (185.0, 80.5)
- added TP11: 1.35V, TestPoint:TestPoint_THTPad_1.5x1.5mm_Drill0.7mm, F.Cu at (185.0, 70.0)
- added TP12: 1.8V, TestPoint:TestPoint_THTPad_1.5x1.5mm_Drill0.7mm, F.Cu at (214.0, 66.5)
- added TP3: 1.2VA, TestPoint:TestPoint_THTPad_1.5x1.5mm_Drill0.7mm, F.Cu at (146.0, 87.5)
- added TP4: 1.2V, TestPoint:TestPoint_THTPad_1.5x1.5mm_Drill0.7mm, F.Cu at (108.0, 49.5)
- added TP5: 5V, TestPoint:TestPoint_THTPad_1.5x1.5mm_Drill0.7mm, F.Cu at (197.5, 91.5)
- added TP6: GND, TestPoint:TestPoint_THTPad_1.5x1.5mm_Drill0.7mm, F.Cu at (111.0, 49.5)
- added TP7: GND, TestPoint:TestPoint_THTPad_1.5x1.5mm_Drill0.7mm, F.Cu at (181.5, 75.0)
- added TP8: 1.2VT, TestPoint:TestPoint_THTPad_1.5x1.5mm_Drill0.7mm, F.Cu at (146.0, 91.5)
- added TP9: 3.3V, TestPoint:TestPoint_THTPad_1.5x1.5mm_Drill0.7mm, F.Cu at (214.0, 79.0)
- C144, C145, C146, C148, C149, C150, C152, C153, C154, C155, C157, C158, C160: footprint Capacitor_SMD:C_0402_1005Metric -> Capacitor_SMD:C_0201_0603Metric
- moved C182 16.2 mm to (192.0, 91.0), turned to 270 degrees
- moved L10 4.95 mm to (140.4, 88.2)
- moved L7 4.95 mm to (140.4, 86.6)
- moved L8 4.95 mm to (140.4, 91.4)
- moved L9 4.95 mm to (140.4, 89.8)
- moved C15 4.61 mm to (197.0, 70.0)
- moved C16 4.61 mm to (210.5, 82.1)
- moved C17 4.61 mm to (196.5, 80.6)
- moved C18 4.61 mm to (210.5, 70.0)
- moved C19 4.61 mm to (191.5, 69.5)
- moved C20 4.61 mm to (205.0, 82.0)
- moved C21 4.61 mm to (191.0, 80.5)
- moved C22 4.61 mm to (205.0, 69.5)
- moved C23 4.61 mm to (190.0, 73.0)
- moved C24 4.61 mm to (201.0, 84.5)
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
Commit message: hardware/mainboard: Set up layers and design rules
Signed-off-by: David Shah <dave@ds0.me>
Other:
- copper layers 2 -> 8
- net class Default: clearance 0.2 -> 0.0889; trace_width 0.25 -> 0.0889; via_dia 0.8 -> 0.4; via_drill 0.4 -> 0.2
- rule trace_clearance: 0.2 -> 0.0889
- rule trace_min: 0.2 -> 0.0889
- rule via_min_drill: 0.3 -> 0.2
Changed lines of the file:
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@@
   (layers
     (0 F.Cu signal)
+    (1 In1.Cu signal)
+    (2 In2.Cu signal)
+    (3 In3.Cu signal)
+    (4 In4.Cu signal)
+    (5 In5.Cu signal)
+    (6 In6.Cu signal)
     (31 B.Cu signal)
     (32 B.Adhes user)
@@
   )
   (setup
-    (last_trace_width 0.25)
-    (trace_clearance 0.2)
+    (last_trace_width 0.0889)
+    (user_trace_width 0.1)
+    (user_trace_width 0.15)
+    (user_trace_width 0.2)
+    (user_trace_width 0.25)
+    (user_trace_width 0.35)
+    (user_trace_width 0.5)
+    (user_trace_width 0.8)
+    (user_trace_width 1)
+    (trace_clearance 0.0889)
     (zone_clearance 0.508)
     (zone_45_only no)
-    (trace_min 0.2)
+    (trace_min 0.0889)
     (segment_width 0.2)
     (edge_width 0.15)
-    (via_size 0.8)
-    (via_drill 0.4)
+    (via_size 0.4)
+    (via_drill 0.2)
     (via_min_size 0.4)
-    (via_min_drill 0.3)
+    (via_min_drill 0.2)
+    (user_via 0.6 0.3)
+    (user_via 0.8 0.5)
+    (user_via 1 0.6)
+    (user_via 1.5 1)
+    (user_via 2 1.5)
     (uvia_size 0.3)
     (uvia_drill 0.1)
@@
   (net 718 "Net-(J2-Pad4)")
   (net_class Default "This is the default net class."
-    (clearance 0.2)
-    (trace_width 0.25)
-    (via_dia 0.8)
-    (via_drill 0.4)
+    (clearance 0.0889)
+    (trace_width 0.0889)
+    (via_dia 0.4)
+    (via_drill 0.2)
     (uvia_dia 0.3)
     (uvia_drill 0.1)

Commit message: hardware/mainboard: Creating power/ground planes
Signed-off-by: David Shah <dave@ds0.me>
Routing:
- net +1V35: track 0.00 -> 1.79 mm, vias 0 -> 1
- added copper zone on In4.Cu, net +1V2
- added copper zone on In3.Cu, net +1V35
- added copper zone on In3.Cu, net +3V3
- added copper zone on B.Cu, net GND
- added copper zone on In1.Cu, net GND
- added copper zone on In6.Cu, net GND
Changed lines of the file:
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@@
     (thickness 1.6)
     (drawings 12)
-    (tracks 0)
+    (tracks 7)
     (zones 0)
     (modules 508)
@@
     (user_trace_width 1)
     (trace_clearance 0.0889)
-    (zone_clearance 0.508)
+    (zone_clearance 0.254)
     (zone_45_only no)
     (trace_min 0.0889)
@@
   (gr_line (start 240.25 23.75) (end 240.25 122.15) (layer Edge.Cuts) (width 0.15))
   (gr_line (start 198.3 23.75) (end 240.25 23.75) (layer Edge.Cuts) (width 0.15))
+  (via (at 161.75 75.9) (size 0.4) (drill 0.2) (layers F.Cu B.Cu) (net 195))
+  (segment (start 162.1 76.2) (end 162.05 76.2) (width 0.0889) (layer F.Cu) (net 195))
+  (segment (start 162.05 76.2) (end 161.75 75.9) (width 0.0889) (layer F.Cu) (net 195))
+  (segment (start 161.75 75.935) (end 161.285 76.4) (width 0.0889) (layer B.Cu) (net 195))
+  (segment (start 161.75 75.9) (end 161.75 75.935) (width 0.0889) (layer B.Cu) (net 195))
+  (segment (start 161.715 75.9) (end 161.3 75.485) (width 0.0889) (layer B.Cu) (net 195))
+  (segment (start 161.75 75.9) (end 161.715 75.9) (width 0.0889) (layer B.Cu) (net 195))
+  (zone (net 24) (net_name GND) (layer In1.Cu) (hatch edge 0.508)
+    (connect_pads (clearance 0.254))
+    (min_thickness 0.254)
+    (fill yes (arc_segments 16) (thermal_gap 0.508) (thermal_bridge_width 0.508))
+    (polygon
+      (pts
+        (xy 35 140) (xy 35 20) (xy 245 20) (xy 245 140)
+      )
+    )
+  )
+  (zone (net 24) (net_name GND) (layer In6.Cu) (hatch edge 0.508)
+    (connect_pads (clearance 0.254))
+    (min_thickness 0.254)
+    (fill yes (arc_segments 16) (thermal_gap 0.508) (thermal_bridge_width 0.508))
+    (polygon
+      (pts
+        (xy 246 141) (xy 34 141) (xy 34 19) (xy 246 19)
+      )
+    )
+  )
+  (zone (net 24) (net_name GND) (layer B.Cu) (hatch edge 0.508)
+    (connect_pads (clearance 0.254))
+    (min_thickness 0.254)
+    (fill yes (arc_segments 16) (thermal_gap 0.508) (thermal_bridge_width 0.508))
+    (polygon
+      (pts
+        (xy 247 18) (xy 33 18) (xy 33 142) (xy 247 142)
+      )
+    )
+  )
+  (zone (net 196) (net_name +1V2) (layer In4.Cu) (hatch edge 0.508)
+    (connect_pads (clearance 0.254))
+    (min_thickness 0.254)
+    (fill yes (arc_segments 16) (thermal_gap 0.508) (thermal_bridge_width 0.508))
+    (polygon
+      (pts
+        (xy 130.5 75) (xy 105 75) (xy 105 47) (xy 130.5 47)
+      )
+    )
+  )
+  (zone (net 195) (net_name +1V35) (layer In3.Cu) (hatch edge 0.508)
+    (priority 2)
+    (connect_pads (clearance 0.254))
+    (min_thickness 0.254)
+    (fill yes (arc_segments 16) (thermal_gap 0.508) (thermal_bridge_width 0.508))
+    (polygon
+      (pts
+        (xy 178.5 95.75) (xy 190.75 95.75) (xy 190.75 87.25) (xy 183.25 87.25) (xy 183.25 62.25)
+        (xy 151 62.25) (xy 151 57.25) (xy 132.75 57.25) (xy 132.75 61.75) (xy 132 61.75)
+        (xy 132 63.75) (xy 130.5 63.75) (xy 130.5 65.5) (xy 128.5 65.5) (xy 128.5 73.75)
+        (xy 131 73.75) (xy 131 77.75) (xy 137.375 77.75) (xy 143.25 77.75) (xy 143.25 82.75)
+        (xy 155.5 82.75) (xy 155.5 102.75) (xy 178.5 102.75)
+      )
+    )
+  )
+  (zone (net 12) (net_name +3V3) (layer In3.Cu) (hatch edge 0.508)
+    (connect_pads (clearance 0.254))
+    (min_thickness 0.254)
+    (fill yes (arc_segments 16) (thermal_gap 0.508) (thermal_bridge_width 0.508))
+    (polygon
+      (pts
+        (xy 43 27) (xy 43 42) (xy 43 119) (xy 58 119) (xy 116 119)
+        (xy 225 119) (xy 225 105) (xy 237 105) (xy 237 27)
+      )
+    )
+  )
 )

Commit message: hardware/mainboard: FPGA power/ground routing
Signed-off-by: David Shah <dave@ds0.me>
Parts:
- turned C60 to 90 degrees
- turned C65 to 0 degrees
- turned C75 to 0 degrees
- turned C82 to 270 degrees
Routing:
- net GND: track 0.00 -> 175.8 mm, vias 0 -> 208
- net +1V2: track 0.00 -> 33.8 mm, vias 0 -> 34
- net /FPGA Core Power/VCCAUX: track 0.00 -> 14.5 mm, vias 0 -> 11
- net /FPGA Core Power/VCCA1: track 0.00 -> 13.2 mm, vias 0 -> 11
- net /FPGA Core Power/VCCA0: track 0.00 -> 12.6 mm, vias 0 -> 10
- net +1V35: track 1.79 -> 12.5 mm, vias 1 -> 9
- net +3V3: track 0.00 -> 7.28 mm, vias 0 -> 5
- net /FPGA IO/VCCIO7: track 0.00 -> 6.81 mm, vias 0 -> 4
- net /FPGA IO/VCCIO6: track 0.00 -> 6.59 mm, vias 0 -> 3
- net /FPGA Core Power/VCCHTX0: track 0.00 -> 1.94 mm, vias 0 -> 2
- net /FPGA Core Power/VCCHTX1: track 0.00 -> 1.76 mm, vias 0 -> 2

Commit message: hardware/mainboard: Tidying up
Signed-off-by: David Shah <dave@ds0.me>
Parts:
- moved C175 8.06 mm to (168.2, 82.2)
- moved C177 8.06 mm to (164.7, 92.4)
- moved C180 8.06 mm to (175.0, 60.0)
- moved C183 8.06 mm to (175.2, 88.6)
- moved C184 8.06 mm to (171.5, 71.4)
- moved C185 8.06 mm to (168.7, 68.3)
- moved C186 8.06 mm to (163.4, 68.7)
- moved C187 8.06 mm to (161.8, 67.8)
- moved C188 8.06 mm to (159.8, 68.4)
- moved C189 8.06 mm to (168.7, 79.3)
- moved C190 8.06 mm to (160.6, 79.2)
- moved C191 8.06 mm to (160.3, 84.2)
- moved C192 8.06 mm to (171.1, 61.8)
- moved C193 8.06 mm to (159.2, 79.7)
- moved C194 8.06 mm to (159.5, 62.2)
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Connections:
- U15 pad K26: DDR3_DQ7 -> Net-(U15-PadK26)
- U15 pad K28: DDR3_DM0 -> Net-(U15-PadK28)
- U15 pad L26: DDR3_DQ5 -> Net-(U15-PadL26)
- U15 pad L27: DDR3_DQ4 -> Net-(U15-PadL27)
- U15 pad L29: DDR3_DQ6 -> Net-(U15-PadL29)
- U15 pad N26: DDR3_DQ1 -> Net-(U15-PadN26)
- U15 pad N27: DDR3_DQ3 -> Net-(U15-PadN27)
- U15 pad P26: DDR3_DQ0 -> Net-(U15-PadP26)
- U15 pad P27: DDR3_DQ2 -> Net-(U15-PadP27)
Other:
- board text added: "3A"
- board text added: "3A PCIe Power"
- board text added: "ACT"
- board text added: "DONE"
- board text added: "David Shah"
- board text added: "PROG"
- board text added: "Rev 1.0 (Nov 18)"
- board text added: "TrellisBoard"
- board text added: "~INIT"
