File: hardware/ecp5_mainboard/miscio.sch (KiCad schematic (older format))
At the start: 26 parts, among them SW1 CHP-081TA, SW2 SW_Push, SW3 SW_Push, SW4 SW_Push, SW5 SW_Push

Commit message: hardware/mainboard: Assign more footprints
Signed-off-by: David Shah <dave@ds0.me>
Parts:
- SW2, SW3, SW4, SW5: footprint (none) -> Button_Switch_SMD:SW_SPST_B3S-1000
Changed lines of the file:
@@
 F 0 "SW2" H 4750 4735 50  0000 C CNN
 F 1 "SW_Push" H 4750 4644 50  0000 C CNN
-F 2 "" H 4750 4650 50  0001 C CNN
+F 2 "Button_Switch_SMD:SW_SPST_B3S-1000" H 4750 4650 50  0001 C CNN
 F 3 "" H 4750 4650 50  0001 C CNN
 	1    4750 4450
@@
 F 0 "SW3" H 4750 5085 50  0000 C CNN
 F 1 "SW_Push" H 4750 4994 50  0000 C CNN
-F 2 "" H 4750 5000 50  0001 C CNN
+F 2 "Button_Switch_SMD:SW_SPST_B3S-1000" H 4750 5000 50  0001 C CNN
 F 3 "" H 4750 5000 50  0001 C CNN
 	1    4750 4800
@@
 F 0 "SW4" H 4750 5435 50  0000 C CNN
 F 1 "SW_Push" H 4750 5344 50  0000 C CNN
-F 2 "" H 4750 5350 50  0001 C CNN
+F 2 "Button_Switch_SMD:SW_SPST_B3S-1000" H 4750 5350 50  0001 C CNN
 F 3 "" H 4750 5350 50  0001 C CNN
 	1    4750 5150
@@
 F 0 "SW5" H 4750 5835 50  0000 C CNN
 F 1 "SW_Push" H 4750 5744 50  0000 C CNN
-F 2 "" H 4750 5750 50  0001 C CNN
+F 2 "Button_Switch_SMD:SW_SPST_B3S-1000" H 4750 5750 50  0001 C CNN
 F 3 "" H 4750 5750 50  0001 C CNN
 	1    4750 5550

Commit message: hardware/mainboard: More footprint assignment, other small tweaks
Signed-off-by: David Shah <dave@ds0.me>
Parts:
- D14, D15, D16, D17, D18, D19, D20, D21, D22, D23, D24, D25: footprint (none) -> Custom Parts:LED_Kingbright_APHB1608
- SW1: footprint (none) -> Custom Parts:DipSW_CHP-081TA
Changed lines of the file:
@@
 F 0 "D14" H 2400 1375 50  0000 C CNN
 F 1 "APHB1608QBDSYKC" H 2400 1284 50  0000 C CNN
-F 2 "" H 2430 950 50  0001 C CNN
+F 2 "Custom Parts:LED_Kingbright_APHB1608" H 2430 950 50  0001 C CNN
 F 3 "~" H 2430 950 50  0001 C CNN
 	1    2400 950
@@
 F 0 "D15" H 2400 2075 50  0000 C CNN
 F 1 "APHB1608QBDSYKC" H 2400 1984 50  0000 C CNN
-F 2 "" H 2430 1650 50  0001 C CNN
+F 2 "Custom Parts:LED_Kingbright_APHB1608" H 2430 1650 50  0001 C CNN
 F 3 "~" H 2430 1650 50  0001 C CNN
 	1    2400 1650
@@
 F 0 "D16" H 2400 2775 50  0000 C CNN
 F 1 "APHB1608QBDSYKC" H 2400 2684 50  0000 C CNN
-F 2 "" H 2430 2350 50  0001 C CNN
+F 2 "Custom Parts:LED_Kingbright_APHB1608" H 2430 2350 50  0001 C CNN
 F 3 "~" H 2430 2350 50  0001 C CNN
 	1    2400 2350
@@
 F 0 "D17" H 2400 3525 50  0000 C CNN
 F 1 "APHB1608QBDSYKC" H 2400 3434 50  0000 C CNN
-F 2 "" H 2430 3100 50  0001 C CNN
+F 2 "Custom Parts:LED_Kingbright_APHB1608" H 2430 3100 50  0001 C CNN
 F 3 "~" H 2430 3100 50  0001 C CNN
 	1    2400 3100
@@
 F 0 "D18" H 5100 1375 50  0000 C CNN
 F 1 "APHB1608QBDCGKC" H 5100 1284 50  0000 C CNN
-F 2 "" H 5130 950 50  0001 C CNN
+F 2 "Custom Parts:LED_Kingbright_APHB1608" H 5130 950 50  0001 C CNN
 F 3 "~" H 5130 950 50  0001 C CNN
 	1    5100 950
@@
 F 0 "D19" H 5100 2075 50  0000 C CNN
 F 1 "APHB1608QBDCGKC" H 5100 1984 50  0000 C CNN
-F 2 "" H 5130 1650 50  0001 C CNN
+F 2 "Custom Parts:LED_Kingbright_APHB1608" H 5130 1650 50  0001 C CNN
 F 3 "~" H 5130 1650 50  0001 C CNN
 	1    5100 1650
@@
 F 0 "D20" H 5100 2775 50  0000 C CNN
 F 1 "APHB1608QBDCGKC" H 5100 2684 50  0000 C CNN
-F 2 "" H 5130 2350 50  0001 C CNN
+F 2 "Custom Parts:LED_Kingbright_APHB1608" H 5130 2350 50  0001 C CNN
 F 3 "~" H 5130 2350 50  0001 C CNN
 	1    5100 2350
@@
 F 0 "D21" H 5100 3525 50  0000 C CNN
 F 1 "APHB1608QBDCGKC" H 5100 3434 50  0000 C CNN
-F 2 "" H 5130 3100 50  0001 C CNN
+F 2 "Custom Parts:LED_Kingbright_APHB1608" H 5130 3100 50  0001 C CNN
 F 3 "~" H 5130 3100 50  0001 C CNN
 	1    5100 3100
@@
 F 0 "D22" H 7850 1375 50  0000 C CNN
 F 1 "APHB1608CGKSURKC" H 7850 1284 50  0000 C CNN
-F 2 "" H 7880 950 50  0001 C CNN
+F 2 "Custom Parts:LED_Kingbright_APHB1608" H 7880 950 50  0001 C CNN
 F 3 "~" H 7880 950 50  0001 C CNN
 	1    7850 950
@@
 F 0 "D23" H 7850 2075 50  0000 C CNN
 F 1 "APHB1608CGKSURKC" H 7850 1984 50  0000 C CNN
-F 2 "" H 7880 1650 50  0001 C CNN
+F 2 "Custom Parts:LED_Kingbright_APHB1608" H 7880 1650 50  0001 C CNN
 F 3 "~" H 7880 1650 50  0001 C CNN
 	1    7850 1650
@@
 F 0 "D24" H 7850 2775 50  0000 C CNN
 F 1 "APHB1608CGKSURKC" H 7850 2684 50  0000 C CNN
-F 2 "" H 7880 2350 50  0001 C CNN
+F 2 "Custom Parts:LED_Kingbright_APHB1608" H 7880 2350 50  0001 C CNN
 F 3 "~" H 7880 2350 50  0001 C CNN
 	1    7850 2350
@@
 F 0 "D25" H 7850 3525 50  0000 C CNN
 F 1 "APHB1608CGKSURKC" H 7850 3434 50  0000 C CNN
-F 2 "" H 7880 3100 50  0001 C CNN
+F 2 "Custom Parts:LED_Kingbright_APHB1608" H 7880 3100 50  0001 C CNN
 F 3 "~" H 7880 3100 50  0001 C CNN
 	1    7850 3100
@@
 F 0 "SW1" H 2550 5517 50  0000 C CNN
 F 1 " CHP-081TA" H 2550 5426 50  0000 C CNN
-F 2 "" H 2550 4850 50  0001 C CNN
+F 2 "Custom Parts:DipSW_CHP-081TA" H 2550 4850 50  0001 C CNN
 F 3 "" H 2550 4850 50  0001 C CNN
 	1    2550 4850

Commit message: hardware/mainboard: Change LEDs to larger Wurth 3528 LEDs
Signed-off-by: David Shah <dave@ds0.me>
Parts:
- D14, D15, D16, D17: value APHB1608QBDSYKC -> 150141YB73100; footprint Custom Parts:LED_Kingbright_APHB1608 -> Custom Parts:Wurth_BiLED_150141_3528; symbol Device:LED_Dual_ACAC -> Device:LED_Dual_AACC
- D18, D19: value APHB1608QBDCGKC -> 150141YB73100; footprint Custom Parts:LED_Kingbright_APHB1608 -> Custom Parts:Wurth_BiLED_150141_3528; symbol Device:LED_Dual_ACAC -> Device:LED_Dual_AACC
- D20, D21: value APHB1608QBDCGKC -> 150141RV73100; footprint Custom Parts:LED_Kingbright_APHB1608 -> Custom Parts:Wurth_BiLED_150141_3528; symbol Device:LED_Dual_ACAC -> Device:LED_Dual_AACC
- D22, D23, D24, D25: value APHB1608CGKSURKC -> 150141RV73100; footprint Custom Parts:LED_Kingbright_APHB1608 -> Custom Parts:Wurth_BiLED_150141_3528; symbol Device:LED_Dual_ACAC -> Device:LED_Dual_AACC
- RN11, RN7: value 1k -> 2.2k
Changed lines of the file:
@@
 $EndDescr
 $Comp
-L Device:LED_Dual_ACAC D14
+L Device:LED_Dual_AACC D14
 U 1 1 61049D89
 P 2400 950
 F 0 "D14" H 2400 1375 50  0000 C CNN
-F 1 "APHB1608QBDSYKC" H 2400 1284 50  0000 C CNN
-F 2 "Custom Parts:LED_Kingbright_APHB1608" H 2430 950 50  0001 C CNN
+F 1 " 150141YB73100" H 2400 1284 50  0000 C CNN
+F 2 "Custom Parts:Wurth_BiLED_150141_3528" H 2430 950 50  0001 C CNN
 F 3 "~" H 2430 950 50  0001 C CNN
 	1    2400 950
@@
 Wire Wire Line
 	2750 950  2750 850
-Text Notes 2000 850  0    50   ~ 0
-BLUE
-Text Notes 2500 1200 0    50   ~ 0
+Text Notes 2700 1150 0    50   ~ 0
+BLUE
+Text Notes 1950 850  0    50   ~ 0
 YELLOW
 Text GLabel 1950 1000 0    50   Input ~ 0
@@
 	2050 1000 2050 950
 $Comp
-L Device:LED_Dual_ACAC D15
+L Device:LED_Dual_AACC D15
 U 1 1 6104A4AF
 P 2400 1650
 F 0 "D15" H 2400 2075 50  0000 C CNN
-F 1 "APHB1608QBDSYKC" H 2400 1984 50  0000 C CNN
-F 2 "Custom Parts:LED_Kingbright_APHB1608" H 2430 1650 50  0001 C CNN
+F 1 " 150141YB73100" H 2400 1984 50  0000 C CNN
+F 2 "Custom Parts:Wurth_BiLED_150141_3528" H 2430 1650 50  0001 C CNN
 F 3 "~" H 2430 1650 50  0001 C CNN
 	1    2400 1650
@@
 Wire Wire Line
 	2750 1650 2750 1550
-Text Notes 2000 1550 0    50   ~ 0
-BLUE
-Text Notes 2500 1900 0    50   ~ 0
+Text Notes 2700 1850 0    50   ~ 0
+BLUE
+Text Notes 1950 1550 0    50   ~ 0
 YELLOW
 Text GLabel 1950 1700 0    50   Input ~ 0
@@
 	2050 1700 2050 1650
 $Comp
-L Device:LED_Dual_ACAC D16
+L Device:LED_Dual_AACC D16
 U 1 1 6104A7EB
 P 2400 2350
 F 0 "D16" H 2400 2775 50  0000 C CNN
-F 1 "APHB1608QBDSYKC" H 2400 2684 50  0000 C CNN
-F 2 "Custom Parts:LED_Kingbright_APHB1608" H 2430 2350 50  0001 C CNN
+F 1 " 150141YB73100" H 2400 2684 50  0000 C CNN
+F 2 "Custom Parts:Wurth_BiLED_150141_3528" H 2430 2350 50  0001 C CNN
 F 3 "~" H 2430 2350 50  0001 C CNN
 	1    2400 2350
@@
 Wire Wire Line
 	2750 2350 2750 2250
-Text Notes 2000 2250 0    50   ~ 0
-BLUE
-Text Notes 2500 2600 0    50   ~ 0
+Text Notes 2650 2550 0    50   ~ 0
+BLUE
+Text Notes 1950 2250 0    50   ~ 0
 YELLOW
 Text GLabel 1950 2400 0    50   Input ~ 0
@@
 	2050 2400 2050 2350
 $Comp
-L Device:LED_Dual_ACAC D17
+L Device:LED_Dual_AACC D17
 U 1 1 6104AE36
 P 2400 3100
 F 0 "D17" H 2400 3525 50  0000 C CNN
-F 1 "APHB1608QBDSYKC" H 2400 3434 50  0000 C CNN
-F 2 "Custom Parts:LED_Kingbright_APHB1608" H 2430 3100 50  0001 C CNN
+F 1 " 150141YB73100" H 2400 3434 50  0000 C CNN
+F 2 "Custom Parts:Wurth_BiLED_150141_3528" H 2430 3100 50  0001 C CNN
 F 3 "~" H 2430 3100 50  0001 C CNN
 	1    2400 3100
@@
 Wire Wire Line
 	2750 3100 2750 3000
-Text Notes 2000 3000 0    50   ~ 0
-BLUE
-Text Notes 2500 3350 0    50   ~ 0
+Text Notes 2650 3300 0    50   ~ 0
+BLUE
+Text Notes 1950 3000 0    50   ~ 0
 YELLOW
 Text GLabel 1950 3150 0    50   Input ~ 0
@@
 	2050 3150 2050 3100
 $Comp
-L Device:LED_Dual_ACAC D18
+L Device:LED_Dual_AACC D18
 U 1 1 6104D817
 P 5100 950
 F 0 "D18" H 5100 1375 50  0000 C CNN
-F 1 "APHB1608QBDCGKC" H 5100 1284 50  0000 C CNN
-F 2 "Custom Parts:LED_Kingbright_APHB1608" H 5130 950 50  0001 C CNN
+F 1 " 150141YB73100" H 5100 1284 50  0000 C CNN
+F 2 "Custom Parts:Wurth_BiLED_150141_3528" H 5130 950 50  0001 C CNN
 F 3 "~" H 5130 950 50  0001 C CNN
 	1    5100 950
@@
 Wire Wire Line
 	5450 950  5450 850
-Text Notes 4700 850  0    50   ~ 0
-BLUE
-Text Notes 5200 1200 0    50   ~ 0
-GREEN
+Text Notes 5350 1150 0    50   ~ 0
+BLUE
+Text Notes 4650 850  0    50   ~ 0
+YELLOW
 Text GLabel 4650 1000 0    50   Input ~ 0
 LED4
@@
 	4750 1000 4750 950
 $Comp
-L Device:LED_Dual_ACAC D19
+L Device:LED_Dual_AACC D19
 U 1 1 610547CD
 P 5100 1650
 F 0 "D19" H 5100 2075 50  0000 C CNN
-F 1 "APHB1608QBDCGKC" H 5100 1984 50  0000 C CNN
-F 2 "Custom Parts:LED_Kingbright_APHB1608" H 5130 1650 50  0001 C CNN
+F 1 " 150141YB73100" H 5100 1984 50  0000 C CNN
+F 2 "Custom Parts:Wurth_BiLED_150141_3528" H 5130 1650 50  0001 C CNN
 F 3 "~" H 5130 1650 50  0001 C CNN
 	1    5100 1650
@@
 Wire Wire Line
 	5450 1650 5450 1550
-Text Notes 4700 1550 0    50   ~ 0
-BLUE
-Text Notes 5200 1900 0    50   ~ 0
-GREEN
+Text Notes 5350 1850 0    50   ~ 0
+BLUE
+Text Notes 4650 1550 0    50   ~ 0
+YELLOW
 Text GLabel 4650 1700 0    50   Input ~ 0
 LED5
@@
 	4750 1700 4750 1650
 $Comp
-L Device:LED_Dual_ACAC D20
+L Device:LED_Dual_AACC D20
 U 1 1 61055BAD
 P 5100 2350
 F 0 "D20" H 5100 2775 50  0000 C CNN
-F 1 "APHB1608QBDCGKC" H 5100 2684 50  0000 C CNN
-F 2 "Custom Parts:LED_Kingbright_APHB1608" H 5130 2350 50  0001 C CNN
+F 1 "150141RV73100" H 5100 2684 50  0000 C CNN
+F 2 "Custom Parts:Wurth_BiLED_150141_3528" H 5130 2350 50  0001 C CNN
 F 3 "~" H 5130 2350 50  0001 C CNN
 	1    5100 2350
@@
 	5450 2350 5450 2250
 Text Notes 4700 2250 0    50   ~ 0
-BLUE
+RED
 Text Notes 5200 2600 0    50   ~ 0
 GREEN
@@
 	4750 2400 4750 2350
 $Comp
-L Device:LED_Dual_ACAC D21
+L Device:LED_Dual_AACC D21
 U 1 1 610575DB
 P 5100 3100
 F 0 "D21" H 5100 3525 50  0000 C CNN
-F 1 "APHB1608QBDCGKC" H 5100 3434 50  0000 C CNN
-F 2 "Custom Parts:LED_Kingbright_APHB1608" H 5130 3100 50  0001 C CNN
+F 1 "150141RV73100" H 5100 3434 50  0000 C CNN
+F 2 "Custom Parts:Wurth_BiLED_150141_3528" H 5130 3100 50  0001 C CNN
 F 3 "~" H 5130 3100 50  0001 C CNN
 	1    5100 3100
@@
 	5450 3100 5450 3000
 Text Notes 4700 3000 0    50   ~ 0
-BLUE
+RED
 Text Notes 5200 3350 0    50   ~ 0
 GREEN
@@
 	4750 3150 4750 3100
 $Comp
-L Device:LED_Dual_ACAC D22
+L Device:LED_Dual_AACC D22
 U 1 1 61061FE6
 P 7850 950
 F 0 "D22" H 7850 1375 50  0000 C CNN
-F 1 "APHB1608CGKSURKC" H 7850 1284 50  0000 C CNN
-F 2 "Custom Parts:LED_Kingbright_APHB1608" H 7880 950 50  0001 C CNN
+F 1 "150141RV73100" H 7850 1284 50  0000 C CNN
+F 2 "Custom Parts:Wurth_BiLED_150141_3528" H 7880 950 50  0001 C CNN
 F 3 "~" H 7880 950 50  0001 C CNN
 	1    7850 950
@@
 	7500 1000 7500 950
 $Comp
-L Device:LED_Dual_ACAC D23
+L Device:LED_Dual_AACC D23
 U 1 1 6106ADE3
 P 7850 1650
 F 0 "D23" H 7850 2075 50  0000 C CNN
-F 1 "APHB1608CGKSURKC" H 7850 1984 50  0000 C CNN
-F 2 "Custom Parts:LED_Kingbright_APHB1608" H 7880 1650 50  0001 C CNN
+F 1 "150141RV73100" H 7850 1984 50  0000 C CNN
+F 2 "Custom Parts:Wurth_BiLED_150141_3528" H 7880 1650 50  0001 C CNN
 F 3 "~" H 7880 1650 50  0001 C CNN
 	1    7850 1650
@@
 	7500 1700 7500 1650
 $Comp
-L Device:LED_Dual_ACAC D24
+L Device:LED_Dual_AACC D24
 U 1 1 6106FCCD
 P 7850 2350
 F 0 "D24" H 7850 2775 50  0000 C CNN
-F 1 "APHB1608CGKSURKC" H 7850 2684 50  0000 C CNN
-F 2 "Custom Parts:LED_Kingbright_APHB1608" H 7880 2350 50  0001 C CNN
+F 1 "150141RV73100" H 7850 2684 50  0000 C CNN
+F 2 "Custom Parts:Wurth_BiLED_150141_3528" H 7880 2350 50  0001 C CNN
 F 3 "~" H 7880 2350 50  0001 C CNN
 	1    7850 2350
@@
 	7500 2400 7500 2350
 $Comp
-L Device:LED_Dual_ACAC D25
+L Device:LED_Dual_AACC D25
 U 1 1 61073A02
 P 7850 3100
 F 0 "D25" H 7850 3525 50  0000 C CNN
-F 1 "APHB1608CGKSURKC" H 7850 3434 50  0000 C CNN
-F 2 "Custom Parts:LED_Kingbright_APHB1608" H 7880 3100 50  0001 C CNN
+F 1 "150141RV73100" H 7850 3434 50  0000 C CNN
+F 2 "Custom Parts:Wurth_BiLED_150141_3528" H 7880 3100 50  0001 C CNN
 F 3 "~" H 7880 3100 50  0001 C CNN
 	1    7850 3100
@@
 P 1250 1050
 F 0 "RN7" V 833 1050 50  0000 C CNN
-F 1 "1k" V 924 1050 50  0000 C CNN
+F 1 "2.2k" V 924 1050 50  0000 C CNN
 F 2 "Resistor_SMD:R_Array_Convex_4x0402" V 1525 1050 50  0001 C CNN
 F 3 "~" H 1250 1050 50  0001 C CNN
@@
 P 3950 1050
 F 0 "RN11" V 3533 1050 50  0000 C CNN
-F 1 "1k" V 3624 1050 50  0000 C CNN
+F 1 "2.2k" V 3624 1050 50  0000 C CNN
 F 2 "Resistor_SMD:R_Array_Convex_4x0402" V 4225 1050 50  0001 C CNN
 F 3 "~" H 3950 1050 50  0001 C CNN
