File: hardware/ecp5_mainboard/ports.sch (KiCad schematic (older format))
At the start: 93 parts

Commit message: hardware/mainboard: Re-annotate and fix ERC
Signed-off-by: David Shah <dave@ds0.me>
Parts:
- gave numbers to parts that had none: 93
Connections:
- net +1V2: now also C162.1

Commit message: hardware/mainboard: add microSD
Signed-off-by: David Shah <dave@ds0.me>
Parts:
- added C?: 10µ, symbol Device:C_Small
- added J?: Micro_SD_Card, symbol Connector:Micro_SD_Card
- added R?: 10k, symbol Device:R_Small
- added RN?: 10k, symbol Device:R_Pack04
Connections:
- net +3V3: now also C?.1, J?.4 (VDD), R?.1, RN?.5 (R4.2), RN?.6 (R3.2), RN?.7 (R2.2), RN?.8 (R1.2)
- net GND: now also C?.2, J?.6 (VSS), J?.9 (SHIELD)
- new net USD_CLK: J?.5 (CLK)
- new net USD_CMD: J?.3 (CMD), RN?.3 (R3.1)
- new net USD_D0: J?.7 (DAT0), RN?.4 (R4.1)
- new net USD_D1: J?.8 (DAT1), R?.2
- new net USD_D2: J?.1 (DAT2), RN?.1 (R1.1)
- new net USD_D3: J?.2 (DAT3/CD), RN?.2 (R2.1)
Other:
- moved on the sheet: C132, C133, C134, C135, P4, R63, R64

Commit message: hardware/mainboard: Assign some footprints
Signed-off-by: David Shah <dave@ds0.me>
Parts:
- C119, C120, C123, C124, C125: footprint (none) -> Capacitor_SMD:C_0805_2012Metric
- C121, C122, C126, C127, C128, C129, C130, C131, C132, C133, C134, C135, C136, C140, C141, C143, C144, C145, C146, C147, C148, C149, C150, C151, C152, C153, C154, C155, C156, C157, C158, C159, C160, C162, C163, C166, C167, C168, C169, C170, C171: footprint (none) -> Capacitor_SMD:C_0402_1005Metric
- C138, C139, C142, C161, C164, C165, C172, C173: footprint (none) -> Capacitor_SMD:C_0603_1608Metric
- C255: renamed from C?; footprint (none) -> Capacitor_SMD:C_0805_2012Metric
- FB4, FB5, FB6, FB7, FB8, FB9: footprint (none) -> Inductor_SMD:L_0603_1608Metric
- R59, R60, R61, R62, R63, R64, R65, R66, R67, R68, R69, R70, R71, R72, R73, R74: footprint (none) -> Resistor_SMD:R_0402_1005Metric
- R96: renamed from R?; footprint (none) -> Resistor_SMD:R_0402_1005Metric
- RN24: renamed from RN?; footprint (none) -> Resistor_SMD:R_Array_Convex_4x0402
- RN4, RN5, RN6: footprint (none) -> Resistor_SMD:R_Array_Convex_4x0402
- U18: footprint (none) -> Package_SO:VSSOP-8_2.3x2mm_P0.5mm
- U19: footprint (none) -> Package_QFP:HTQFP-64-1EP_10x10mm_P0.5mm_EP8x8mm_Mask4.4x4.4mm_ThermalVias
- gave numbers to parts that had none: 1

Commit message: hardware: Adding USB-A and MagJack footprints
Signed-off-by: David Shah <dave@ds0.me>
Parts:
- P4: value JK0654219 -> JK0654219NL
Changed lines of the file:
@@
 P 5300 1700
 F 0 "P4" H 5194 2765 50  0000 C CNN
-F 1 "JK0654219" H 5194 2674 50  0000 C CNN
+F 1 "JK0654219NL" H 5194 2674 50  0000 C CNN
 F 2 "" H 6450 1400 50  0001 C CNN
 F 3 "" H 6450 1400 50  0001 C CNN

Commit message: hardware/mainboard: Assign more footprints
Signed-off-by: David Shah <dave@ds0.me>
Parts:
- C137: footprint (none) -> Capacitor_SMD:CP_Elec_6.3x5.8
- DA5, DA6: footprint (none) -> Custom Parts:USON10
- J13: footprint (none) -> Connector_Card:microSD_HC_Hirose_DM3AT-SF-PEJM5
- J4: footprint (none) -> Custom Parts:292303-7
- P4: footprint (none) -> Custom Parts:Pulse_MagJack_JK0654219NL
Changed lines of the file:
@@
 F 0 "P4" H 5194 2765 50  0000 C CNN
 F 1 "JK0654219NL" H 5194 2674 50  0000 C CNN
-F 2 "" H 6450 1400 50  0001 C CNN
+F 2 "Custom Parts:Pulse_MagJack_JK0654219NL" H 6450 1400 50  0001 C CNN
 F 3 "" H 6450 1400 50  0001 C CNN
 	1    5300 1700
@@
 F 0 "J4" H 12155 9717 50  0000 C CNN
 F 1 "USB_A" H 12155 9626 50  0000 C CNN
-F 2 "" H 12250 9200 50  0001 C CNN
+F 2 "Custom Parts:292303-7" H 12250 9200 50  0001 C CNN
 F 3 " ~" H 12250 9200 50  0001 C CNN
 	1    12100 9250
@@
 F 0 "C137" H 9088 7596 50  0000 L CNN
 F 1 "100u" H 9088 7505 50  0000 L CNN
-F 2 "" H 9000 7550 50  0001 C CNN
+F 2 "Capacitor_SMD:CP_Elec_6.3x5.8" H 9000 7550 50  0001 C CNN
 F 3 "~" H 9000 7550 50  0001 C CNN
 	1    9000 7550
@@
 F 0 "DA5" H 4800 5237 60  0000 C CNN
 F 1 "TPD4E02B04" H 4800 5131 60  0000 C CNN
-F 2 "" H 4800 4450 60  0001 C CNN
+F 2 "Custom Parts:USON10" H 4800 4450 60  0001 C CNN
 F 3 "" H 4800 4450 60  0001 C CNN
 	1    4800 4450
@@
 F 0 "DA6" H 6500 5237 60  0000 C CNN
 F 1 "TPD4E02B04" H 6500 5131 60  0000 C CNN
-F 2 "" H 6500 4450 60  0001 C CNN
+F 2 "Custom Parts:USON10" H 6500 4450 60  0001 C CNN
 F 3 "" H 6500 4450 60  0001 C CNN
 	1    6500 4450
@@
 F 0 "J13" H 1500 2267 50  0000 C CNN
 F 1 "Micro_SD_Card" H 1500 2176 50  0000 C CNN
-F 2 "" H 2700 1850 50  0001 C CNN
+F 2 "Connector_Card:microSD_HC_Hirose_DM3AT-SF-PEJM5" H 2700 1850 50  0001 C CNN
 F 3 "http://katalog.we-online.de/em/datasheet/693072010801.pdf" H 1550 1550 50  0001 C CNN
 	1    1550 1550

Commit message: hardware/mainboard: More footprint assignment, other small tweaks
Signed-off-by: David Shah <dave@ds0.me>
Parts:
- J3: footprint (none) -> Custom Parts:Molex_HDMI_A_47151-0001
- Y2, Y3: footprint (none) -> Custom Parts:Crystal_Epsom_TSX-3225
Changed lines of the file:
@@
 F 0 "Y2" H 9300 4968 50  0000 C CNN
 F 1 "25MHz" H 9300 4877 50  0000 C CNN
-F 2 "" H 9300 4700 50  0001 C CNN
+F 2 "Custom Parts:Crystal_Epsom_TSX-3225" H 9300 4700 50  0001 C CNN
 F 3 "~" H 9300 4700 50  0001 C CNN
 	1    9300 4700
@@
 F 0 "Y3" H 11950 8118 50  0000 C CNN
 F 1 "24MHz" H 11950 8027 50  0000 C CNN
-F 2 "" H 11950 7850 50  0001 C CNN
+F 2 "Custom Parts:Crystal_Epsom_TSX-3225" H 11950 7850 50  0001 C CNN
 F 3 "~" H 11950 7850 50  0001 C CNN
 	1    11950 7850
@@
 F 0 "J3" H 2380 7296 50  0000 L CNN
 F 1 "HDMI_A" H 2380 7205 50  0000 L CNN
-F 2 "" H 1975 7250 50  0001 C CNN
+F 2 "Custom Parts:Molex_HDMI_A_47151-0001" H 1975 7250 50  0001 C CNN
 F 3 "https://en.wikipedia.org/wiki/HDMI" H 1975 7250 50  0001 C CNN
 	1    1950 7250

Commit message: hardware/mainboard: Small design tweaks
Signed-off-by: David Shah <dave@ds0.me>
Parts:
- C144, C145, C146, C148, C149, C150, C152, C153, C154, C155, C157, C158, C160: footprint Capacitor_SMD:C_0402_1005Metric -> Capacitor_SMD:C_0201_0603Metric
Changed lines of the file:
@@
 F 0 "C155" H 12942 1746 50  0000 L CNN
 F 1 "10n" H 12942 1655 50  0000 L CNN
-F 2 "Capacitor_SMD:C_0402_1005Metric" H 12850 1700 50  0001 C CNN
+F 2 "Capacitor_SMD:C_0201_0603Metric" H 12850 1700 50  0001 C CNN
 F 3 "~" H 12850 1700 50  0001 C CNN
 	1    12850 1700
@@
 F 0 "C158" H 13242 1746 50  0000 L CNN
 F 1 "10n" H 13242 1655 50  0000 L CNN
-F 2 "Capacitor_SMD:C_0402_1005Metric" H 13150 1700 50  0001 C CNN
+F 2 "Capacitor_SMD:C_0201_0603Metric" H 13150 1700 50  0001 C CNN
 F 3 "~" H 13150 1700 50  0001 C CNN
 	1    13150 1700
@@
 F 0 "C160" H 13542 1746 50  0000 L CNN
 F 1 "10n" H 13542 1655 50  0000 L CNN
-F 2 "Capacitor_SMD:C_0402_1005Metric" H 13450 1700 50  0001 C CNN
+F 2 "Capacitor_SMD:C_0201_0603Metric" H 13450 1700 50  0001 C CNN
 F 3 "~" H 13450 1700 50  0001 C CNN
 	1    13450 1700
@@
 F 0 "C154" H 12942 1346 50  0000 L CNN
 F 1 "10n" H 12942 1255 50  0000 L CNN
-F 2 "Capacitor_SMD:C_0402_1005Metric" H 12850 1300 50  0001 C CNN
+F 2 "Capacitor_SMD:C_0201_0603Metric" H 12850 1300 50  0001 C CNN
 F 3 "~" H 12850 1300 50  0001 C CNN
 	1    12850 1300
@@
 F 0 "C157" H 13242 1346 50  0000 L CNN
 F 1 "10n" H 13242 1255 50  0000 L CNN
-F 2 "Capacitor_SMD:C_0402_1005Metric" H 13150 1300 50  0001 C CNN
+F 2 "Capacitor_SMD:C_0201_0603Metric" H 13150 1300 50  0001 C CNN
 F 3 "~" H 13150 1300 50  0001 C CNN
 	1    13150 1300
@@
 F 0 "C153" H 12792 946 50  0000 L CNN
 F 1 "10n" H 12792 855 50  0000 L CNN
-F 2 "Capacitor_SMD:C_0402_1005Metric" H 12700 900 50  0001 C CNN
+F 2 "Capacitor_SMD:C_0201_0603Metric" H 12700 900 50  0001 C CNN
 F 3 "~" H 12700 900 50  0001 C CNN
 	1    12700 900
@@
 F 0 "C152" H 12542 946 50  0000 L CNN
 F 1 "10n" H 12542 855 50  0000 L CNN
-F 2 "Capacitor_SMD:C_0402_1005Metric" H 12450 900 50  0001 C CNN
+F 2 "Capacitor_SMD:C_0201_0603Metric" H 12450 900 50  0001 C CNN
 F 3 "~" H 12450 900 50  0001 C CNN
 	1    12450 900
@@
 F 0 "C150" H 12292 946 50  0000 L CNN
 F 1 "10n" H 12292 855 50  0000 L CNN
-F 2 "Capacitor_SMD:C_0402_1005Metric" H 12200 900 50  0001 C CNN
+F 2 "Capacitor_SMD:C_0201_0603Metric" H 12200 900 50  0001 C CNN
 F 3 "~" H 12200 900 50  0001 C CNN
 	1    12200 900
@@
 F 0 "C149" H 12042 946 50  0000 L CNN
 F 1 "10n" H 12042 855 50  0000 L CNN
-F 2 "Capacitor_SMD:C_0402_1005Metric" H 11950 900 50  0001 C CNN
+F 2 "Capacitor_SMD:C_0201_0603Metric" H 11950 900 50  0001 C CNN
 F 3 "~" H 11950 900 50  0001 C CNN
 	1    11950 900
@@
 F 0 "C148" H 11792 946 50  0000 L CNN
 F 1 "10n" H 11792 855 50  0000 L CNN
-F 2 "Capacitor_SMD:C_0402_1005Metric" H 11700 900 50  0001 C CNN
+F 2 "Capacitor_SMD:C_0201_0603Metric" H 11700 900 50  0001 C CNN
 F 3 "~" H 11700 900 50  0001 C CNN
 	1    11700 900
@@
 F 0 "C144" H 9792 946 50  0000 L CNN
 F 1 "10n" H 9792 855 50  0000 L CNN
-F 2 "Capacitor_SMD:C_0402_1005Metric" H 9700 900 50  0001 C CNN
+F 2 "Capacitor_SMD:C_0201_0603Metric" H 9700 900 50  0001 C CNN
 F 3 "~" H 9700 900 50  0001 C CNN
 	1    9700 900
@@
 F 0 "C146" H 10092 946 50  0000 L CNN
 F 1 "10n" H 10092 855 50  0000 L CNN
-F 2 "Capacitor_SMD:C_0402_1005Metric" H 10000 900 50  0001 C CNN
+F 2 "Capacitor_SMD:C_0201_0603Metric" H 10000 900 50  0001 C CNN
 F 3 "~" H 10000 900 50  0001 C CNN
 	1    10000 900
@@
 F 0 "C145" H 9608 1254 50  0000 R CNN
 F 1 "10n" H 9608 1345 50  0000 R CNN
-F 2 "Capacitor_SMD:C_0402_1005Metric" H 9700 1300 50  0001 C CNN
+F 2 "Capacitor_SMD:C_0201_0603Metric" H 9700 1300 50  0001 C CNN
 F 3 "~" H 9700 1300 50  0001 C CNN
 	1    9700 1300
