File: hardware/ecp5_mainboard/ports.sch (KiCad schematic (older format))
At the start: 97 parts, among them J13 Micro_SD_Card, J3 HDMI_A, J4 USB_A, P4 JK0654219NL, U17 TPS2041B, U18 PCA9306, U19 TFP410, U20 TPS2041B, U21 KSZ9031RNXCA, U22 USB3300-EZK, Y2 25MHz, Y3 24MHz

Commit message: hardware/mainboard: Add and place M.2 connector footprint
Signed-off-by: David Shah <davey1576@gmail.com>
Parts:
- U19: symbol pkl_texas:TFP410 -> ecp5_mainboard-rescue:TFP410-pkl_texas
Changed lines of the file:
@@
 	10800 6700 10800 6750
 $Comp
-L pkl_texas:TFP410 U19
+L ecp5_mainboard-rescue:TFP410-pkl_texas U19
 U 1 1 5DD5619A
 P 6450 8000
